File: F0-nolib/Chiller/kicad/Chiller_control.sch (KiCad schematic (older format))
At the start: 53 parts, among them J1 DB9_Female, J2 12VIN, J3 Ext. devices, J4 Tsens, J5 Cooler, J6 Heater, J7 Pump, Q1 SI2300, Q2 SI2300, Q3 SI2300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

Commit message: Chiller works
Parts:
- C1, C10, C11, C12, C13, C2, C3, C5, C6, C7, C8, C9: symbol C -> Chiller_control-rescue:C
- C4: symbol CP -> Chiller_control-rescue:CP
- D1: symbol D -> Chiller_control-rescue:D
- J1: symbol DB9_Female -> Chiller_control-rescue:DB9_Female
- J2, J5, J6, J7: symbol Conn_01x02 -> Chiller_control-rescue:Conn_01x02
- J3: symbol Conn_02x07_Odd_Even -> Chiller_control-rescue:Conn_02x07_Odd_Even
- J4: symbol Conn_02x04_Odd_Even -> Chiller_control-rescue:Conn_02x04_Odd_Even
- L1: symbol L -> Chiller_control-rescue:L
- Q1, Q2, Q3: symbol Q_NMOS_GSD -> Chiller_control-rescue:Q_NMOS_GSD
- Q4, Q5: symbol Q_NMOS_GDS -> Chiller_control-rescue:Q_NMOS_GDS
- R1, R10, R11, R12, R13, R14, R15, R16, R17, R18, R19, R2, R20, R21, R3, R4, R5, R6, R7, R8, R9: symbol R -> Chiller_control-rescue:R
- SW1, SW2: symbol SW_Push -> Chiller_control-rescue:SW_Push
- U1: symbol LM1117-3.3 -> Chiller_control-rescue:LM1117-3.3
- U2: symbol MAX3232 -> Chiller_control-rescue:MAX3232
- U3: symbol STM32F030F4Px -> Chiller_control-rescue:STM32F030F4Px

Commit message: Change chiller schematics: fix bugs, prepare for manufacture production
Parts:
- removed J3: Ext. devices, Connector_PinSocket_2.54mm:PinSocket_2x07_P2.54mm_Vertical, symbol Chiller_control-rescue:Conn_02x07_Odd_Even
- removed J4: Tsens, Connector_PinSocket_2.54mm:PinSocket_2x04_P2.54mm_Vertical, symbol Chiller_control-rescue:Conn_02x04_Odd_Even
- added BZ1: Buzzer, Buzzer_Beeper:Buzzer_12x9.5RM7.6, symbol Device:Buzzer
- added C14, C16: 1u, Capacitor_SMD:C_0805_2012Metric_Pad1.29x1.40mm_HandSolder, symbol Chiller_control-rescue:C
- added C15: 100u, Capacitor_THT:CP_Radial_D8.0mm_P3.50mm, symbol Chiller_control-rescue:CP
- added C17, C18, C19, C20, C21: 0.1, Capacitor_SMD:C_0603_1608Metric_Pad0.99x1.00mm_HandSolder, symbol Chiller_control-rescue:C
- added J3, J4: DC3-10P, Connector_IDC:IDC-Header_2x05_P2.54mm_Vertical, symbol Connector_Generic:Conn_02x05_Odd_Even
- added R22, R23, R26: 220, Resistor_SMD:R_0805_2012Metric_Pad1.29x1.40mm_HandSolder, symbol Chiller_control-rescue:R
- added R24, R25: 0, Resistor_SMD:R_0805_2012Metric_Pad1.29x1.40mm_HandSolder, symbol Chiller_control-rescue:R
- added U4: L7805, TO_SOT_Packages_THT:TO-220-3_Vertical, symbol Regulator_Linear:L7805
- C1, C12, C2, C3, C5, C8, C9: footprint Capacitor_SMD.pretty:C_0603_HandSoldering -> Capacitor_SMD:C_0603_1608Metric_Pad0.99x1.00mm_HandSolder
- Q4, Q5: footprint TO_SOT_Packages_THT:TO-220_Horizontal -> TO_SOT_Packages_THT:TO-220-3_Vertical
- R11: value 47 -> 220
- R7: value 47 -> 220; footprint Resistors_SMD.pretty:R_0805_HandSoldering -> Resistor_SMD:R_0805_2012Metric_Pad1.29x1.40mm_HandSolder
Connections:
- net labels added: +5V, IN, Out1, Out2
- net labels removed: Alrm, EF, In1, In2
- wire segments 130 -> 165
Other:
- note added: "*"
- note added: "* Solder R6,\nR8 and R9\nif necessary"
- note added: "5/3.3V MCU power source"
- note added: "Alarm Buzzer"
- note added: "DIG in/out"
- note added: "EXT in/out"
- note added: "Solder only\nR24 or R25"
- note removed: "3.3V MCU power source\nwith short-circuit protection"
- note removed: "TLE5205"
- note removed: "TLE5205\nFor Peltier"
- moved on the sheet: C10, C11, C12, C13, C3, C4, C5, C8, C9, J1, Q1, Q2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
