File: F0-nolib/Servo/kicad/Servo_control.kicad_pcb (KiCad board)
At the start: 2 copper layers, 58 parts, among them J1 USB_B_Micro, J2 ADC_in, J3 Jumper0, J4 Jumper1, J5 Conn_01x03, J6 Ext_LED, J7 Servo1, J8 Servo2, J9 Servo3, Q1 2N7002, Q2 SI2300, Q3 2N7002, Q4 2N7002, Q5 2N7002, SW1 Reset, SW2 Boot, U1 LM1117-3.3, U2 CH340G, U3 STM32F030F4Px, U4 STM32F030F4Px, Y1 12MHz

Commit message: draw servo-control PCB
Parts:
- removed U4: STM32F030F4Px, Package_SSOP:TSSOP-20_4.4x6.5mm_P0.65mm
- added D5: SS14, Diode_SMD:D_SMA_Handsoldering, F.Cu at (181.3, 59.8)
- added J10: 5V, Connector_PinHeader_2.54mm:PinHeader_1x02_P2.54mm_Vertical, F.Cu at (173.6, 77.0)
- added REF**: VIA, modules:VIA, F.Cu at (159.6, 53.0)
- added REF**: VIA, modules:VIA, F.Cu at (187.2, 67.0)
- added REF**: VIA, modules:VIA, F.Cu at (168.7, 44.6)
- added REF**: VIA, modules:VIA, F.Cu at (192.4, 46.6)
- C1, C12, C14, C4, C5, C6, C7, C8, C9, D1, D2, J1, Q1, Q2, Q3, Q4, Q5, R12, R13, R14, R15, R16, R17, R2, R3, R4, R5, R6, R7, R8, R9, U2: moved to B.Cu
- J5: value Conn_01x03 -> Dig_In
- U1: footprint Package_TO_SOT_SMD:SOT-223 -> Package_TO_SOT_SMD:SOT-223-3_TabPin2; moved to B.Cu
- moved R4 167.3 mm to (154.3, 57.7), turned to 180 degrees
- moved C12 164.4 mm to (157.5, 49.5), turned to 90 degrees
- moved C11 163.7 mm to (154.1, 55.2), turned to 180 degrees
- moved R5 163.0 mm to (154.3, 60.3), turned to 180 degrees
- moved R2 162.0 mm to (154.3, 52.6), turned to 180 degrees
- moved C10 159.7 mm to (154.1, 57.7), turned to 180 degrees
- moved J3 157.3 mm to (161.1, 77.0), turned to 180 degrees
- moved R3 156.2 mm to (154.3, 55.2), turned to 180 degrees
- moved J2 154.9 mm to (149.4, 62.8), turned to 180 degrees
- moved D2 151.9 mm to (161.0, 56.0), turned to 270 degrees
- moved J4 151.1 mm to (165.3, 76.9), turned to 180 degrees
- moved C4 150.1 mm to (184.5, 45.3), turned to 270 degrees
- moved C5 144.2 mm to (187.1, 45.5), turned to 270 degrees
- moved C9 141.0 mm to (169.6, 67.8), turned to 90 degrees
- moved U1 138.2 mm to (178.7, 46.1), turned to 90 degrees
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Connections:
- BZ1 pad 1: +3V3 -> +5V
- D1 pad 8: +5V -> Net-(D1-Pad8)
- D2 pad 1: /ADC0 -> /ADC1
- D2 pad 3: /ADC1 -> /ADC0
- D2 pad 4: /ADC2 -> /ADC3
- D2 pad 5: /ADC3 -> /ADC2
- J2 pad 6: +3V3 -> +3.3VADC
- U3 pad 10: /DigIn0 -> /Jumper0
- U3 pad 11: /DigIn1 -> /Jumper1
- U3 pad 19: /Jumper0 -> /DigIn0
- U3 pad 20: /Jumper1 -> /DigIn1
Routing:
- net GND: track 5.72 -> 484.6 mm
- net +5V: track 0.00 -> 180.2 mm, vias 0 -> 2
- net +3V3: track 5.74 -> 83.8 mm, vias 0 -> 3
- net /DigOut0: track 0.00 -> 36.7 mm, vias 0 -> 1
- net +3.3VADC: track 0.00 -> 34.6 mm, vias 0 -> 1
- net /DigIn0: track 0.00 -> 29.9 mm
- net /TIM3_CH2: track 0.00 -> 25.9 mm, vias 0 -> 1
- net Net-(D1-Pad4): track 0.00 -> 24.4 mm
- net /NRST: track 0.00 -> 22.1 mm
- net /Jumper1: track 0.00 -> 22.0 mm, vias 0 -> 1
- net /Jumper0: track 0.00 -> 21.9 mm, vias 0 -> 1
- net /ADC0: track 0.00 -> 20.6 mm, vias 0 -> 1
- net /TIM3_CH4: track 0.00 -> 20.3 mm, vias 0 -> 1
- net /DigIn1: track 0.00 -> 20.0 mm
- net /ADC3: track 0.00 -> 18.2 mm, vias 0 -> 1
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- added copper zone on B.Cu, net GND
- added copper zone on F.Cu, net GND
Other:
- board outline added: 53 x 47 mm
- net class 2: trace_width 2 -> 1
- board text added: "#1"
- board text added: "#2"
- board text added: "#3"
- board text added: "+"
- board text added: "+ -"
- board text added: "+ 0 1 2 3"
- board text added: "+ 0 1 2 3 gnd"
- board text added: "-5v+"
- board text added: "1 + s"
- board text added: "1 0 gnd"
- board text added: "1-2"
- board text added: "2 + s"
- board text added: "3 + s"
- board text added: "5V in - +"
- board text added: "ADC"
- board text added: "BOOT"
- board text added: "Boot"
- board text added: "DigIn"
- board text added: "J1"
- board text added: "J2"
- board text added: "LED"
- board text added: "RESET"
- board text added: "gnd +5 sig"
