File: F1-nolib/chronometer_v1/kicad/chrono.sch (KiCad schematic (older format))
At the start: 83 parts, among them J1 Power 12V, J10 LIDAR, J11 Bluetooth, J12 SWD, J2 GPS_ext, J3 PPS, J4 Ext_trig1, J5 Ext_trig0, J6 USB_B_Mini, J7 Ext_trig2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

Commit message: Add SPI DMA Tx example
Parts:
- D2, D6: value IN5819 -> 1N5819
Changed lines of the file:
@@
 P 2375 3050
 F 0 "D2" H 2350 2875 50  0000 C CNN
-F 1 "IN5819" H 2375 2950 50  0000 C CNN
+F 1 "1N5819" H 2375 2950 50  0000 C CNN
 F 2 "Diode_SMD:D_SOD-323" H 2375 3050 50  0001 C CNN
 F 3 "~" H 2375 3050 50  0001 C CNN
@@
 P 3275 2325
 F 0 "D6" V 3175 2250 50  0000 C CNN
-F 1 "IN5819" H 3250 2425 50  0000 C CNN
+F 1 "1N5819" H 3250 2425 50  0000 C CNN
 F 2 "Diode_SMD:D_SOD-323" H 3275 2325 50  0001 C CNN
 F 3 "~" H 3275 2325 50  0001 C CNN
