File: F0-nolib/canbus/kicad/stm32.sch (KiCad schematic (older format))
At the start: 61 parts, among them J1 CONN_02X03, J2 DB9_Female, J3 DB9_Male, J4 Conn_01x07, J5 12v, J6 Conn_01x01, P12 USART_BOOT, P13 USB_A, P15 Hole, P16 Hole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

Commit message: Start modifying "usbcdc"
Parts:
- C1, C11, C12, C13, C14, C15, C5, C6: symbol C -> stm32-rescue:C
- C2: symbol CP -> stm32-rescue:CP
- D1: symbol SP0502BAHT -> stm32-rescue:SP0502BAHT
- D2, D5, D6: symbol LED-RESCUE-stm32 -> stm32-rescue:LED-RESCUE-stm32
- D3: symbol PESD1CAN -> stm32-rescue:PESD1CAN
- D4: symbol D_Schottky -> stm32-rescue:D_Schottky
- D7: symbol USB6B1 -> stm32-rescue:USB6B1
- D8, D9: symbol D_Zener -> stm32-rescue:D_Zener
- J1: symbol CONN_02X03 -> stm32-rescue:CONN_02X03
- J2: symbol DB9_Female -> stm32-rescue:DB9_Female
- J3: symbol DB9_Male -> stm32-rescue:DB9_Male
- J4: symbol Conn_01x07 -> stm32-rescue:Conn_01x07
- J5: symbol Conn_01x02 -> stm32-rescue:Conn_01x02
- J6: symbol Conn_01x01 -> stm32-rescue:Conn_01x01
- JP1: symbol Jumper_NO_Small -> stm32-rescue:Jumper_NO_Small
- P12: symbol CONN_01X03 -> stm32-rescue:CONN_01X03
- P13: symbol USB_A-RESCUE-stm32 -> stm32-rescue:USB_A-RESCUE-stm32
- P15, P16, P17, P18: symbol CONN_01X01 -> stm32-rescue:CONN_01X01
- Q1: symbol Q_PMOS_GSD -> stm32-rescue:Q_PMOS_GSD
- Q2, Q3, Q4: symbol Q_NMOS_GSD -> stm32-rescue:Q_NMOS_GSD
- R1, R10, R11, R12, R13, R14, R2, R27, R28, R29, R3, R30, R34, R35, R4, R5, R6, R7, R8, R9: symbol R -> stm32-rescue:R
- SW1, SW2: symbol SW_Push -> stm32-rescue:SW_Push
- U1, U2: symbol LM1117-3.3-RESCUE-stm32 -> stm32-rescue:LM1117-3.3-RESCUE-stm32
- U4: symbol MCP2551-I/SN -> stm32-rescue:MCP2551-I_SN
- U7: symbol STM32F042C6Tx -> stm32-rescue:STM32F042C6Tx
Connections:
- wire segments 155 -> 197
