File: F3:F303/Multistepper/kicad/multistepper/ADC.kicad_sch (KiCad schematic)
At the start: 6 parts, among them J4 ADC

Commit message: multistp
Parts:
- removed J4: ADC, Connector_IDC:IDC-Header_2x05_P2.54mm_Vertical, symbol Connector_Generic:Conn_02x05_Odd_Even
- added J4: ADC2, Connector_JST:JST_PH_B4B-PH-K_1x04_P2.00mm_Vertical, symbol Connector:Conn_01x04_Female
- added J5: ADC1, Connector_JST:JST_PH_B4B-PH-K_1x04_P2.00mm_Vertical, symbol Connector:Conn_01x04_Female
Connections:
- net +3V3: now also R9.1; no longer R9.2
- net ADC0: now also J4.2 (Pin_2); no longer R10.1, R11.2
- net ADC1: now also J4.3 (Pin_3); no longer R12.1, R13.2
- net ADC2: now also J5.2 (Pin_2)
- net ADC3: now also J5.3 (Pin_3)
- net ADC4: now also R10.1, R11.2
- net ADC5: now also R12.1, R13.2
- net GND: now also J4.4 (Pin_4), J5.4 (Pin_4)
- new net: J4.1 (Pin_1), J5.1 (Pin_1), R9.2
Other:
- moved on the sheet: R9
Changed lines of the file:
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@@
 (kicad_sch (version 20211123) (generator eeschema)
   (paper "A4")
-  (junction (at 69.85 44.196) (diameter 0) (color 0 0 0 0)
-  )
-  (junction (at 69.85 49.276) (diameter 0) (color 0 0 0 0)
-  )
-  (junction (at 69.85 46.736) (diameter 0) (color 0 0 0 0)
-  )
-  (junction (at 69.85 41.656) (diameter 0) (color 0 0 0 0)
-  )
-  (wire (pts (xy 69.85 44.196) (xy 69.85 46.736))
-    (stroke (width 0) (type default) (color 0 0 0 0))
-  )
-  (wire (pts (xy 69.85 46.736) (xy 69.85 49.276))
-    (stroke (width 0) (type default) (color 0 0 0 0))
-  )
-  (wire (pts (xy 69.85 39.116) (xy 69.85 41.656))
-    (stroke (width 0) (type default) (color 0 0 0 0))
-  )
-  (wire (pts (xy 69.85 41.656) (xy 69.85 44.196))
+  (junction (at 64.008 56.134) (diameter 0) (color 0 0 0 0)
+  )
+  (wire (pts (xy 49.022 56.134) (xy 64.008 56.134))
     (stroke (width 0) (type default) (color 0 0 0 0))
   )
@@
     (effects (font (size 1.27 1.27)) (justify left bottom))
   )
-  (global_label "ADC1" (shape input) (at 133.985 39.751 0) (fields_autoplaced)
-    (effects (font (size 1.27 1.27)) (justify left))
-    (property "Intersheet References" "${INTERSHEET_REFS}" (id 0) (at 141.2362 39.6716 0)
-      (effects (font (size 1.27 1.27)) (justify left) hide)
-    )
-  )
-  (global_label "ADC3" (shape input) (at 82.55 44.196 0) (fields_autoplaced)
-    (effects (font (size 1.27 1.27)) (justify left))
-    (property "Intersheet References" "${INTERSHEET_REFS}" (id 0) (at 89.8012 44.1166 0)
-      (effects (font (size 1.27 1.27)) (justify left) hide)
-    )
-  )
-  (global_label "ADC2" (shape input) (at 82.55 41.656 0) (fields_autoplaced)
-    (effects (font (size 1.27 1.27)) (justify left))
-    (property "Intersheet References" "${INTERSHEET_REFS}" (id 0) (at 89.8012 41.5766 0)
-      (effects (font (size 1.27 1.27)) (justify left) hide)
-    )
-  )
-  (global_label "ADC4" (shape input) (at 82.55 46.736 0) (fields_autoplaced)
-    (effects (font (size 1.27 1.27)) (justify left))
-    (property "Intersheet References" "${INTERSHEET_REFS}" (id 0) (at 89.8012 46.6566 0)
-      (effects (font (size 1.27 1.27)) (justify left) hide)
-    )
-  )
-  (global_label "ADC5" (shape input) (at 82.55 49.276 0) (fields_autoplaced)
-    (effects (font (size 1.27 1.27)) (justify left))
-    (property "Intersheet References" "${INTERSHEET_REFS}" (id 0) (at 89.8012 49.3554 0)
-      (effects (font (size 1.27 1.27)) (justify left) hide)
-    )
-  )
-  (global_label "ADC0" (shape input) (at 114.427 33.02 0) (fields_autoplaced)
+  (global_label "ADC1" (shape input) (at 49.022 61.214 0) (fields_autoplaced)
+    (effects (font (size 1.27 1.27)) (justify left))
+    (property "Intersheet References" "${INTERSHEET_REFS}" (id 0) (at 56.2732 61.1346 0)
+      (effects (font (size 1.27 1.27)) (justify left) hide)
+    )
+  )
+  (global_label "ADC3" (shape input) (at 64.008 61.214 180) (fields_autoplaced)
+    (effects (font (size 1.27 1.27)) (justify right))
+    (property "Intersheet References" "${INTERSHEET_REFS}" (id 0) (at 56.7568 61.2934 0)
+      (effects (font (size 1.27 1.27)) (justify right) hide)
+    )
+  )
+  (global_label "ADC2" (shape input) (at 64.008 58.674 180) (fields_autoplaced)
+    (effects (font (size 1.27 1.27)) (justify right))
+    (property "Intersheet References" "${INTERSHEET_REFS}" (id 0) (at 56.7568 58.7534 0)
+      (effects (font (size 1.27 1.27)) (justify right) hide)
+    )
+  )
+  (global_label "ADC4" (shape input) (at 114.427 33.02 0) (fields_autoplaced)
     (effects (font (size 1.27 1.27)) (justify left))
     (property "Intersheet References" "${INTERSHEET_REFS}" (id 0) (at 121.6782 32.9406 0)
+      (effects (font (size 1.27 1.27)) (justify left) hide)
+    )
+  )
+  (global_label "ADC5" (shape input) (at 133.985 39.751 0) (fields_autoplaced)
+    (effects (font (size 1.27 1.27)) (justify left))
+    (property "Intersheet References" "${INTERSHEET_REFS}" (id 0) (at 141.2362 39.8304 0)
+      (effects (font (size 1.27 1.27)) (justify left) hide)
+    )
+  )
+  (global_label "ADC0" (shape input) (at 49.022 58.674 0) (fields_autoplaced)
+    (effects (font (size 1.27 1.27)) (justify left))
+    (property "Intersheet References" "${INTERSHEET_REFS}" (id 0) (at 56.2732 58.5946 0)
       (effects (font (size 1.27 1.27)) (justify left) hide)
     )
@@
     (pin "1")
   )
-  (symbol (lib_id "Device:R") (at 86.36 39.116 90) (unit 1)
-    (in_bom yes) (on_board yes)
-    (property "Reference" "R9" (id 0) (at 86.36 37.084 90))
-    (property "Value" "22" (id 1) (at 86.36 39.116 90))
-    (property "Footprint" "Resistor_SMD:R_0603_1608Metric_Pad0.98x0.95mm_HandSolder" (id 2) (at 86.36 40.894 90)
-      (effects (font (size 1.27 1.27)) hide)
-    )
-    (property "Datasheet" "~" (id 3) (at 86.36 39.116 0)
+  (symbol (lib_id "Device:R") (at 64.008 52.324 0) (unit 1)
+    (in_bom yes) (on_board yes)
+    (property "Reference" "R9" (id 0) (at 66.548 52.07 0))
+    (property "Value" "22" (id 1) (at 64.008 52.324 90))
+    (property "Footprint" "Resistor_SMD:R_0603_1608Metric_Pad0.98x0.95mm_HandSolder" (id 2) (at 62.23 52.324 90)
+      (effects (font (size 1.27 1.27)) hide)
+    )
+    (property "Datasheet" "~" (id 3) (at 64.008 52.324 0)
       (effects (font (size 1.27 1.27)) hide)
     )
@@
     (pin "2")
   )
+  (symbol (lib_id "stm32-rescue:GND") (at 49.022 63.754 0) (unit 1)
+    (in_bom yes) (on_board yes)
+    (property "Reference" "#PWR013" (id 0) (at 49.022 70.104 0)
+      (effects (font (size 1.27 1.27)) hide)
+    )
+    (property "Value" "GND" (id 1) (at 49.022 67.564 0))
+    (property "Footprint" "" (id 2) (at 49.022 63.754 0))
+    (property "Datasheet" "" (id 3) (at 49.022 63.754 0))
+    (pin "1")
+  )
   (symbol (lib_id "Device:R") (at 114.427 36.83 180) (unit 1)
     (in_bom yes) (on_board yes)
@@
     (pin "2")
   )
-  (symbol (lib_id "stm32-rescue:GND") (at 69.85 49.276 0) (unit 1)
-    (in_bom yes) (on_board yes)
-    (property "Reference" "#PWR0118" (id 0) (at 69.85 55.626 0)
-      (effects (font (size 1.27 1.27)) hide)
-    )
-    (property "Value" "GND" (id 1) (at 69.85 53.086 0))
-    (property "Footprint" "" (id 2) (at 69.85 49.276 0))
-    (property "Datasheet" "" (id 3) (at 69.85 49.276 0))
-    (pin "1")
-  )
   (symbol (lib_id "Device:R") (at 133.985 43.561 180) (unit 1)
     (in_bom yes) (on_board yes)
@@
     (pin "2")
   )
+  (symbol (lib_id "Connector:Conn_01x04_Female") (at 69.088 58.674 0) (unit 1)
+    (in_bom yes) (on_board yes) (fields_autoplaced)
+    (property "Reference" "J5" (id 0) (at 69.7992 59.1093 0)
+      (effects (font (size 1.27 1.27)) (justify left))
+    )
+    (property "Value" "ADC1" (id 1) (at 69.7992 61.6462 0)
+      (effects (font (size 1.27 1.27)) (justify left))
+    )
+    (property "Footprint" "Connector_JST:JST_PH_B4B-PH-K_1x04_P2.00mm_Vertical" (id 2) (at 69.088 58.674 0)
+      (effects (font (size 1.27 1.27)) hide)
+    )
+    (property "Datasheet" "~" (id 3) (at 69.088 58.674 0)
+      (effects (font (size 1.27 1.27)) hide)
+    )
+    (pin "1")
+    (pin "2")
+    (pin "3")
+    (pin "4")
+  )
+  (symbol (lib_id "Connector:Conn_01x04_Female") (at 43.942 58.674 0) (mirror y) (unit 1)
+    (in_bom yes) (on_board yes) (fields_autoplaced)
+    (property "Reference" "J4" (id 0) (at 44.577 51.977 0))
+    (property "Value" "ADC2" (id 1) (at 44.577 54.5139 0))
+    (property "Footprint" "Connector_JST:JST_PH_B4B-PH-K_1x04_P2.00mm_Vertical" (id 2) (at 43.942 58.674 0)
+      (effects (font (size 1.27 1.27)) hide)
+    )
+    (property "Datasheet" "~" (id 3) (at 43.942 58.674 0)
+      (effects (font (size 1.27 1.27)) hide)
+    )
+    (pin "1")
+    (pin "2")
+    (pin "3")
+    (pin "4")
+  )
+  (symbol (lib_id "stm32-rescue:GND") (at 64.008 63.754 0) (unit 1)
+    (in_bom yes) (on_board yes)
+    (property "Reference" "#PWR014" (id 0) (at 64.008 70.104 0)
+      (effects (font (size 1.27 1.27)) hide)
+    )
+    (property "Value" "GND" (id 1) (at 64.008 67.564 0))
+    (property "Footprint" "" (id 2) (at 64.008 63.754 0))
+    (property "Datasheet" "" (id 3) (at 64.008 63.754 0))
+    (pin "1")
+  )
   (symbol (lib_id "Device:R") (at 133.985 35.941 180) (unit 1)
     (in_bom yes) (on_board yes)
@@
     (pin "1")
   )
-  (symbol (lib_id "power:+3V3") (at 90.17 39.116 0) (unit 1)
-    (in_bom yes) (on_board yes) (fields_autoplaced)
-    (property "Reference" "#PWR0119" (id 0) (at 90.17 42.926 0)
-      (effects (font (size 1.27 1.27)) hide)
-    )
-    (property "Value" "+3V3" (id 1) (at 90.17 35.5402 0))
-    (property "Footprint" "" (id 2) (at 90.17 39.116 0)
-      (effects (font (size 1.27 1.27)) hide)
-    )
-    (property "Datasheet" "" (id 3) (at 90.17 39.116 0)
+  (symbol (lib_id "power:+3V3") (at 64.008 48.514 0) (unit 1)
+    (in_bom yes) (on_board yes) (fields_autoplaced)
+    (property "Reference" "#PWR0119" (id 0) (at 64.008 52.324 0)
+      (effects (font (size 1.27 1.27)) hide)
+    )
+    (property "Value" "+3V3" (id 1) (at 64.008 44.9382 0))
+    (property "Footprint" "" (id 2) (at 64.008 48.514 0)
+      (effects (font (size 1.27 1.27)) hide)
+    )
+    (property "Datasheet" "" (id 3) (at 64.008 48.514 0)
       (effects (font (size 1.27 1.27)) hide)
     )
@@
     (pin "1")
   )
-  (symbol (lib_id "Connector_Generic:Conn_02x05_Odd_Even") (at 74.93 44.196 0) (unit 1)
-    (in_bom yes) (on_board yes)
-    (property "Reference" "J4" (id 0) (at 76.2 36.576 0))
-    (property "Value" "ADC" (id 1) (at 74.93 51.816 0))
-    (property "Footprint" "Connector_IDC:IDC-Header_2x05_P2.54mm_Vertical" (id 2) (at 74.93 44.196 0)
-      (effects (font (size 1.27 1.27)) hide)
-    )
-    (property "Datasheet" "~" (id 3) (at 74.93 44.196 0)
-      (effects (font (size 1.27 1.27)) hide)
-    )
-    (pin "1")
-    (pin "10")
-    (pin "2")
-    (pin "3")
-    (pin "4")
-    (pin "5")
-    (pin "6")
-    (pin "7")
-    (pin "8")
-    (pin "9")
-  )
 )
