File: F3:F303/Multistepper/kicad/multistepper/mcubase.kicad_sch (KiCad schematic)
At the start: 53 parts, among them J1 Prog, J2 buttons_I2C, J3 screen, SW1 reset, SW2 boot, U1 STM32F303VDTx, Y1 8MHz

Commit message: multistepper ..
Connections:
- net A0: now also RN5.8 (R1.2); no longer RN5.5 (R4.2)
- net A1: now also RN5.7 (R2.2); no longer RN5.6 (R3.2)
- net A2: now also RN5.6 (R3.2); no longer RN5.7 (R2.2)
- net A3: now also RN5.5 (R4.2); no longer RN5.8 (R1.2)
- net ADC0: now also RN5.1 (R1.1); no longer RN5.4 (R4.1)
- net ADC1: now also RN5.2 (R2.1); no longer RN5.3 (R3.1)
- net ADC2: now also RN5.3 (R3.1); no longer RN5.2 (R2.1)
- net ADC3: now also RN5.4 (R4.1); no longer RN5.1 (R1.1)
- net BTN0: now also D1.6 (K); no longer D1.1 (K)
- net BTN1: now also D1.5 (K); no longer D1.3 (K)
- net BTN3_SCL: now also D1.1 (K); no longer D1.6 (K)
- net BTN6: now also D3.4 (K); no longer D3.1 (K)
- net M2_L0: now also D3.3 (K); no longer D3.6 (K)
- net M2_L1: now also D3.1 (K); no longer D3.5 (K)
- net M3_L0: now also D3.5 (K); no longer D3.4 (K)
- net M3_L1: now also D3.6 (K); no longer D3.3 (K)
- net SWDIO: now also D1.3 (K); no longer D1.5 (K)
Changed lines of the file:
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@@
     (stroke (width 0) (type default) (color 0 0 0 0))
   )
-  (wire (pts (xy 177.038 77.47) (xy 186.182 77.47))
+  (wire (pts (xy 177.038 72.39) (xy 186.182 72.39))
     (stroke (width 0) (type default) (color 0 0 0 0))
   )
@@
     (effects (font (size 1.27 1.27)) (justify right bottom))
   )
-  (label "BTN0" (at 186.182 33.528 180)
+  (label "BTN0" (at 186.182 23.368 180)
     (effects (font (size 1.27 1.27)) (justify right bottom))
   )
@@
     (effects (font (size 1.27 1.27)) (justify right bottom))
   )
-  (label "BTN1" (at 186.182 30.988 180)
+  (label "BTN1" (at 186.182 25.908 180)
     (effects (font (size 1.27 1.27)) (justify right bottom))
   )
@@
     (effects (font (size 1.27 1.27)) (justify right bottom))
   )
-  (label "BTN3_SCL" (at 186.182 23.368 180)
+  (label "BTN3_SCL" (at 186.182 33.528 180)
     (effects (font (size 1.27 1.27)) (justify right bottom))
   )
@@
     (effects (font (size 1.27 1.27)) (justify left bottom))
   )
-  (label "SWDIO" (at 186.182 25.908 180)
+  (label "SWDIO" (at 186.182 30.988 180)
     (effects (font (size 1.27 1.27)) (justify right bottom))
   )
@@
     (effects (font (size 1.27 1.27)) (justify right bottom))
   )
-  (label "BTN6" (at 177.038 77.47 180)
+  (label "BTN6" (at 177.038 72.39 180)
     (effects (font (size 1.27 1.27)) (justify right bottom))
   )
@@
     )
   )
-  (global_label "M2_L1" (shape input) (at 186.182 69.85 180) (fields_autoplaced)
-    (effects (font (size 1.27 1.27)) (justify right))
-    (property "Intersheet References" "${INTERSHEET_REFS}" (id 0) (at 177.9027 69.9294 0)
+  (global_label "M2_L1" (shape input) (at 186.182 77.47 180) (fields_autoplaced)
+    (effects (font (size 1.27 1.27)) (justify right))
+    (property "Intersheet References" "${INTERSHEET_REFS}" (id 0) (at 177.9027 77.5494 0)
       (effects (font (size 1.27 1.27)) (justify right) hide)
     )
@@
     )
   )
-  (global_label "M3_L0" (shape input) (at 186.182 72.39 180) (fields_autoplaced)
-    (effects (font (size 1.27 1.27)) (justify right))
-    (property "Intersheet References" "${INTERSHEET_REFS}" (id 0) (at 177.9027 72.3106 0)
+  (global_label "M3_L0" (shape input) (at 186.182 69.85 180) (fields_autoplaced)
+    (effects (font (size 1.27 1.27)) (justify right))
+    (property "Intersheet References" "${INTERSHEET_REFS}" (id 0) (at 177.9027 69.7706 0)
       (effects (font (size 1.27 1.27)) (justify right) hide)
     )
@@
     )
   )
-  (global_label "M3_L1" (shape input) (at 186.182 74.93 180) (fields_autoplaced)
-    (effects (font (size 1.27 1.27)) (justify right))
-    (property "Intersheet References" "${INTERSHEET_REFS}" (id 0) (at 177.9027 74.8506 0)
+  (global_label "M3_L1" (shape input) (at 186.182 67.31 180) (fields_autoplaced)
+    (effects (font (size 1.27 1.27)) (justify right))
+    (property "Intersheet References" "${INTERSHEET_REFS}" (id 0) (at 177.9027 67.2306 0)
       (effects (font (size 1.27 1.27)) (justify right) hide)
     )
@@
     )
   )
-  (global_label "M2_L0" (shape input) (at 186.182 67.31 180) (fields_autoplaced)
-    (effects (font (size 1.27 1.27)) (justify right))
-    (property "Intersheet References" "${INTERSHEET_REFS}" (id 0) (at 177.9027 67.3894 0)
+  (global_label "M2_L0" (shape input) (at 186.182 74.93 180) (fields_autoplaced)
+    (effects (font (size 1.27 1.27)) (justify right))
+    (property "Intersheet References" "${INTERSHEET_REFS}" (id 0) (at 177.9027 75.0094 0)
       (effects (font (size 1.27 1.27)) (justify right) hide)
     )
@@
     (pin "1")
   )
-  (symbol (lib_id "Device:R_Pack04") (at 139.573 40.64 90) (unit 1)
+  (symbol (lib_id "Device:R_Pack04") (at 139.573 43.18 90) (mirror x) (unit 1)
     (in_bom yes) (on_board yes)
-    (property "Reference" "RN5" (id 0) (at 139.7 35.56 90))
-    (property "Value" "330" (id 1) (at 139.573 33.655 90))
-    (property "Footprint" "Resistor_SMD:R_Array_Convex_4x0603" (id 2) (at 139.573 33.655 90)
-      (effects (font (size 1.27 1.27)) hide)
-    )
-    (property "Datasheet" "~" (id 3) (at 139.573 40.64 0)
-      (effects (font (size 1.27 1.27)) hide)
-    )
+    (property "Reference" "RN5" (id 0) (at 139.446 33.909 90))
+    (property "Value" "330" (id 1) (at 139.446 35.814 90))
+    (property "Footprint" "Resistor_SMD:R_Array_Convex_4x0603" (id 2) (at 139.573 50.165 90)
+      (effects (font (size 1.27 1.27)) hide)
+    )
+    (property "Datasheet" "~" (id 3) (at 139.573 43.18 0)
+      (effects (font (size 1.27 1.27)) hide)
+    )

Commit message: multistp
Parts:
- removed D22, D24: SS14, Diode_SMD:D_SOD-323_HandSoldering, symbol Device:D_Schottky
- added J6: MOT_MUL, Connector_JST:JST_PH_B5B-PH-K_1x05_P2.00mm_Vertical, symbol Connector:Conn_01x05_Male
- added J7: ADC2, Connector_JST:JST_PH_B4B-PH-K_1x04_P2.00mm_Vertical, symbol Connector:Conn_01x04_Female
- added R14, R15: 330, Resistor_SMD:R_0603_1608Metric_Pad0.98x0.95mm_HandSolder, symbol Device:R
- added RN6: 330, Resistor_SMD:R_Array_Convex_4x0603, symbol Device:R_Pack04
- R4: value 22 -> 7.5
- R5: value 22 -> 5.1
- Y1: value 8MHz -> NX5032GA-8MHz; footprint Crystal:Crystal_HC49-U_Vertical -> Crystal:Crystal_SMD_5032-2Pin_5.0x3.2mm
Connections:
- net +3V3: no longer D16.1 (K)
- net +5V: now also R5.1; no longer R5.2
- net A0: now also D16.1 (K); no longer D17.1 (K)
- net A1: now also D17.1 (K); no longer D18.1 (K)
- net A2: now also D18.1 (K); no longer D19.1 (K)
- net A3: now also D19.1 (K); no longer D20.1 (K)
- net A4: now also D20.1 (K); no longer D21.1 (K)
- net A5: now also D21.1 (K)
- net BTN0: now also D1.4 (K), RN3.1 (R1.1); no longer D1.6 (K), RN1.5 (R4.2)
- net BTN1: now also RN3.2 (R2.1); no longer RN3.4 (R4.1)
- net BTN2_SDA: now also D1.6 (K), RN3.3 (R3.1); no longer D1.4 (K), RN1.6 (R3.2)
- net BTN3_SCL: now also RN3.4 (R4.1); no longer RN3.3 (R3.1)
- net BTN4: now also RN1.6 (R3.2); no longer RN1.7 (R2.2)
- net BTN5: now also RN1.7 (R2.2); no longer RN3.2 (R2.1)
- net GND: now also D16.2 (A), J2.9 (Pin_9), J3.10 (Pin_10), J3.2 (Pin_2), J6.1 (Pin_1), J7.1 (Pin_1); no longer J2.10 (Pin_10), J3.1 (Pin_1), J3.9 (Pin_9)
- net M0_L0: now also D5.4 (K); no longer D5.5 (K)
- net M0_L1: now also D5.3 (K); no longer D5.6 (K)
- net M5_L0: now also D8.1 (K); no longer D8.6 (K)
- net M5_L1: now also D8.3 (K); no longer D8.5 (K)
- net M6_L0: now also D8.6 (K); no longer D8.4 (K)
- net M6_L1: now also D8.5 (K); no longer D8.3 (K)
- net M7_L0: now also D6.4 (K); no longer D6.1 (K)
- net M7_L1: now also D6.5 (K); no longer D6.3 (K)
- net MOT_MUL0: now also D4.6 (K), RN6.8 (R1.2); no longer D4.4 (K)
- net MOT_MUL1: now also RN6.7 (R2.2)
- net MOT_MUL2: now also D4.4 (K), RN6.6 (R3.2); no longer D4.6 (K)
- net MOT_MUL_EN: now also RN6.5 (R4.2)
- net OUT0: now also D6.3 (K), RN2.8 (R1.2); no longer D6.6 (K)
- net OUT1: now also D6.1 (K), RN2.7 (R2.2); no longer D6.5 (K)
- net OUT2: now also D6.6 (K), RN2.6 (R3.2); no longer D6.4 (K)
- net SCRN_CS: now also D8.4 (K), RN4.4 (R4.1); no longer D8.1 (K), RN4.3 (R3.1)
- net SCRN_DCRS: now also D7.4 (K), RN4.1 (R1.1); no longer D7.1 (K), RN4.2 (R2.1)
- net SCRN_MISO: now also D7.6 (K), R15.1; no longer D7.4 (K), RN2.6 (R3.2)
- net SCRN_MOSI: now also D7.3 (K), RN4.2 (R2.1); no longer D7.5 (K), RN2.7 (R2.2)
- net SCRN_RST: now also D7.1 (K), RN4.3 (R3.1); no longer D7.6 (K), RN4.4 (R4.1)
- net SCRN_SCK: now also D7.5 (K), R14.1; no longer D7.3 (K), RN2.5 (R4.2)
- net USART1_RX: now also D5.6 (K); no longer D5.4 (K)
- net USART1_TX: now also D5.5 (K); no longer D5.3 (K)
- net at RN2.1 (R1.1): now also J7.4 (Pin_4)
- net at RN2.2 (R2.1): now also J7.3 (Pin_3); no longer J3.7 (Pin_7)
- net at RN2.3 (R3.1): now also J7.2 (Pin_2); no longer J3.5 (Pin_5)
- net at J3.3 (Pin_3): now also RN4.5 (R4.2); no longer RN2.4 (R4.1)
- net at R4.1: now also J3.1 (Pin_1); no longer J3.2 (Pin_2)
- net at J3.4 (Pin_4): now also R5.2; no longer RN4.5 (R4.2)
- net at RN4.6 (R3.2): now also J3.5 (Pin_5); no longer J3.6 (Pin_6)
- net at J3.8 (Pin_8): now also R14.2; no longer RN4.7 (R2.2)
- net at RN3.5 (R4.2): now also J2.10 (Pin_10); no longer J2.4 (Pin_4)
- net at RN3.6 (R3.2): now also J2.8 (Pin_8); no longer J2.6 (Pin_6)
- net at RN3.7 (R2.2): now also J2.6 (Pin_6); no longer J2.8 (Pin_8)
- net at RN3.8 (R1.2): now also J2.4 (Pin_4)
- net at J2.3 (Pin_3): now also RN1.1 (R1.1); no longer RN1.4 (R4.1)
- net at J2.5 (Pin_5): now also RN1.2 (R2.1); no longer RN1.3 (R3.1)
- net at J2.7 (Pin_7): now also RN1.3 (R3.1); no longer RN1.2 (R2.1)
- net at RN4.8 (R1.2): now also J3.9 (Pin_9)
- new net: J6.5 (Pin_5), RN6.1 (R1.1)
- new net: J6.4 (Pin_4), RN6.2 (R2.1)
- new net: J6.3 (Pin_3), RN6.3 (R3.1)
- new net: J6.2 (Pin_2), RN6.4 (R4.1)
- new net: J3.6 (Pin_6), R15.2
- new net: J3.7 (Pin_7), RN4.7 (R2.2)
- no-connect marks 6 -> 4
Other:
- moved on the sheet: D15, D23, D6, R5, RN1, RN4
