File: F3:F303/Multistepper/kicad/multistepper/multistepper.kicad_sch (KiCad schematic)
At the start: 0 parts

Commit message: multistp
Parts:
- added C10, C11: 1, Capacitor_SMD:C_0805_2012Metric_Pad1.15x1.40mm_HandSolder, symbol stm32-rescue:C
- added D22: MBRS130L, Diode_SMD:D_SMB_Handsoldering, symbol Device:D_Schottky
- added D24: PESD1CAN, Package_TO_SOT_SMD:SOT-23, symbol elements:PESD1CAN
- added J8: USB_B, Connector_USB:USB_B_OST_USB-B1HSxx_Horizontal, symbol Connector:USB_B
- added J9: Screw_Terminal_01x03, TerminalBlock_Phoenix:TerminalBlock_Phoenix_MKDS-1,5-3_1x03_P5.00mm_Horizontal, symbol Connector:Screw_Terminal_01x03
- added Q1: B0505S, my_footprints:B0x0xS, symbol elements:B0505S
- added R16, R17: 22, Resistor_SMD:R_0603_1608Metric_Pad1.05x0.95mm_HandSolder, symbol stm32-rescue:R
- added R18: 120, Resistor_SMD:R_1210_3225Metric_Pad1.42x2.65mm_HandSolder, symbol stm32-rescue:R
- added SW3: SW_DIP_x01, Button_Switch_THT:SW_DIP_SPSTx01_Slide_6.7x4.1mm_W7.62mm_P2.54mm_LowProfile, symbol Switch:SW_DIP_x01
- added TP1: 5V, TestPoint:TestPoint_THTPad_1.5x1.5mm_Drill0.7mm, symbol Connector:TestPoint
- added U2: ISO1050DUB, Package_SO:SOP-8_6.62x9.15mm_P2.54mm, symbol Interface_CAN_LIN:ISO1050DUB
- added U3: USBLC6-2SC6, Package_TO_SOT_SMD:SOT-23-6, symbol Power_Protection:USBLC6-2SC6
Connections:
- new net: J8.2 (D-), R16.1
- new net: J8.3 (D+), R17.1
- new net: R18.1, SW3.1
- new net: C11.1, Q1.4 (+Vo), U2.8 (VCC2)
- new net: R17.2, U3.1 (I/O1)
- new net: R16.2, U3.3 (I/O2)
- new net +5V: C10.1, D22.1 (K), Q1.2 (Vin), TP1.1, U2.1 (VCC1)
- new net CANH: D24.2 (K), J9.3 (Pin_3), R18.2, U2.7 (CANH)
- new net CANL: D24.1 (K), J9.1 (Pin_1), SW3.2, U2.6 (CANL)
- new net CAN_Rx: U2.2 (RXD)
- new net CAN_Tx: U2.3 (TXD)
- new net Earth: C11.2, D24.3 (O), J9.2 (Pin_2), Q1.3 (0V), U2.5 (GND2)
- new net GND: C10.2, J8.4 (GND), J8.5 (Shield), Q1.1 (GND), U2.4 (GND1), U3.2 (GND)
- new net USB_DM: U3.4 (I/O2)
- new net USB_DP: U3.6 (I/O1)
- new net VB: D22.2 (A), J8.1 (VBUS), U3.5 (VBUS)
Other:
- added sheet Motors (motors.kicad_sch)
- added sheet Power (power.kicad_sch)
- note added: "CAN"
- note added: "CAN connectors"
- note added: "Terminal on/off"
- note added: "USB"
