File: F0:F030,F042,F072/CANbus4BTA/kicad/stm32.kicad_pcb (KiCad board)
At the start: 2 copper layers, 121.5 x 136.5 mm, 155 parts, among them J1 0, J10 RelayB, J15 PB10, J16 PB11, J17 PA15, J18 SSI/422, J19 I2C, J2 1, J20 SPI, J21 Ain, J22 PWMout, J23 Vin, J24 Power, J25 RelayA, J26 Vout, J27 5Vout, J28 CAN, J29 USB_B, J3 4, J30 EXT_IN, J38 PA8, J4 5, J5 6, J6 7, J7 2, J8 3, J9 PROG, K1 HF115F-024-2ZS4, P1 Hole, P2 Hole, P3 Hole, P4 Hole, P5 Hole, P6 Hole, Q1 B0505S-1W, Q2 VRB2405YMD, Q3 B0505S-2W, Q4 SI2300, Q5 SI2300, Q6 SI2308, Q7 IRF9310, Q8 B0505S-1W, SW1 SW_Push, SW2 SW_DIP_x04, SW3 SW_Push, SW4 SW_DIP_x01, U1 74HC4051, U10 LM1117-3.3, U11 PC817, U12 PC817, U13 PC817, U14 PC817, U15 PC817, U16 PC817, U17 PC817, U18 PC817, U2 74HC4051, U3 ISO3086, U4 STM32F072C8Tx, U5 ISO7241C, U6 IP4220CZ6, U7 ADUM4160, U8 ISO1050DUB, U9 LM2576-5.0, Y1 8MHz

Commit message: fixed silkscreen bug in CANbus4BTA
Other:
- board text added: "GND 4.6V 5V 3.3V"
Changed lines of the file:
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@@
       (psa4output false)
       (plotreference true)
-      (plotvalue false)
+      (plotvalue true)
       (plotinvisibletext false)
       (sketchpadsonfab false)
@@
     (effects (font (size 2 2) (thickness 0.25)))
   )
+  (gr_text "GND\n4.6V\n5V\n3.3V" (at 75.184 56.6928) (layer "F.SilkS")
+    (effects (font (size 1.2 1.2) (thickness 0.14)))
+  )
   (gr_text "5V" (at 46.0348 141.847 45) (layer "F.SilkS")

Commit message: fixed bug with dc-dc polarity in CANbus4BTA
Connections:
- Q3 pad 1: GND -> +5V
- Q3 pad 2: +5V -> GND
Routing:
- net GND: track 935.8 -> 1027.3 mm, vias 22 -> 30
- net +5V: track 394.7 -> 397.6 mm
Other:
- board text removed: "GND 4.6V 5V 3.3V"
