File: F3:F303/Multistepper/kicad/multistepper.kicad_pcb (KiCad board)
At the start: 4 copper layers, 63 parts, among them J1 Prog, J2 buttons_I2C, J3 screen, J4 ADC2, J5 ADC1, J6 MOT_MUL, J7 ADC2, SW1 reset, SW2 boot, U1 STM32F303VDTx, Y1 NX5032GA-8MHz

Commit message: multistepper: cont
Parts:
- added C10: 1u, Capacitor_SMD:C_0603_1608Metric_Pad1.08x0.95mm_HandSolder, F.Cu at (300.9, 113.2)
- added C11: 1u, Capacitor_SMD:C_0603_1608Metric_Pad1.08x0.95mm_HandSolder, F.Cu at (282.3, 122.3)
- added C12: 47u 6V, Capacitor_Tantalum_SMD:CP_EIA-3216-18_Kemet-A_Pad1.58x1.35mm_HandSolder, F.Cu at (292.1, 145.0)
- added C13: 0.1, Capacitor_SMD:C_0603_1608Metric_Pad1.08x0.95mm_HandSolder, F.Cu at (289.0, 151.4)
- added C14: 100u 16V, Capacitor_THT:CP_Radial_D8.0mm_P3.50mm, F.Cu at (295.5, 132.8)
- added C15: 0.1, Capacitor_SMD:C_0603_1608Metric_Pad1.08x0.95mm_HandSolder, F.Cu at (289.0, 153.9)
- added C16: 47u 6V, Capacitor_Tantalum_SMD:CP_EIA-3216-18_Kemet-A_Pad1.58x1.35mm_HandSolder, F.Cu at (289.9, 148.5)
- added C17: 47u 10V, Capacitor_Tantalum_SMD:CP_EIA-6032-28_Kemet-C_Pad2.25x2.35mm_HandSolder, F.Cu at (293.5, 141.1)
- added C18: 0.1, Capacitor_SMD:C_0603_1608Metric_Pad1.08x0.95mm_HandSolder, F.Cu at (300.1, 142.5)
- added C19: 100u 35V, Capacitor_THT:CP_Radial_D8.0mm_P3.50mm, F.Cu at (345.6, 100.7)
- added D22: MBRS130L, Diode_SMD:D_SMB_Handsoldering, F.Cu at (285.3, 118.3)
- added D24: PESD1CAN, Package_TO_SOT_SMD:SOT-23, F.Cu at (305.5, 104.0)
- added D25: MM3Z7V5, Diode_SMD:D_0805_2012Metric_Pad1.15x1.40mm_HandSolder, F.Cu at (304.4, 136.0)
- added D26: 1N5822, Diode_THT:D_DO-201_P3.81mm_Vertical_AnodeUp, F.Cu at (281.0, 151.3)
- added D27: MBRS130L, Diode_SMD:D_SMB_Handsoldering, F.Cu at (272.4, 150.7)
- added J10: Screw_Terminal_01x02, TerminalBlock_Phoenix:TerminalBlock_Phoenix_MKDS-1,5-2_1x02_P5.00mm_Horizontal, F.Cu at (270.7, 142.3)
- added J11: Conn_01x03_Male, Connector_PinHeader_2.54mm:PinHeader_1x03_P2.54mm_Vertical, F.Cu at (340.0, 110.5)
- added J12: Conn_01x03_Male, Connector_PinHeader_2.54mm:PinHeader_1x03_P2.54mm_Vertical, F.Cu at (344.7, 107.8)
- added J13: Conn_01x04_Male, Connector_PinHeader_2.54mm:PinHeader_1x04_P2.54mm_Vertical, F.Cu at (340.0, 98.2)
- added J8: USB_B, Connector_USB:USB_B_OST_USB-B1HSxx_Horizontal, F.Cu at (270.0, 103.5)
- added J9: Screw_Terminal_01x03, TerminalBlock_Phoenix:TerminalBlock_Phoenix_MKDS-1,5-3_1x03_P5.00mm_Horizontal, F.Cu at (289.6, 102.1)
- added JP1: SolderJumper_2_Bridged, Jumper:SolderJumper-2_P1.3mm_Open_TrianglePad1.0x1.5mm, F.Cu at (291.0, 122.8)
- added JP10: SolderJumper_3_Open, Jumper:SolderJumper-3_P2.0mm_Open_TrianglePad1.0x1.5mm, F.Cu at (332.5, 118.5)
- added JP11: SolderJumper_3_Open, Jumper:SolderJumper-3_P2.0mm_Open_TrianglePad1.0x1.5mm, F.Cu at (362.6, 97.7)
- added JP12: SolderJumper_3_Open, Jumper:SolderJumper-3_P2.0mm_Open_TrianglePad1.0x1.5mm, F.Cu at (355.6, 97.7)
- added JP13: SolderJumper_2_Bridged, Jumper:SolderJumper-2_P1.3mm_Open_TrianglePad1.0x1.5mm, F.Cu at (344.5, 116.9)
- added JP14: SolderJumper_2_Bridged, Jumper:SolderJumper-2_P1.3mm_Open_TrianglePad1.0x1.5mm, F.Cu at (353.3, 107.2)
- added JP15: SolderJumper_2_Bridged, Jumper:SolderJumper-2_P1.3mm_Open_TrianglePad1.0x1.5mm, F.Cu at (349.2, 112.0)
- added JP16: SolderJumper_2_Bridged, Jumper:SolderJumper-2_P1.3mm_Open_TrianglePad1.0x1.5mm, F.Cu at (361.3, 104.0)
- added JP17: SolderJumper_2_Bridged, Jumper:SolderJumper-2_P1.3mm_Open_TrianglePad1.0x1.5mm, F.Cu at (338.2, 119.6)
- added JP2: SolderJumper_2_Bridged, Jumper:SolderJumper-2_P1.3mm_Open_TrianglePad1.0x1.5mm, F.Cu at (286.6, 122.8)
- added JP3: SolderJumper_2_Bridged, Jumper:SolderJumper-2_P1.3mm_Open_TrianglePad1.0x1.5mm, F.Cu at (322.3, 129.8)
- added JP4: SolderJumper_2_Bridged, Jumper:SolderJumper-2_P1.3mm_Open_TrianglePad1.0x1.5mm, F.Cu at (312.6, 129.8)
- added JP5: SolderJumper_2_Bridged, Jumper:SolderJumper-2_P1.3mm_Open_TrianglePad1.0x1.5mm, F.Cu at (295.1, 148.4)
- added JP6: SolderJumper_2_Bridged, Jumper:SolderJumper-2_P1.3mm_Open_TrianglePad1.0x1.5mm, F.Cu at (351.7, 126.3)
- added JP7: SolderJumper_2_Bridged, Jumper:SolderJumper-2_P1.3mm_Open_TrianglePad1.0x1.5mm, F.Cu at (356.0, 128.8)
- added JP8: SolderJumper_3_Open, Jumper:SolderJumper-3_P2.0mm_Open_TrianglePad1.0x1.5mm, F.Cu at (325.5, 118.5)
- added JP9: SolderJumper_3_Open, Jumper:SolderJumper-3_P2.0mm_Open_TrianglePad1.0x1.5mm, F.Cu at (355.6, 101.6)
- added L1: 100u, Inductor_THT:L_Toroid_Horizontal_D6.5mm_P10.00mm_Diameter7-5mm_Amidon-T25, F.Cu at (268.9, 132.1)
- added Q1: B0505S, stepper:B0x0xS, F.Cu at (292.4, 113.7)
- added Q2: IRF9310, Package_SO:SO-8_3.9x4.9mm_P1.27mm, F.Cu at (306.2, 131.3)
- added R16: 22, Resistor_SMD:R_0603_1608Metric_Pad0.98x0.95mm_HandSolder, F.Cu at (310.2, 103.0)
- added R17: 22, Resistor_SMD:R_0603_1608Metric_Pad0.98x0.95mm_HandSolder, F.Cu at (316.1, 97.2)
- added R18: 120, Resistor_SMD:R_1210_3225Metric_Pad1.30x2.65mm_HandSolder, F.Cu at (301.7, 109.9)
- added R19: 4k7, Resistor_SMD:R_0603_1608Metric_Pad0.98x0.95mm_HandSolder, F.Cu at (269.3, 154.8)
- added R20: 4k7, Resistor_SMD:R_0603_1608Metric_Pad0.98x0.95mm_HandSolder, F.Cu at (273.7, 154.8)
- added R21: 100, Resistor_SMD:R_0603_1608Metric_Pad0.98x0.95mm_HandSolder, F.Cu at (351.7, 129.3)
- added R22: 100, Resistor_SMD:R_0603_1608Metric_Pad0.98x0.95mm_HandSolder, F.Cu at (356.0, 125.8)
- added R23: 100, Resistor_SMD:R_0603_1608Metric_Pad0.98x0.95mm_HandSolder, F.Cu at (361.3, 101.0)
- added RN7: 330, Resistor_SMD:R_Array_Convex_4x0603, F.Cu at (343.1, 138.3)
- added RN8: 330, Resistor_SMD:R_Array_Convex_4x0603, F.Cu at (349.1, 107.8)
- added SW3: SW_DIP_x01, Button_Switch_THT:SW_DIP_SPSTx01_Slide_6.7x4.1mm_W7.62mm_P2.54mm_LowProfile, F.Cu at (304.7, 98.8)
- added TP1: 5V, TestPoint:TestPoint_THTPad_1.5x1.5mm_Drill0.7mm, F.Cu at (306.5, 108.0)
- added TP2: 5V, TestPoint:TestPoint_THTPad_1.5x1.5mm_Drill0.7mm, F.Cu at (312.2, 133.4)
- added TP3: Gnd, TestPoint:TestPoint_THTPad_1.5x1.5mm_Drill0.7mm, F.Cu at (293.0, 151.9)
- added TP4: 5V, TestPoint:TestPoint_THTPad_1.5x1.5mm_Drill0.7mm, F.Cu at (299.0, 145.6)
- added TP5: 3.3V, TestPoint:TestPoint_THTPad_1.5x1.5mm_Drill0.7mm, F.Cu at (305.6, 139.3)
- added U2: ISO1050DUB, Package_SO:SOP-8_6.62x9.15mm_P2.54mm, F.Cu at (273.6, 118.8)
- added U3: USBLC6-2SC6, Package_TO_SOT_SMD:SOT-23-6, F.Cu at (293.1, 117.7)
- added U4: LM4050A(b)EX3-3.3, Package_TO_SOT_SMD:SOT-323_SC-70_Handsoldering, F.Cu at (313.2, 141.2)
- added U5: LM2576-5.0, Package_TO_SOT_THT:TO-220-5_P3.4x3.7mm_StaggerEven_Lead3.8mm_Vertical, F.Cu at (283.1, 133.3)
- added U6: LM1117-3.3, Package_TO_SOT_SMD:SOT-223-3_TabPin2, F.Cu at (284.1, 142.8)
- added U7: 74HC4051, Package_SO:SOIC-16_3.9x9.9mm_P1.27mm, F.Cu at (345.3, 130.2)
- added XX1: stepper_module, stepper:stepper_module, F.Cu at (329.8, 106.3)
Connections:
- U1 pad 100: +3V3 -> Net-(JP3-Pad1)
- U1 pad 22: +3V3 -> Net-(JP3-Pad1)
- U1 pad 28: +3V3 -> Net-(JP3-Pad1)
- U1 pad 50: +3V3 -> Net-(JP3-Pad1)
- U1 pad 6: +3V3 -> Net-(JP3-Pad1)
- U1 pad 75: +3V3 -> Net-(JP3-Pad1)

Commit message: multistepper schematic
Parts:
- removed the J11 at (340.0, 110.5)
- removed JP16, JP17: SolderJumper_2_Bridged, Jumper:SolderJumper-2_P1.3mm_Open_TrianglePad1.0x1.5mm
- added J13: UART, Connector_JST:JST_PH_B3B-PH-K_1x03_P2.00mm_Vertical, F.Cu at (117.4, 110.2)
- added R24: 22, Resistor_SMD:R_0603_1608Metric_Pad0.98x0.95mm_HandSolder, B.Cu at (116.5, 108.4)
- added R25: 22, Resistor_SMD:R_0603_1608Metric_Pad0.98x0.95mm_HandSolder, B.Cu at (116.5, 106.9)
- D22, JP10, JP11, JP12, JP13, JP14, JP15, JP2, JP3, JP7, JP8, JP9, R16, R17, R23, U3, U7: moved to B.Cu
- J11: renamed from J12; value Conn_01x03_Male -> LimS; footprint Connector_PinHeader_2.54mm:PinHeader_1x03_P2.54mm_Vertical -> Connector_JST:JST_EH_B4B-EH-A_1x04_P2.50mm_Vertical
- J12: renamed from J13; value Conn_01x04_Male -> Stepper; footprint Connector_PinHeader_2.54mm:PinHeader_1x04_P2.54mm_Vertical -> Connector_JST:JST_EH_B4B-EH-A_1x04_P2.50mm_Vertical
- J2: value buttons_I2C -> Buttons/I2C
- J3: value screen -> Screen
- J7: value ADC2 -> GPO
- SW1: value reset -> Reset
- SW2: value boot -> Boot
- TP1: value 5V -> 5Vusb
- moved R23 276.0 mm to (88.5, 143.3), turned to 180 degrees
- moved R22 273.8 mm to (87.0, 74.9)
- moved JP9 265.0 mm to (93.2, 138.9), turned to -90 degrees
- moved JP11 265.0 mm to (100.8, 138.9), turned to -90 degrees
- moved JP12 260.6 mm to (98.3, 138.9), turned to -90 degrees
- moved JP7 260.6 mm to (101.7, 72.3), turned to -90 degrees
- moved J11 259.2 mm to (87.6, 141.2), turned to 90 degrees
- moved JP14 254.1 mm to (100.6, 133.6), turned to 90 degrees
- moved JP15 252.0 mm to (98.0, 133.6), turned to 90 degrees
- moved RN8 250.8 mm to (99.1, 128.3), turned to 90 degrees
- moved J12 247.0 mm to (98.1, 148.3)
- moved U7 246.3 mm to (104.1, 79.8), turned to 180 degrees
- moved C19 243.4 mm to (105.4, 140.2), turned to 90 degrees
- moved JP13 242.0 mm to (103.1, 133.6), turned to 90 degrees
- moved JP8 230.6 mm to (95.8, 138.9), turned to -90 degrees
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Connections:
- net /Motors/stepper_M/CLK renamed /Motors/stepper_M1/CLK
- net /Motors/stepper_M/MS1 renamed /Motors/stepper_M1/MS1
- net /Motors/stepper_M/MS2 renamed /Motors/stepper_M1/MS2
- net /Motors/stepper_M/SPR renamed /Motors/stepper_M1/SPR
- net USART1_RX renamed /MCU base/USART1_RX
- net USART1_TX renamed /MCU base/USART1_TX
- C19 pad 1: Net-(C19-Pad1) -> /Motors/Vm
- C3 pad 2: +3V3 -> /MCU base/MCU3v3
- C5 pad 1: +3V3 -> /MCU base/MCU3v3
- C6 pad 1: +3V3 -> /MCU base/MCU3v3
- C7 pad 1: +3V3 -> /MCU base/MCU3v3
- C8 pad 1: +3V3 -> /MCU base/MCU3v3
- C9 pad 1: +3V3 -> /MCU base/MCU3v3
- D10 pad 1: +3V3 -> /MCU base/MCU3v3
- D11 pad 1: +3V3 -> /MCU base/MCU3v3
- D12 pad 1: +3V3 -> /MCU base/MCU3v3
- D13 pad 1: +3V3 -> /MCU base/MCU3v3
- D14 pad 1: +3V3 -> /MCU base/MCU3v3
- D15 pad 1: +3V3 -> /MCU base/MCU3v3
- D2 pad 3: M4_L0 -> M3_L0
- D2 pad 4: M4_L1 -> M3_L1
- D3 pad 1: M2_L1 -> M1_L1
- D3 pad 3: M2_L0 -> M1_L0
- D3 pad 5: M3_L0 -> M2_L0
- D3 pad 6: M3_L1 -> M2_L1
- D4 pad 1: M1_L0 -> M0_L0
- D4 pad 3: M1_L1 -> M0_L1
- D5 pad 3: M0_L1 -> M7_L1
- D5 pad 4: M0_L0 -> M7_L0
- D6 pad 4: M7_L0 -> M6_L0
- D6 pad 5: M7_L1 -> M6_L1
- D8 pad 1: M5_L0 -> M4_L0
- D8 pad 3: M5_L1 -> M4_L1
- D8 pad 5: M6_L1 -> M5_L1
- D8 pad 6: M6_L0 -> M5_L0
- D9 pad 1: +3V3 -> /MCU base/MCU3v3
- J11 pad 1: GND -> Net-(J11-Pad1)
- J11 pad 3: Net-(J11-Pad3) -> M0_L1
- JP10 pad 3: /Motors/stepper_M/Vio -> /Motors/Vio
- JP11 pad 3: /Motors/stepper_M/Vio -> /Motors/Vio
- JP12 pad 3: /Motors/stepper_M/Vio -> /Motors/Vio
- JP14 pad 2: /Motors/USART0-3 -> /Motors/stepper_M1/U
- JP3 pad 1: Net-(JP3-Pad1) -> /MCU base/MCU3v3
- JP7 pad 2: Net-(JP7-Pad2) -> /Motors/Vio
- JP8 pad 2: /Motors/USART0-3 -> /Motors/stepper_M1/U
- JP8 pad 3: /Motors/stepper_M/Vio -> /Motors/Vio
- R2 pad 1: +3V3 -> /MCU base/MCU3v3
- R23 pad 1: /Motors/stepper_M/Vio -> /Motors/Vio
- R23 pad 2: Net-(J11-Pad3) -> Net-(J11-Pad1)
- R9 pad 1: +3V3 -> /MCU base/MCU3v3
- RN8 pad 2: M0_DIR -> /Motors/stepper_M1/DIRx
- RN8 pad 3: M0_STEP -> /Motors/stepper_M1/STEPx
- RN8 pad 4: M0_EN -> /Motors/stepper_M1/~{ENx}
- SW2 pad 2: +3V3 -> /MCU base/MCU3v3
- U1 pad 10: M1_STEP -> M0_STEP
- U1 pad 100: Net-(JP3-Pad1) -> /MCU base/MCU3v3
- U1 pad 11: M1_L1 -> M0_L1
- U1 pad 22: Net-(JP3-Pad1) -> /MCU base/MCU3v3
- U1 pad 28: Net-(JP3-Pad1) -> /MCU base/MCU3v3
- U1 pad 35: M0_STEP -> M7_STEP
- U1 pad 36: M0_EN -> M7_EN
- U1 pad 37: M0_DIR -> M7_DIR
- U1 pad 38: M0_L0 -> M7_L0
- U1 pad 39: M0_L1 -> M7_L1
- U1 pad 40: M7_STEP -> M6_STEP
- U1 pad 41: M7_EN -> M6_EN
- U1 pad 42: M7_DIR -> M6_DIR
- U1 pad 43: M7_L0 -> M6_L0
- U1 pad 44: M7_L1 -> M6_L1
- U1 pad 50: Net-(JP3-Pad1) -> /MCU base/MCU3v3
- U1 pad 57: M6_L1 -> M5_L1
- U1 pad 58: M6_L0 -> M5_L0
- U1 pad 59: M6_STEP -> M5_STEP
- U1 pad 6: Net-(JP3-Pad1) -> /MCU base/MCU3v3
- U1 pad 60: M6_DIR -> M5_DIR
- U1 pad 61: M6_EN -> M5_EN
- U1 pad 62: M5_L1 -> M4_L1
- U1 pad 63: M5_STEP -> M4_STEP
- U1 pad 64: M5_L0 -> M4_L0
- U1 pad 65: M5_DIR -> M4_DIR
- U1 pad 66: M5_EN -> M4_EN
- U1 pad 7: M1_EN -> M0_EN
- U1 pad 75: Net-(JP3-Pad1) -> /MCU base/MCU3v3
- U1 pad 77: M4_STEP -> M3_STEP
- U1 pad 78: M4_EN -> M3_EN
- U1 pad 79: M4_DIR -> M3_DIR
- U1 pad 8: M1_DIR -> M0_DIR
- U1 pad 80: M4_L0 -> M3_L0
- U1 pad 83: M4_L1 -> M3_L1
- U1 pad 87: M3_L1 -> M2_L1
- U1 pad 88: M3_L0 -> M2_L0
- U1 pad 9: M1_L0 -> M0_L0
- U1 pad 90: M3_DIR -> M2_DIR
- U1 pad 91: M3_STEP -> M2_STEP
- U1 pad 92: M3_EN -> M2_EN
- U1 pad 93: M2_L1 -> M1_L1
- U1 pad 95: M2_STEP -> M1_STEP
- U1 pad 96: M2_L0 -> M1_L0
- U1 pad 97: M2_DIR -> M1_DIR
- U1 pad 98: M2_EN -> M1_EN
- U7 pad 16: Net-(JP7-Pad2) -> /Motors/Vio
- XX1 pad 1: M0_EN -> /Motors/stepper_M1/~{ENx}
- XX1 pad 10: /Motors/stepper_M/Vio -> /Motors/Vio
- XX1 pad 16: Net-(C19-Pad1) -> /Motors/Vm
- XX1 pad 5: /Motors/USART0-3 -> /Motors/stepper_M1/U
- XX1 pad 7: M0_STEP -> /Motors/stepper_M1/STEPx
- XX1 pad 8: M0_DIR -> /Motors/stepper_M1/DIRx
Routing:
- net +3V3: track 200.3 -> 22.4 mm, vias 9 -> 1
- net /MCU base/MCU3v3: track 0.00 -> 141.3 mm, vias 0 -> 8
- net GND: track 313.9 -> 444.4 mm, vias 13 -> 16
- net /Motors/Vm: track 0.00 -> 32.0 mm
- net /VB: track 0.00 -> 26.9 mm
- net /Motors/Vio: track 0.00 -> 25.2 mm
- net M4_EN: track 5.60 -> 30.2 mm
- net M4_DIR: track 5.49 -> 28.2 mm
- net M0_L1: track 15.9 -> 38.4 mm
- net M4_L0: track 7.54 -> 28.3 mm
- net M4_STEP: track 5.71 -> 26.0 mm
- net Net-(J12-Pad3): track 0.00 -> 18.1 mm
- net Net-(J12-Pad2): track 0.00 -> 18.1 mm
- net Net-(J12-Pad4): track 0.00 -> 17.9 mm
- net Net-(J12-Pad1): track 0.00 -> 17.9 mm
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
Commit message: Multistepper PCB almost ready
Parts:
- added C20: 100u 35V, Capacitor_THT:CP_Radial_D8.0mm_P3.50mm, F.Cu at (65.2, 49.6)
- added C21: 100u 35V, Capacitor_THT:CP_Radial_D8.0mm_P3.50mm, F.Cu at (92.6, 49.6)
- added C22: 100u 35V, Capacitor_THT:CP_Radial_D8.0mm_P3.50mm, F.Cu at (119.7, 49.5)
- added C23: 100u 35V, Capacitor_THT:CP_Radial_D8.0mm_P3.50mm, F.Cu at (135.3, 132.9)
- added C24: 100u 35V, Capacitor_THT:CP_Radial_D8.0mm_P3.50mm, F.Cu at (105.2, 133.0)
- added C25: 100u 35V, Capacitor_THT:CP_Radial_D8.0mm_P3.50mm, F.Cu at (75.4, 133.0)
- added C26: 100u 35V, Capacitor_THT:CP_Radial_D8.0mm_P3.50mm, F.Cu at (66.4, 111.5)
- added H1: MountingHole, MountingHole:MountingHole_3.2mm_M3_DIN965_Pad, F.Cu at (59.0, 42.0)
- added H2: MountingHole, MountingHole:MountingHole_3.2mm_M3_DIN965_Pad, F.Cu at (165.5, 42.0)
- added H3: MountingHole, MountingHole:MountingHole_3.2mm_M3_DIN965_Pad, F.Cu at (59.0, 140.5)
- added H4: MountingHole, MountingHole:MountingHole_3.2mm_M3_DIN965_Pad, F.Cu at (165.5, 140.5)
- added J14: LimS, Connector_JST:JST_EH_B4B-EH-A_1x04_P2.50mm_Vertical, F.Cu at (83.0, 48.7)
- added J15: Stepper, Connector_JST:JST_EH_B4B-EH-A_1x04_P2.50mm_Vertical, F.Cu at (72.5, 41.6)
- added J16: LimS, Connector_JST:JST_EH_B4B-EH-A_1x04_P2.50mm_Vertical, F.Cu at (110.4, 48.6)
- added J17: Stepper, Connector_JST:JST_EH_B4B-EH-A_1x04_P2.50mm_Vertical, F.Cu at (99.9, 41.5)
- added J18: LimS, Connector_JST:JST_EH_B4B-EH-A_1x04_P2.50mm_Vertical, F.Cu at (137.5, 48.6)
- added J19: Stepper, Connector_JST:JST_EH_B4B-EH-A_1x04_P2.50mm_Vertical, F.Cu at (127.0, 41.4)
- added J20: LimS, Connector_JST:JST_EH_B4B-EH-A_1x04_P2.50mm_Vertical, F.Cu at (117.5, 133.9)
- added J21: Stepper, Connector_JST:JST_EH_B4B-EH-A_1x04_P2.50mm_Vertical, F.Cu at (128.0, 141.0)
- added J22: LimS, Connector_JST:JST_EH_B4B-EH-A_1x04_P2.50mm_Vertical, F.Cu at (87.5, 133.9)
- added J23: Stepper, Connector_JST:JST_EH_B4B-EH-A_1x04_P2.50mm_Vertical, F.Cu at (97.9, 141.1)
- added J24: LimS, Connector_JST:JST_EH_B4B-EH-A_1x04_P2.50mm_Vertical, F.Cu at (57.6, 133.9)
- added J25: Stepper, Connector_JST:JST_EH_B4B-EH-A_1x04_P2.50mm_Vertical, F.Cu at (68.1, 141.1)
- added J26: LimS, Connector_JST:JST_EH_B4B-EH-A_1x04_P2.50mm_Vertical, F.Cu at (65.5, 93.7)
- added J27: Stepper, Connector_JST:JST_EH_B4B-EH-A_1x04_P2.50mm_Vertical, F.Cu at (58.3, 104.2)
- added JP16: SolderJumper_3_Open, Jumper:SolderJumper-3_P2.0mm_Open_TrianglePad1.0x1.5mm, B.Cu at (74.8, 50.9)
- added JP17: SolderJumper_3_Open, Jumper:SolderJumper-3_P2.0mm_Open_TrianglePad1.0x1.5mm, B.Cu at (77.4, 50.9)
- added JP18: SolderJumper_3_Open, Jumper:SolderJumper-3_P2.0mm_Open_TrianglePad1.0x1.5mm, B.Cu at (62.9, 54.2)
- added JP19: SolderJumper_3_Open, Jumper:SolderJumper-3_P2.0mm_Open_TrianglePad1.0x1.5mm, B.Cu at (69.8, 50.9)
- added JP20: SolderJumper_3_Open, Jumper:SolderJumper-3_P2.0mm_Open_TrianglePad1.0x1.5mm, B.Cu at (72.3, 50.9)
- added JP21: SolderJumper_2_Bridged, Jumper:SolderJumper-2_P1.3mm_Open_TrianglePad1.0x1.5mm, B.Cu at (67.5, 56.2)
- added JP22: SolderJumper_2_Bridged, Jumper:SolderJumper-2_P1.3mm_Open_TrianglePad1.0x1.5mm, B.Cu at (70.0, 56.2)
- added JP23: SolderJumper_2_Bridged, Jumper:SolderJumper-2_P1.3mm_Open_TrianglePad1.0x1.5mm, B.Cu at (72.6, 56.2)
- added JP24: SolderJumper_3_Open, Jumper:SolderJumper-3_P2.0mm_Open_TrianglePad1.0x1.5mm, B.Cu at (102.3, 50.9)
- added JP25: SolderJumper_3_Open, Jumper:SolderJumper-3_P2.0mm_Open_TrianglePad1.0x1.5mm, B.Cu at (104.8, 50.9)
- added JP26: SolderJumper_3_Open, Jumper:SolderJumper-3_P2.0mm_Open_TrianglePad1.0x1.5mm, B.Cu at (90.3, 54.2)
- added JP27: SolderJumper_3_Open, Jumper:SolderJumper-3_P2.0mm_Open_TrianglePad1.0x1.5mm, B.Cu at (97.2, 50.9)
- added JP28: SolderJumper_3_Open, Jumper:SolderJumper-3_P2.0mm_Open_TrianglePad1.0x1.5mm, B.Cu at (99.7, 50.9)
- added JP29: SolderJumper_2_Bridged, Jumper:SolderJumper-2_P1.3mm_Open_TrianglePad1.0x1.5mm, B.Cu at (94.9, 56.2)
- added JP30: SolderJumper_2_Bridged, Jumper:SolderJumper-2_P1.3mm_Open_TrianglePad1.0x1.5mm, B.Cu at (97.4, 56.2)
- added JP31: SolderJumper_2_Bridged, Jumper:SolderJumper-2_P1.3mm_Open_TrianglePad1.0x1.5mm, B.Cu at (100.0, 56.2)
- added JP32: SolderJumper_3_Open, Jumper:SolderJumper-3_P2.0mm_Open_TrianglePad1.0x1.5mm, B.Cu at (129.4, 50.8)
- added JP33: SolderJumper_3_Open, Jumper:SolderJumper-3_P2.0mm_Open_TrianglePad1.0x1.5mm, B.Cu at (131.9, 50.8)
- added JP34: SolderJumper_3_Open, Jumper:SolderJumper-3_P2.0mm_Open_TrianglePad1.0x1.5mm, B.Cu at (117.4, 54.1)
- added JP35: SolderJumper_3_Open, Jumper:SolderJumper-3_P2.0mm_Open_TrianglePad1.0x1.5mm, B.Cu at (124.3, 50.8)
- added JP36: SolderJumper_3_Open, Jumper:SolderJumper-3_P2.0mm_Open_TrianglePad1.0x1.5mm, B.Cu at (126.8, 50.8)
- added JP37: SolderJumper_2_Bridged, Jumper:SolderJumper-2_P1.3mm_Open_TrianglePad1.0x1.5mm, B.Cu at (122.0, 56.1)
- added JP38: SolderJumper_2_Bridged, Jumper:SolderJumper-2_P1.3mm_Open_TrianglePad1.0x1.5mm, B.Cu at (124.5, 56.1)
- added JP39: SolderJumper_2_Bridged, Jumper:SolderJumper-2_P1.3mm_Open_TrianglePad1.0x1.5mm, B.Cu at (127.1, 56.1)
- added JP40: SolderJumper_3_Open, Jumper:SolderJumper-3_P2.0mm_Open_TrianglePad1.0x1.5mm, B.Cu at (125.7, 131.6)
- added JP41: SolderJumper_3_Open, Jumper:SolderJumper-3_P2.0mm_Open_TrianglePad1.0x1.5mm, B.Cu at (123.1, 131.6)
- added JP42: SolderJumper_3_Open, Jumper:SolderJumper-3_P2.0mm_Open_TrianglePad1.0x1.5mm, B.Cu at (137.6, 128.3)
- added JP43: SolderJumper_3_Open, Jumper:SolderJumper-3_P2.0mm_Open_TrianglePad1.0x1.5mm, B.Cu at (130.7, 131.6)
- added JP44: SolderJumper_3_Open, Jumper:SolderJumper-3_P2.0mm_Open_TrianglePad1.0x1.5mm, B.Cu at (128.2, 131.6)
- added JP45: SolderJumper_2_Bridged, Jumper:SolderJumper-2_P1.3mm_Open_TrianglePad1.0x1.5mm, B.Cu at (133.0, 126.3)
- added JP46: SolderJumper_2_Bridged, Jumper:SolderJumper-2_P1.3mm_Open_TrianglePad1.0x1.5mm, B.Cu at (130.5, 126.3)
- added JP47: SolderJumper_2_Bridged, Jumper:SolderJumper-2_P1.3mm_Open_TrianglePad1.0x1.5mm, B.Cu at (127.9, 126.3)
- added JP48: SolderJumper_3_Open, Jumper:SolderJumper-3_P2.0mm_Open_TrianglePad1.0x1.5mm, B.Cu at (95.6, 131.7)
- added JP49: SolderJumper_3_Open, Jumper:SolderJumper-3_P2.0mm_Open_TrianglePad1.0x1.5mm, B.Cu at (93.1, 131.7)
- added JP50: SolderJumper_3_Open, Jumper:SolderJumper-3_P2.0mm_Open_TrianglePad1.0x1.5mm, B.Cu at (107.5, 128.4)
- added JP51: SolderJumper_3_Open, Jumper:SolderJumper-3_P2.0mm_Open_TrianglePad1.0x1.5mm, B.Cu at (100.7, 131.7)
- added JP52: SolderJumper_3_Open, Jumper:SolderJumper-3_P2.0mm_Open_TrianglePad1.0x1.5mm, B.Cu at (98.1, 131.7)
- added JP53: SolderJumper_2_Bridged, Jumper:SolderJumper-2_P1.3mm_Open_TrianglePad1.0x1.5mm, B.Cu at (103.0, 126.4)
- added JP54: SolderJumper_2_Bridged, Jumper:SolderJumper-2_P1.3mm_Open_TrianglePad1.0x1.5mm, B.Cu at (100.4, 126.4)
- added JP55: SolderJumper_2_Bridged, Jumper:SolderJumper-2_P1.3mm_Open_TrianglePad1.0x1.5mm, B.Cu at (97.9, 126.4)
- added JP56: SolderJumper_3_Open, Jumper:SolderJumper-3_P2.0mm_Open_TrianglePad1.0x1.5mm, B.Cu at (65.7, 131.7)
- added JP57: SolderJumper_3_Open, Jumper:SolderJumper-3_P2.0mm_Open_TrianglePad1.0x1.5mm, B.Cu at (63.2, 131.7)
- added JP58: SolderJumper_3_Open, Jumper:SolderJumper-3_P2.0mm_Open_TrianglePad1.0x1.5mm, B.Cu at (77.7, 128.4)
- added JP59: SolderJumper_3_Open, Jumper:SolderJumper-3_P2.0mm_Open_TrianglePad1.0x1.5mm, B.Cu at (70.8, 131.7)
- added JP60: SolderJumper_3_Open, Jumper:SolderJumper-3_P2.0mm_Open_TrianglePad1.0x1.5mm, B.Cu at (68.3, 131.7)
- added JP61: SolderJumper_2_Bridged, Jumper:SolderJumper-2_P1.3mm_Open_TrianglePad1.0x1.5mm, B.Cu at (73.1, 126.4)
- added JP62: SolderJumper_2_Bridged, Jumper:SolderJumper-2_P1.3mm_Open_TrianglePad1.0x1.5mm, B.Cu at (70.6, 126.4)
- added JP63: SolderJumper_2_Bridged, Jumper:SolderJumper-2_P1.3mm_Open_TrianglePad1.0x1.5mm, B.Cu at (68.0, 126.4)
- added JP64: SolderJumper_3_Open, Jumper:SolderJumper-3_P2.0mm_Open_TrianglePad1.0x1.5mm, B.Cu at (67.7, 101.8)
- added JP65: SolderJumper_3_Open, Jumper:SolderJumper-3_P2.0mm_Open_TrianglePad1.0x1.5mm, B.Cu at (67.7, 99.3)
- added JP66: SolderJumper_3_Open, Jumper:SolderJumper-3_P2.0mm_Open_TrianglePad1.0x1.5mm, B.Cu at (71.0, 113.8)
- added JP67: SolderJumper_3_Open, Jumper:SolderJumper-3_P2.0mm_Open_TrianglePad1.0x1.5mm, B.Cu at (67.7, 106.9)
- added JP68: SolderJumper_3_Open, Jumper:SolderJumper-3_P2.0mm_Open_TrianglePad1.0x1.5mm, B.Cu at (67.7, 104.4)
- added JP69: SolderJumper_2_Bridged, Jumper:SolderJumper-2_P1.3mm_Open_TrianglePad1.0x1.5mm, B.Cu at (73.0, 109.2)
- added JP70: SolderJumper_2_Bridged, Jumper:SolderJumper-2_P1.3mm_Open_TrianglePad1.0x1.5mm, B.Cu at (73.0, 106.6)
- added JP71: SolderJumper_2_Bridged, Jumper:SolderJumper-2_P1.3mm_Open_TrianglePad1.0x1.5mm, B.Cu at (73.0, 104.1)
- added R26: 100, Resistor_SMD:R_0603_1608Metric_Pad0.98x0.95mm_HandSolder, B.Cu at (82.1, 46.5)
- added R27: 100, Resistor_SMD:R_0603_1608Metric_Pad0.98x0.95mm_HandSolder, B.Cu at (109.5, 46.5)
- added R28: 100, Resistor_SMD:R_0603_1608Metric_Pad0.98x0.95mm_HandSolder, B.Cu at (136.6, 46.4)
- added R29: 100, Resistor_SMD:R_0603_1608Metric_Pad0.98x0.95mm_HandSolder, B.Cu at (118.4, 136.0)
- added R30: 100, Resistor_SMD:R_0603_1608Metric_Pad0.98x0.95mm_HandSolder, B.Cu at (88.4, 136.1)
- added R31: 100, Resistor_SMD:R_0603_1608Metric_Pad0.98x0.95mm_HandSolder, B.Cu at (58.5, 136.1)
- added R32: 100, Resistor_SMD:R_0603_1608Metric_Pad0.98x0.95mm_HandSolder, B.Cu at (63.3, 94.6)
- added RN10: 330, Resistor_SMD:R_Array_Convex_4x0603, F.Cu at (99.0, 61.5)
- added RN11: 330, Resistor_SMD:R_Array_Convex_4x0603, F.Cu at (126.1, 61.5)
- added RN12: 330, Resistor_SMD:R_Array_Convex_4x0603, F.Cu at (129.0, 121.0)
- added RN13: 330, Resistor_SMD:R_Array_Convex_4x0603, F.Cu at (98.9, 121.0)
- added RN14: 330, Resistor_SMD:R_Array_Convex_4x0603, F.Cu at (69.0, 121.0)
- added RN15: 330, Resistor_SMD:R_Array_Convex_4x0603, F.Cu at (78.4, 105.1)
- added RN9: 330, Resistor_SMD:R_Array_Convex_4x0603, F.Cu at (71.5, 61.6)
- added TP6: 3V3ADC, TestPoint:TestPoint_THTPad_1.5x1.5mm_Drill0.7mm, F.Cu at (127.0, 109.7)
- added TP7: 5V, TestPoint:TestPoint_THTPad_1.5x1.5mm_Drill0.7mm, F.Cu at (161.5, 91.9)
- added XX2: stepper_module, stepper:stepper_module, F.Cu at (68.8, 52.4)
- added XX3: stepper_module, stepper:stepper_module, F.Cu at (96.2, 52.4)
- added XX4: stepper_module, stepper:stepper_module, F.Cu at (123.3, 52.3)
- added XX5: stepper_module, stepper:stepper_module, F.Cu at (131.8, 130.1)
- added XX6: stepper_module, stepper:stepper_module, F.Cu at (101.7, 130.2)
- added XX7: stepper_module, stepper:stepper_module, F.Cu at (71.8, 130.2)
- added XX8: stepper_module, stepper:stepper_module, F.Cu at (69.2, 107.9)
- C10, C11, C13, C15, C16, C17, C18, D24, D25, D27, Q2, R18, R19, R20, R21, R22, U4, U6: moved to B.Cu
- C12: value 47u 6V -> 1u; footprint Capacitor_Tantalum_SMD:CP_EIA-3216-18_Kemet-A_Pad1.58x1.35mm_HandSolder -> Capacitor_SMD:C_0603_1608Metric_Pad1.08x0.95mm_HandSolder; moved to B.Cu
- C14: value 100u 16V -> 47u 35V; footprint Capacitor_THT:CP_Radial_D8.0mm_P3.50mm -> Capacitor_Tantalum_SMD:CP_EIA-6032-28_Kemet-C_Pad2.25x2.35mm_HandSolder
- JP1: value SolderJumper_2_Bridged -> CAN; moved to B.Cu
- JP2: value SolderJumper_2_Bridged -> USB5V
- JP3: value SolderJumper_2_Bridged -> MCU
- JP4: value SolderJumper_2_Bridged -> 3V3ADC; moved to B.Cu
- JP5: value SolderJumper_2_Bridged -> 3V3; moved to B.Cu
- JP6: value SolderJumper_2_Bridged -> Vdrive; moved to B.Cu
- JP7: value SolderJumper_2_Bridged -> Vio
- TP2: value 5V -> Vin
- TP4: value 5V -> 5Vext
- moved RN7 231.8 mm to (114.0, 103.2)
- moved JP6 197.7 mm to (154.3, 138.8), turned to 180 degrees
- moved U4 186.4 mm to (129.6, 109.4), turned to 90 degrees
- moved JP5 179.9 mm to (127.6, 82.8)
- moved TP5 178.9 mm to (130.8, 101.2)
- moved JP4 177.6 mm to (136.1, 110.2), turned to 180 degrees
- moved C18 177.1 mm to (130.5, 91.8), turned to 90 degrees
- moved C15 175.7 mm to (127.5, 84.8), turned to 180 degrees
- moved C10 167.9 mm to (143.7, 54.4), turned to 180 degrees
- moved C16 167.4 mm to (130.8, 96.4), turned to -90 degrees
- moved U6 166.7 mm to (126.0, 90.0), turned to -90 degrees
- moved C12 162.8 mm to (132.6, 112.3)
- moved JP1 159.4 mm to (144.6, 59.6), turned to 90 degrees
- moved Q1 156.8 mm to (146.6, 56.1)
- moved SW3 156.3 mm to (155.3, 52.8), turned to -90 degrees
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Connections:
- net /MCU base/Diag renamed /MCU base/Diagn
- net /MCU base/MCU3v3 renamed MCU3v3
- net DIAG renamed DIAGNOST
- D6 pad 4: M6_L0 -> M6_L1
- D6 pad 5: M6_L1 -> M6_L0
- RN7 pad 1: unconnected-(RN7-Pad1) -> /Motors/SCK
- RN7 pad 2: /Motors/MOSI -> /Motors/MISO
- RN7 pad 3: /Motors/MISO -> /Motors/MOSI
- RN7 pad 4: /Motors/SCK -> unconnected-(RN7-Pad4)
- RN7 pad 5: TMC_SCK -> unconnected-(RN7-Pad5)
- RN7 pad 6: TMC_MISO -> TMC_MOSI
- RN7 pad 7: TMC_MOSI -> TMC_MISO
- RN7 pad 8: unconnected-(RN7-Pad8) -> TMC_SCK
- U1 pad 11: M0_L1 -> M0_EN
- U1 pad 41: M6_EN -> M6_L1
- U1 pad 42: M6_DIR -> M6_L0
- U1 pad 43: M6_L0 -> M6_DIR
- U1 pad 44: M6_L1 -> M6_EN
- U1 pad 7: M0_EN -> M0_L1
- U1 pad 78: M3_EN -> M3_L0
- U1 pad 79: M3_DIR -> M3_L1
- U1 pad 8: M0_DIR -> M0_L0
- U1 pad 80: M3_L0 -> M3_DIR
- U1 pad 83: M3_L1 -> M3_EN
- U1 pad 9: M0_L0 -> M0_DIR
- U2 pad 2: /CAN_Rx -> CAN_RX
- U2 pad 3: /CAN_Tx -> CAN_TX
Routing:
- net GND: track 444.4 -> 1108.3 mm, vias 16 -> 21
- net /Motors/Vio: track 25.2 -> 587.4 mm, vias 0 -> 11
- net /Motors/Vm: track 32.0 -> 502.7 mm, vias 0 -> 3
- net /Motors/MISO: track 0.00 -> 355.2 mm, vias 0 -> 16
- net /Motors/SCK: track 0.00 -> 291.8 mm, vias 0 -> 19
- net /Motors/MOSI: track 6.48 -> 239.2 mm, vias 1 -> 19
- net /Motors/USART4-7: track 0.00 -> 157.2 mm, vias 0 -> 11
- net +5V: track 27.8 -> 177.6 mm, vias 3 -> 8
- net /Motors/USART0-3: track 11.9 -> 130.0 mm, vias 1 -> 12
- net Vdrive: track 0.00 -> 111.2 mm, vias 0 -> 7
- net /Motors/DIAG4: track 0.00 -> 110.0 mm, vias 0 -> 7
- net M6_L1: track 12.5 -> 109.3 mm, vias 1 -> 3
- net M5_L1: track 20.9 -> 108.6 mm
- net M6_L0: track 15.3 -> 98.5 mm, vias 1 -> 3
- net M5_L0: track 21.5 -> 99.8 mm
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- added copper zone on In2.Cu, net /Motors/Vm
- added copper zone on In1.Cu, net GND
Other:
- board outline added: 113.5 x 105.5 mm
