File: F3:F303/Multistepper/kicad/stepper_M.kicad_sch (KiCad schematic)
At the start: 17 parts, among them J11 Conn_01x03_Male, J12 Conn_01x03_Male, J13 Conn_01x04_Male

Commit message: multistepper schematic
Parts:
- removed J11: Conn_01x03_Male, Connector_PinHeader_2.54mm:PinHeader_1x03_P2.54mm_Vertical, symbol Connector:Conn_01x03_Male
- removed JP16, JP17: SolderJumper_2_Bridged, Jumper:SolderJumper-2_P1.3mm_Open_TrianglePad1.0x1.5mm, symbol Jumper:SolderJumper_2_Bridged
- J11: renamed from J12; value Conn_01x03_Male -> LimS; footprint Connector_PinHeader_2.54mm:PinHeader_1x03_P2.54mm_Vertical -> Connector_JST:JST_EH_B4B-EH-A_1x04_P2.50mm_Vertical; symbol Connector:Conn_01x03_Male -> Connector:Conn_01x04_Male
- J12: renamed from J13; value Conn_01x04_Male -> Stepper; footprint Connector_PinHeader_2.54mm:PinHeader_1x04_P2.54mm_Vertical -> Connector_JST:JST_EH_B4B-EH-A_1x04_P2.50mm_Vertical
Connections:
- net DIR: no longer RN8.2 (R2.1), XX1.8 (DIR)
- net GND: now also J11.4 (Pin_4); no longer J11.1 (Pin_1)
- net L1/CS: now also J11.3 (Pin_3)
- net STEP: no longer RN8.3 (R3.1), XX1.7 (STEP)
- net UART: no longer JP14.2 (B), JP8.2 (C), XX1.5 (PDN_UART)
- net Vm: now also C19.1, XX1.16 (Vmot)
- net ~{EN}: no longer RN8.4 (R4.1), XX1.1 (~{EN})
- net at R23.2: now also J11.1 (Pin_1); no longer J11.3 (Pin_3)
- net Vio renamed V3v3
- new net DIRx: RN8.2 (R2.1), XX1.8 (DIR)
- new net STEPx: RN8.3 (R3.1), XX1.7 (STEP)
- new net U: JP14.2 (B), JP8.2 (C), XX1.5 (PDN_UART)
- new net ~{ENx}: RN8.4 (R4.1), XX1.1 (~{EN})
Other:
- note removed: "Limit 0"
- note removed: "Limit 1"
- moved on the sheet: R23

Commit message: fixed bug in multisteppers PCB
Changed lines of the file:
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@@
-    (effects (font (size 1.27 1.27)) (justify left bottom))
-  )
-  (label "Vio" (at 83.82 38.354 0)
     (effects (font (size 1.27 1.27)) (justify left bottom))
   )
@@
     (effects (font (size 1.27 1.27)) (justify right bottom))
   )
-  (label "Vio" (at 63.246 39.116 0)
-    (effects (font (size 1.27 1.27)) (justify left bottom))
-  )
   (label "~{ENx}" (at 37.846 42.164 0)
     (effects (font (size 1.27 1.27)) (justify left bottom))
@@
     (effects (font (size 1.27 1.27)) (justify left bottom))
   )
-  (label "Vio" (at 80.01 21.082 0)
-    (effects (font (size 1.27 1.27)) (justify left bottom))
-  )
-  (label "Vio" (at 63.5 21.59 0)
-    (effects (font (size 1.27 1.27)) (justify left bottom))
-  )
   (label "U" (at 103.886 63.246 180)
     (effects (font (size 1.27 1.27)) (justify right bottom))
-  )
-  (label "Vio" (at 149.86 68.326 0)
-    (effects (font (size 1.27 1.27)) (justify left bottom))
   )
   (label "SPR" (at 103.886 60.706 180)
@@
     (effects (font (size 1.27 1.27)) (justify left bottom))
   )
-  (label "Vio" (at 32.131 86.106 270)
-    (effects (font (size 1.27 1.27)) (justify right bottom))
-  )
   (label "DIRx" (at 37.846 47.244 0)
     (effects (font (size 1.27 1.27)) (justify left bottom))
   )
   (label "STEPx" (at 37.846 44.704 0)
-    (effects (font (size 1.27 1.27)) (justify left bottom))
-  )
-  (label "Vio" (at 20.32 18.542 0)
     (effects (font (size 1.27 1.27)) (justify left bottom))
   )
@@
     (effects (font (size 1.27 1.27)) (justify right))
   )
+  (hierarchical_label "V3v3" (shape input) (at 63.5 21.59 180)
+    (effects (font (size 1.27 1.27)) (justify right))
+  )
   (hierarchical_label "L1{slash}CS" (shape bidirectional) (at 32.131 73.406 180)
     (effects (font (size 1.27 1.27)) (justify right))
   )
-  (hierarchical_label "V3v3" (shape input) (at 20.32 18.542 180)
+  (hierarchical_label "V3v3" (shape input) (at 80.01 21.082 180)
     (effects (font (size 1.27 1.27)) (justify right))
+  )
+  (hierarchical_label "V3v3" (shape input) (at 149.86 68.326 0)
+    (effects (font (size 1.27 1.27)) (justify left))
   )
   (hierarchical_label "STEP" (shape input) (at 27.686 44.704 180)
@@
     (effects (font (size 1.27 1.27)) (justify left))
   )
+  (hierarchical_label "V3v3" (shape input) (at 63.246 39.116 180)
+    (effects (font (size 1.27 1.27)) (justify right))
+  )
+  (hierarchical_label "V3v3" (shape input) (at 83.82 38.354 180)
+    (effects (font (size 1.27 1.27)) (justify right))
+  )
   (hierarchical_label "MISO" (shape output) (at 58.166 53.086 180)
     (effects (font (size 1.27 1.27)) (justify right))
   )
+  (hierarchical_label "V3v3" (shape input) (at 32.131 86.106 180)
+    (effects (font (size 1.27 1.27)) (justify right))
+  )

Commit message: change end-switches' connectors to 2mm
Parts:
- J11: footprint Connector_JST:JST_EH_B4B-EH-A_1x04_P2.50mm_Vertical -> Connector_JST:JST_PH_B4B-PH-K_1x04_P2.00mm_Vertical
Changed lines of the file:
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@@
       (effects (font (size 1.27 1.27)) (justify right) hide)
     )
-    (property "Footprint" "Connector_JST:JST_EH_B4B-EH-A_1x04_P2.50mm_Vertical" (id 2) (at 37.211 75.946 0)
+    (property "Footprint" "Connector_JST:JST_PH_B4B-PH-K_1x04_P2.00mm_Vertical" (id 2) (at 37.211 75.946 0)
       (effects (font (size 1.27 1.27)) hide)
     )

Commit message: fixed bug with wrong DIAG output tracking
Connections:
- net Diag: now also XX1.18 (DIAG); no longer XX1.17 (DIAG)
