File: F3:F303/NitrogenFlooding/kicad/nitrogen/MCU.kicad_sch (KiCad schematic)
At the start: 83 parts, among them J1 ADC8,9, J10 IDC2.54_02x05, J11 IDC2.54_02x05, J14 U3/U4, J15 I2C/U1, J16 buzzer, J18 LEDs, J4 IDC2.54_02x05, J6 ADCext, J7 Prog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

Commit message: Finished nitrogen PCB
Changed lines of the file:
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@@
-    (stroke (width 0) (type default) (color 0 0 0 0))
-  )
-  (wire (pts (xy 265.303 20.193) (xy 270.51 20.193))
     (stroke (width 0) (type default) (color 0 0 0 0))
   )
@@
     (stroke (width 0) (type default) (color 0 0 0 0))
   )
-  (wire (pts (xy 247.269 20.193) (xy 252.603 20.193))
-    (stroke (width 0) (type default) (color 0 0 0 0))
-  )
   (wire (pts (xy 269.113 43.307) (xy 269.113 45.847))
     (stroke (width 0) (type default) (color 0 0 0 0))
@@
     (stroke (width 0) (type default) (color 0 0 0 0))
   )
-  (wire (pts (xy 265.303 22.733) (xy 270.51 22.733))
-    (stroke (width 0) (type default) (color 0 0 0 0))
-  )
   (wire (pts (xy 237.363 134.62) (xy 237.363 128.905))
     (stroke (width 0) (type default) (color 0 0 0 0))
@@
     (stroke (width 0) (type default) (color 0 0 0 0))
   )
-  (wire (pts (xy 247.269 25.273) (xy 252.603 25.273))
-    (stroke (width 0) (type default) (color 0 0 0 0))
-  )
   (wire (pts (xy 257.81 154.94) (xy 260.477 154.94))
     (stroke (width 0) (type default) (color 0 0 0 0))
@@
     (stroke (width 0) (type default) (color 0 0 0 0))
   )
-  (wire (pts (xy 247.269 22.733) (xy 252.603 22.733))
-    (stroke (width 0) (type default) (color 0 0 0 0))
-  )
   (wire (pts (xy 169.799 184.277) (xy 164.592 184.277))
     (stroke (width 0) (type default) (color 0 0 0 0))
@@
     (stroke (width 0) (type default) (color 0 0 0 0))
   )
-  (wire (pts (xy 265.303 25.273) (xy 270.51 25.273))
-    (stroke (width 0) (type default) (color 0 0 0 0))
-  )
   (wire (pts (xy 242.189 121.285) (xy 245.11 121.285))
     (stroke (width 0) (type default) (color 0 0 0 0))
@@
     (stroke (width 0) (type default) (color 0 0 0 0))
   )
-  (wire (pts (xy 265.303 27.813) (xy 270.51 27.813))
-    (stroke (width 0) (type default) (color 0 0 0 0))
-  )
   (wire (pts (xy 153.67 176.657) (xy 159.258 176.657))
     (stroke (width 0) (type default) (color 0 0 0 0))
@@
     (stroke (width 0) (type default) (color 0 0 0 0))
   )
-  (wire (pts (xy 247.269 27.813) (xy 252.603 27.813))
-    (stroke (width 0) (type default) (color 0 0 0 0))
-  )

Commit message: Some little fixes + add BOM
Parts:
- J8: footprint Connector_USB:USB_B_OST_USB-B1HSxx_Horizontal -> Connector_USB:USB_B_TE_5787834_Vertical
Connections:
- net ADC0: now also J4.9 (Pin_9); no longer J4.1 (Pin_1)
- net ADC1: now also J4.10 (Pin_10); no longer J4.2 (Pin_2)
- net ADC2: now also J4.7 (Pin_7); no longer J4.3 (Pin_3)
- net ADC3: now also J4.8 (Pin_8); no longer J4.4 (Pin_4)
- net ADC6: now also J4.3 (Pin_3); no longer J4.7 (Pin_7)
- net ADC7: now also J4.4 (Pin_4); no longer J4.8 (Pin_8)
- net GNDPWR: now also J4.1 (Pin_1), J4.2 (Pin_2); no longer J4.10 (Pin_10), J4.9 (Pin_9)
Changed lines of the file:
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@@
       (effects (font (size 1.27 1.27)) (justify right))
     )
-    (property "Footprint" "Connector_USB:USB_B_OST_USB-B1HSxx_Horizontal" (id 2) (at 74.041 143.129 0)
+    (property "Footprint" "Connector_USB:USB_B_TE_5787834_Vertical" (id 2) (at 74.041 143.129 0)
       (effects (font (size 1.27 1.27)) hide)
     )
@@
     (pin "2")
   )
-  (symbol (lib_id "Connector_Generic:Conn_02x05_Odd_Even") (at 257.683 25.273 0) (unit 1)
+  (symbol (lib_id "Connector_Generic:Conn_02x05_Odd_Even") (at 257.683 25.273 0) (mirror x) (unit 1)
     (in_bom yes) (on_board yes)
-    (property "Reference" "J4" (id 0) (at 258.953 17.653 0))
-    (property "Value" "IDC2.54_02x05" (id 1) (at 255.651 33.147 0))
+    (property "Reference" "J4" (id 0) (at 258.953 32.893 0))
+    (property "Value" "IDC2.54_02x05" (id 1) (at 255.651 17.399 0))
     (property "Footprint" "Connector_IDC:IDC-Header_2x05_P2.54mm_Vertical" (id 2) (at 257.683 25.273 0)
       (effects (font (size 1.27 1.27)) hide)
