File: F3:F303/NitrogenFlooding/kicad/nitrogen/nitrogen.kicad_pcb (KiCad board)
At the start: 4 copper layers, 80 x 80 mm, 140 parts, among them J1 ADC8,9, J10 IDC2.54_02x05, J11 IDC2.54_02x05, J12 Power, J13 Screw_Terminal_01x02, J14 U3/U4, J15 I2C/U1, J16 buzzer, J18 LEDs, J2 Screw_Terminal_01x02, J3 Screw_Terminal_01x02, J4 IDC2.54_02x05, J5 Power, J6 ADCext, J7 Prog, J8 USB_B, J9 485/CAN, Q1 AOD4184, Q2 AOD4184, Q3 AOD4184, Q4 AOD4184, Q5 DTA114Y, Q6 SI2300, Q8 IRF9310, Q9 SI2305, U1 MCP2551-I-SN, U2 USBLC6-2SC6, U3 MAX3485, U4 STM32F302VBTx, U5 BME280, U6 LM2576HVS-5, U7 LM1117-3.3, U8 LM1117-3.3, Y1 NX5032GA-8MHz

Commit message: Finished nitrogen PCB
Routing:
- net GND: track 507.1 -> 506.1 mm
Other:
- board text added: "3.3V LED0 LED1 LED2 LED3"
- board text added: "485A"
- board text added: "485B"
- board text added: "ADC0..7"
- board text added: "ADC0..7: 1 3 5 7 G 0 2 4 6 G"
- board text added: "ADC9 ADC8 GND"
- board text added: "Buttons"
- board text added: "Buttons: B0 B1 B2 B3 B4 B5 B6 3v3 Gnd Gnd"
- board text added: "CANH"
- board text added: "CANL"
- board text added: "Ext. ADC:"
- board text added: "G 3.3 5"
- board text added: "GND"
- board text added: "Gnd 3.3 5"
- board text added: "Gnd 5V 3.3V ADC in"
- board text added: "PWM Gnd 0..3"
- board text added: "PWM0"
- board text added: "PWM1"
- board text added: "PWM2"
- board text added: "PWM3"
- board text added: "Prog: SWCLK SWDIO Gnd 3.3V BOOT0 NRST"
- board text added: "Rx Tx Gnd"
- board text added: "SAO RAS"
- board text added: "SCL SDA Gnd"
- board text added: "Screen"
- board text added: "Screen: Gnd 5V MISO SCK Gnd 3.3V NSS RST MOSI DCRS"
- board text added: "Tx Rx Gnd"
- board text added: "https://github.com/eddyem/stm32samples/tree/master/F3:F303/NitrogenFlooding"

Commit message: Some little fixes + add BOM
Parts:
- D1, D2, Q9, R1, R29, R31, R33, R35, R37, R39: moved to F.Cu
- J3, J4, Q5, R13: moved to B.Cu
- J8: footprint Connector_USB:USB_B_OST_USB-B1HSxx_Horizontal -> Connector_USB:USB_B_TE_5787834_Vertical
- moved J4 10.2 mm to (133.1, 53.0)
- moved D5 5.22 mm to (176.5, 90.1)
- moved J3 5.00 mm to (118.5, 119.5), turned to 0 degrees
- moved J8 3.22 mm to (169.4, 91.7), turned to 90 degrees
- moved R13 3.17 mm to (164.0, 95.1)
- moved R14 2.08 mm to (165.6, 102.3)
- moved R1 1.93 mm to (116.5, 58.2)
- moved R39 1.93 mm to (118.5, 58.2)
- moved TP1 1.79 mm to (177.2, 83.7)
- moved Q5 1.50 mm to (165.4, 93.0)
- moved U2 1.43 mm to (163.1, 97.7)
- moved R15 0.82 mm to (168.2, 98.7)
- moved D2 0.72 mm to (114.6, 118.4)
- moved R18 0.57 mm to (168.2, 96.8)
Connections:
- J3 pad 1: /P2 -> /P3
- J3 pad 2: /P3 -> /P2
- J4 pad 1: /MCU/ADC0 -> GNDPWR
- J4 pad 10: GNDPWR -> /MCU/ADC1
- J4 pad 2: /MCU/ADC1 -> GNDPWR
- J4 pad 3: /MCU/ADC2 -> /MCU/ADC6
- J4 pad 4: /MCU/ADC3 -> /MCU/ADC7
- J4 pad 7: /MCU/ADC6 -> /MCU/ADC2
- J4 pad 8: /MCU/ADC7 -> /MCU/ADC3
- J4 pad 9: GNDPWR -> /MCU/ADC0
Routing:
- net GND: track 506.1 -> 498.2 mm
- net /MCU/VB: track 14.7 -> 20.1 mm
- net Net-(D5-Pad1): track 7.81 -> 11.6 mm
- net /P3: track 26.6 -> 23.3 mm
- net /MCU/USB_DP: track 6.43 -> 9.52 mm, vias 1 -> 0
- net Net-(Q5-Pad3): track 5.81 -> 3.32 mm
- net /MCU/MCU3v3: track 123.7 -> 122.1 mm
- net /MCU/USB_DM: track 6.74 -> 5.20 mm
- net +3.3VADC: track 100.1 -> 98.6 mm
- net /MCU/NRST: track 49.4 -> 48.1 mm
- net /MCU/USB_PU: track 8.71 -> 7.73 mm, vias 1 -> 0
- net /MCU/SWDIO: track 23.8 -> 22.9 mm
- net Net-(R18-Pad2): track 2.22 -> 3.09 mm
- net Net-(R15-Pad2): track 2.29 -> 3.09 mm
- net /MCU/BOOT0: track 39.1 -> 38.4 mm
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Other:
- outline, holes or cut-outs redrawn
- board text added: "485B 485A GND CANL CANH"
- board text added: "ADC0..7: G 7 5 3 1 G 6 4 2 0"
- board text added: "NitrogenFlooding"
- board text added: "PWM Gnd"
- board text removed: "485A"
- board text removed: "485B"
- board text removed: "ADC0..7: 1 3 5 7 G 0 2 4 6 G"
- board text removed: "CANH"
- board text removed: "CANL"
- board text removed: "Ext. ADC:"
- board text removed: "G 3.3 5"
- board text removed: "GND"
- board text removed: "PWM Gnd 0..3"
- board text removed: "SAO RAS"
- board text removed: "https://github.com/eddyem/stm32samples/tree/master/F3:F303/NitrogenFlooding"
