File: F3:F303/NitrogenFlooding/kicad/nitrogen/nitrogen.kicad_sch (KiCad schematic)
At the start: 22 parts, among them J2 Screw_Terminal_01x02, J3 Screw_Terminal_01x02, Q1 AOD4184, Q2 AOD4184, Q3 AOD4184, Q4 AOD4184

Commit message: Some little fixes + add BOM
Connections:
- net P2: now also J3.2 (Pin_2); no longer J3.1 (Pin_1)
- net P3: now also J3.1 (Pin_1); no longer J3.2 (Pin_2)
Changed lines of the file:
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@@
     (effects (font (size 1.27 1.27)) (justify left bottom))
   )
-  (label "P3" (at 230.759 85.344 0)
+  (label "P3" (at 230.759 87.884 0)
     (effects (font (size 1.27 1.27)) (justify left bottom))
   )
-  (label "P2" (at 230.759 87.884 0)
+  (label "P2" (at 230.759 85.344 0)
     (effects (font (size 1.27 1.27)) (justify left bottom))
   )
@@
     )
     (path "/6595f7bf-be90-4ec5-9ee8-68919a05962c/8921e3b8-179f-454e-8cfd-6d917224d0b0"
-      (reference "J8") (unit 1) (value "USB_B") (footprint "Connector_USB:USB_B_OST_USB-B1HSxx_Horizontal")
+      (reference "J8") (unit 1) (value "USB_B") (footprint "Connector_USB:USB_B_TE_5787834_Vertical")
     )
     (path "/6595f7bf-be90-4ec5-9ee8-68919a05962c/61aa389c-dca9-4090-8791-3f89cf734c62"
