File: F3:F303/CANbus4BTA/kicad/optocouple.kicad_sch (KiCad schematic)
At the start: 2 parts, among them U11 PC817

Commit message: some code fixes, start to draw new schematic
Parts:
- R31: value 360 -> 3k3; footprint Resistor_SMD:R_0603_1608Metric_Pad0.98x0.95mm_HandSolder -> Resistor_SMD:R_2010_5025Metric_Pad1.40x2.65mm_HandSolder
Other:
- company: (none) -> SAO RAS
Changed lines of the file:
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@@
 	(generator_version "8.99")
 	(paper "A4")
+	(title_block
+		(date "2024-03-18")
+		(company "SAO RAS")
+		(comment 1 "Instead of PEP controller")
+	)
 	(wire
 		(pts
@@
 			)
 		)
-		(property "Value" "360"
+		(property "Value" "3k3"
 			(at 109.093 51.943 90)
 			(effects
@@
 			)
 		)
-		(property "Footprint" "Resistor_SMD:R_0603_1608Metric_Pad0.98x0.95mm_HandSolder"
+		(property "Footprint" "Resistor_SMD:R_2010_5025Metric_Pad1.40x2.65mm_HandSolder"
 			(at 107.442 50.419 90)
 			(effects

Commit message: seems like schematic is ready
Parts:
- renumbered R31 to R39, U11 to U12
Connections:
- net EXT5V renamed EXTV
Other:
- note added: "EXTV=24V -> R=3k3 EXTV=9V -> R=1k"
- moved on the sheet: R39, U12
Changed lines of the file:
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@@
 	(wire
 		(pts
-			(xy 129.413 54.229) (xy 124.46 54.229)
+			(xy 119.38 51.435) (xy 114.3 51.435)
 		)
 		(stroke
@@
 	(wire
 		(pts
-			(xy 124.46 59.309) (xy 129.286 59.309)
+			(xy 114.3 56.515) (xy 119.38 56.515)
 		)
 		(stroke
@@
 		)
 	)
-	(hierarchical_label "EXT5V"
-		(shape input)
-		(at 109.22 46.609 0)
+	(text "EXTV=24V -> R=3k3\nEXTV=9V -> R=1k "
+		(exclude_from_sim no)
+		(at 108.585 38.1 0)
+		(effects
+			(font
+				(size 1.27 1.27)
+			)
+		)
+	)
+	(hierarchical_label "EXTV"
+		(shape input)
+		(at 99.06 43.815 0)
 		(fields_autoplaced yes)
 		(effects
@@
 	(hierarchical_label "In"
 		(shape input)
-		(at 129.413 54.229 0)
+		(at 119.38 51.435 0)
 		(fields_autoplaced yes)
 		(effects
@@
 	(hierarchical_label "gnd"
 		(shape input)
-		(at 129.286 59.309 0)
+		(at 119.38 56.515 0)
 		(fields_autoplaced yes)
 		(effects
@@
 	(hierarchical_label "EXTi"
 		(shape input)
-		(at 109.22 59.309 180)
+		(at 99.06 56.515 180)
 		(fields_autoplaced yes)
 		(effects
@@
 	(symbol
 		(lib_id "Device:R")
-		(at 109.22 50.419 0)
+		(at 99.06 47.625 0)
 		(unit 1)
 		(exclude_from_sim no)
@@
 		(on_board yes)
 		(dnp no)
-		(property "Reference" "R31"
-			(at 110.998 49.5843 0)
+		(property "Reference" "R39"
+			(at 100.838 46.7903 0)
 			(effects
 				(font
@@
 		)
 		(property "Value" "3k3"
-			(at 109.093 51.943 90)
+			(at 98.933 49.149 90)
 			(effects
 				(font
@@
 		)
 		(property "Footprint" "Resistor_SMD:R_2010_5025Metric_Pad1.40x2.65mm_HandSolder"
-			(at 107.442 50.419 90)
+			(at 97.282 47.625 90)
 			(effects
 				(font
@@
 		)
 		(property "Datasheet" "~"
-			(at 109.22 50.419 0)
+			(at 99.06 47.625 0)
 			(effects
 				(font
@@
 		)
 		(property "Description" ""
-			(at 109.22 50.419 0)
+			(at 99.06 47.625 0)
+			(effects
+				(font
+					(size 1.27 1.27)
+				)
+				(hide yes)
+			)
+		)
+		(property "Manufacturer" ""
+			(at 99.06 47.625 0)
 			(effects
 				(font
@@
 			(project "stm32"
 				(path "/f40cbe7e-cd25-45e5-a6cb-d92457495048/311a5cb3-0370-4a86-a5e8-6335fee47f9a"
-					(reference "R31")
+					(reference "R39")
 					(unit 1)
 				)
 				(path "/f40cbe7e-cd25-45e5-a6cb-d92457495048/2b18f3bb-219b-4cc5-8bc9-bc122d6e81e9"
-					(reference "R35")
+					(reference "R43")
 					(unit 1)
 				)
 				(path "/f40cbe7e-cd25-45e5-a6cb-d92457495048/c51c7789-4b67-42c9-a921-b1066b3f95ba"
-					(reference "R37")
+					(reference "R45")
 					(unit 1)
 				)
 				(path "/f40cbe7e-cd25-45e5-a6cb-d92457495048/737c47dd-2cc5-4c23-ab54-7bef18beb2a3"
-					(reference "R32")
+					(reference "R40")
 					(unit 1)
 				)
 				(path "/f40cbe7e-cd25-45e5-a6cb-d92457495048/0ff6ac13-ac49-41f0-9506-376ccd8b8ba4"
-					(reference "R33")
+					(reference "R41")
 					(unit 1)
 				)
 				(path "/f40cbe7e-cd25-45e5-a6cb-d92457495048/1cf77ae7-411e-49cc-bbff-6947c0aa32bd"
-					(reference "R34")
+					(reference "R42")
 					(unit 1)
 				)
 				(path "/f40cbe7e-cd25-45e5-a6cb-d92457495048/d7c9ec36-f6b4-4bc2-8e9a-7a0792b9eff0"
-					(reference "R36")
+					(reference "R44")
 					(unit 1)
 				)
 				(path "/f40cbe7e-cd25-45e5-a6cb-d92457495048/e5255d96-2d32-432c-bf31-9afa6ac7ec6a"
-					(reference "R38")
+					(reference "R46")
 					(unit 1)
 				)
@@
 	(symbol
 		(lib_id "Isolator:PC817")
-		(at 116.84 56.769 0)
+		(at 106.68 53.975 0)
 		(unit 1)
 		(exclude_from_sim no)
@@
 		(dnp no)
 		(fields_autoplaced yes)
-		(property "Reference" "U11"
-			(at 116.84 49.2592 0)
+		(property "Reference" "U12"
+			(at 106.68 46.4652 0)
 			(effects
 				(font
@@
 		)
 		(property "Value" "PC817"
-			(at 116.84 51.7961 0)
+			(at 106.68 49.0021 0)
 			(effects
 				(font
@@
 		)
 		(property "Footprint" "Package_DIP:DIP-4_W7.62mm"
-			(at 111.76 61.849 0)
+			(at 101.6 59.055 0)
 			(effects
 				(font
@@
 		)
 		(property "Datasheet" "http://www.soselectronic.cz/a_info/resource/d/pc817.pdf"
-			(at 116.84 56.769 0)
+			(at 106.68 53.975 0)
 			(effects
 				(font
@@
 		)
 		(property "Description" ""
-			(at 116.84 56.769 0)
+			(at 106.68 53.975 0)
+			(effects
+				(font
+					(size 1.27 1.27)
+				)
+				(hide yes)
+			)
+		)
+		(property "Manufacturer" ""
+			(at 106.68 53.975 0)
 			(effects
 				(font
@@
 			(project "stm32"
 				(path "/f40cbe7e-cd25-45e5-a6cb-d92457495048/311a5cb3-0370-4a86-a5e8-6335fee47f9a"
-					(reference "U11")
+					(reference "U12")
 					(unit 1)
 				)
 				(path "/f40cbe7e-cd25-45e5-a6cb-d92457495048/2b18f3bb-219b-4cc5-8bc9-bc122d6e81e9"
+					(reference "U16")
+					(unit 1)
+				)
+				(path "/f40cbe7e-cd25-45e5-a6cb-d92457495048/c51c7789-4b67-42c9-a921-b1066b3f95ba"
+					(reference "U18")
+					(unit 1)
+				)
+				(path "/f40cbe7e-cd25-45e5-a6cb-d92457495048/737c47dd-2cc5-4c23-ab54-7bef18beb2a3"
+					(reference "U13")
+					(unit 1)
+				)
+				(path "/f40cbe7e-cd25-45e5-a6cb-d92457495048/0ff6ac13-ac49-41f0-9506-376ccd8b8ba4"
+					(reference "U14")
+					(unit 1)
+				)
+				(path "/f40cbe7e-cd25-45e5-a6cb-d92457495048/1cf77ae7-411e-49cc-bbff-6947c0aa32bd"
 					(reference "U15")
 					(unit 1)
 				)
-				(path "/f40cbe7e-cd25-45e5-a6cb-d92457495048/c51c7789-4b67-42c9-a921-b1066b3f95ba"
+				(path "/f40cbe7e-cd25-45e5-a6cb-d92457495048/d7c9ec36-f6b4-4bc2-8e9a-7a0792b9eff0"
 					(reference "U17")
 					(unit 1)
 				)
-				(path "/f40cbe7e-cd25-45e5-a6cb-d92457495048/737c47dd-2cc5-4c23-ab54-7bef18beb2a3"
-					(reference "U12")
-					(unit 1)
-				)
-				(path "/f40cbe7e-cd25-45e5-a6cb-d92457495048/0ff6ac13-ac49-41f0-9506-376ccd8b8ba4"
-					(reference "U13")
-					(unit 1)
-				)
-				(path "/f40cbe7e-cd25-45e5-a6cb-d92457495048/1cf77ae7-411e-49cc-bbff-6947c0aa32bd"
-					(reference "U14")
-					(unit 1)
-				)
-				(path "/f40cbe7e-cd25-45e5-a6cb-d92457495048/d7c9ec36-f6b4-4bc2-8e9a-7a0792b9eff0"
-					(reference "U16")
-					(unit 1)
-				)
 				(path "/f40cbe7e-cd25-45e5-a6cb-d92457495048/e5255d96-2d32-432c-bf31-9afa6ac7ec6a"
-					(reference "U18")
-					(unit 1)
-				)
+					(reference "U19")
+					(unit 1)
+				)

Commit message: optocouples
Parts:
- added U21: EL814, symbol Isolator:EL814
Changed lines of the file:
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@@
+		)
+	)
+	(symbol
+		(lib_id "Isolator:EL814")
+		(at 104.775 71.755 0)
+		(unit 1)
+		(exclude_from_sim no)
+		(in_bom yes)
+		(on_board yes)
+		(dnp no)
+		(fields_autoplaced yes)
+		(property "Reference" "U21"
+			(at 104.775 63.8005 0)
+			(effects
+				(font
+					(size 1.27 1.27)
+				)
+			)
+		)
+		(property "Value" "EL814"
+			(at 104.775 66.2248 0)
+			(effects
+				(font
+					(size 1.27 1.27)
+				)
+			)
+		)
+		(property "Footprint" ""
+			(at 99.695 76.835 0)
+			(effects
+				(font
+					(size 1.27 1.27)
+					(italic yes)
+				)
+				(justify left)
+				(hide yes)
+			)
+		)
+		(property "Datasheet" "http://www.everlight.com/file/ProductFile/EL814.pdf"
+			(at 105.41 71.755 0)
+			(effects
+				(font
+					(size 1.27 1.27)
+				)
+				(justify left)
+				(hide yes)
+			)
+		)
+		(property "Description" "AC/DC NPN Optocoupler, DIP4/SMD4"
+			(at 104.775 71.755 0)
+			(effects
+				(font
+					(size 1.27 1.27)
+				)
+				(hide yes)
+			)
+		)
+		(pin "4"
+		)
+		(pin "3"
+		)
+		(pin "2"
+		)
+		(pin "1"
+		)
+		(instances
+			(project "stm32"
+				(path "/f40cbe7e-cd25-45e5-a6cb-d92457495048/737c47dd-2cc5-4c23-ab54-7bef18beb2a3"
+					(reference "U21")
+					(unit 1)
+				)
+				(path "/f40cbe7e-cd25-45e5-a6cb-d92457495048/311a5cb3-0370-4a86-a5e8-6335fee47f9a"
+					(reference "U20")
+					(unit 1)
+				)
+				(path "/f40cbe7e-cd25-45e5-a6cb-d92457495048/0ff6ac13-ac49-41f0-9506-376ccd8b8ba4"
+					(reference "U22")
+					(unit 1)
+				)
+				(path "/f40cbe7e-cd25-45e5-a6cb-d92457495048/1cf77ae7-411e-49cc-bbff-6947c0aa32bd"
+					(reference "U23")
+					(unit 1)
+				)
+				(path "/f40cbe7e-cd25-45e5-a6cb-d92457495048/2b18f3bb-219b-4cc5-8bc9-bc122d6e81e9"
+					(reference "U24")
+					(unit 1)
+				)
+				(path "/f40cbe7e-cd25-45e5-a6cb-d92457495048/d7c9ec36-f6b4-4bc2-8e9a-7a0792b9eff0"
+					(reference "U25")
+					(unit 1)
+				)
+				(path "/f40cbe7e-cd25-45e5-a6cb-d92457495048/c51c7789-4b67-42c9-a921-b1066b3f95ba"
+					(reference "U26")
+					(unit 1)
+				)
+				(path "/f40cbe7e-cd25-45e5-a6cb-d92457495048/e5255d96-2d32-432c-bf31-9afa6ac7ec6a"
+					(reference "U27")
+					(unit 1)
+				)
+			)
 		)
 	)
