File: F0:F030,F042,F072/usbcan_relay/kicad/stm32.kicad_sch (KiCad schematic)
At the start: 98 parts

Commit message: Add LEDs
Parts:
- C1, C5: value (none) -> 1; footprint (none) -> Capacitor_SMD:C_0805_2012Metric_Pad1.15x1.40mm_HandSolder
- C11, C15, C2, C3, C4, C6, C7, C8, C9: value (none) -> 0.1; footprint (none) -> Capacitor_SMD:C_0603_1608Metric_Pad1.05x0.95mm_HandSolder
- C12: value (none) -> 47u 6V; footprint (none) -> Capacitor_Tantalum_SMD:CP_EIA-3216-18_Kemet-A_Pad1.58x1.35mm_HandSolder
- C13: value (none) -> 47u 10V; footprint (none) -> Capacitor_Tantalum_SMD:CP_EIA-6032-28_Kemet-C_Pad2.25x2.35mm_HandSolder
- C14: value (none) -> 100u 16V; footprint (none) -> Capacitor_THT:CP_Radial_D8.0mm_P3.50mm
- D1: value (none) -> PESD1CAN; footprint (none) -> TO_SOT_Packages_SMD:SOT-23
- D10, D2, D4, D8, D9: value (none) -> SS14; footprint (none) -> Diode_SMD:D_SMA-SMB_Universal_Handsoldering
- D11: value (none) -> 1N5822; footprint (none) -> Diode_THT:D_DO-201_P3.81mm_Vertical_AnodeUp
- D3: value (none) -> USB6B1; footprint (none) -> Package_SO:SOIC-8_3.9x4.9mm_P1.27mm
- D5: value (none) -> MM3Z7V5; footprint (none) -> Diode_SMD:D_0805_2012Metric_Pad1.15x1.40mm_HandSolder
- D6, D7: value (none) -> CESD3v3; footprint (none) -> Diode_SMD:D_SOD-523
- J1: value (none) -> +3.3V; footprint (none) -> Connector_PinHeader_2.54mm:PinHeader_1x01_P2.54mm_Vertical
- J10: value (none) -> Screw_Terminal_01x02; footprint (none) -> TerminalBlock_Phoenix:TerminalBlock_Phoenix_MKDS-1,5-2_1x02_P5.00mm_Horizontal
- J11, J12, J17: value (none) -> Screw_Terminal_01x03; footprint (none) -> TerminalBlock_Phoenix:TerminalBlock_Phoenix_MKDS-1,5-3_1x03_P5.00mm_Horizontal
- J13: value (none) -> USB_B; footprint (none) -> Connectors_USB:USB_B_OST_USB-B1HSxx_Horizontal
- J15: value (none) -> 01x03; footprint (none) -> Connector_PinSocket_2.54mm:PinSocket_1x03_P2.54mm_Vertical
- J16, J9: value (none) -> Conn_01x02_Female; footprint (none) -> Connector_PinSocket_2.54mm:PinSocket_1x02_P2.54mm_Vertical
- J18: value (none) -> 01x05; footprint (none) -> Connector_PinSocket_2.54mm:PinSocket_1x05_P2.54mm_Vertical
- J2: value (none) -> NRST; footprint (none) -> Connector_PinHeader_2.54mm:PinHeader_1x01_P2.54mm_Vertical
- J3: value (none) -> BOOT0; footprint (none) -> Connector_PinHeader_2.54mm:PinHeader_1x01_P2.54mm_Vertical
- J4: value (none) -> SWDIO; footprint (none) -> Connector_PinHeader_2.54mm:PinHeader_1x01_P2.54mm_Vertical
- J5: value (none) -> SWCLK; footprint (none) -> Connector_PinHeader_2.54mm:PinHeader_1x01_P2.54mm_Vertical
- J6: value (none) -> GND; footprint (none) -> Connector_PinHeader_2.54mm:PinHeader_1x01_P2.54mm_Vertical
- J7: value (none) -> 01x05; footprint (none) -> Connector_PinHeader_2.54mm:PinHeader_1x05_P2.54mm_Vertical
- J8: value (none) -> Connector_Generic:Conn_02x04_Odd_Even; footprint (none) -> Connector_PinHeader_2.54mm:PinHeader_2x04_P2.54mm_Vertical
- JP1: value (none) -> NON-ISOL; footprint (none) -> Resistor_THT:R_Axial_DIN0207_L6.3mm_D2.5mm_P5.08mm_Vertical; symbol Device:Jumper -> Jumper:Jumper_2_Open
- K1, K2: value (none) -> G5LE-1; footprint (none) -> Relay_THT:Relay_SPDT_SANYOU_SRD_Series_Form_C
- L1: value (none) -> 100u; footprint (none) -> Inductor_SMD:L_12x12mm_H4.5mm
- P1, P2, P3, P4, P5, P6, P7: value (none) -> Hole; footprint (none) -> my_footprints:Hole_3mm
- Q1: value (none) -> B0505S; footprint (none) -> my_footprints:B0x0xS
- Q2, Q3, Q5, Q6, Q7: value (none) -> SI2300; footprint (none) -> TO_SOT_Packages_SMD:SOT-23_Handsoldering
- Q4: value (none) -> AO3407; footprint (none) -> TO_SOT_Packages_SMD:SOT-23_Handsoldering
- R1, R14, R17, R21, R25, R26, R27, R8: value (none) -> 10k; footprint (none) -> Resistor_SMD:R_0603_1608Metric_Pad1.05x0.95mm_HandSolder
- R10, R11, R3: value (none) -> 22; footprint (none) -> Resistor_SMD:R_0603_1608Metric_Pad1.05x0.95mm_HandSolder
- R12, R16: value (none) -> 2k2; footprint (none) -> Resistor_SMD:R_0603_1608Metric_Pad1.05x0.95mm_HandSolder
- R13: value (none) -> 120; footprint (none) -> Resistor_SMD:R_1210_3225Metric_Pad1.42x2.65mm_HandSolder
- R15, R22, R23, R24, R9: value (none) -> 330; footprint (none) -> Resistor_SMD:R_0603_1608Metric_Pad1.05x0.95mm_HandSolder
- R18: value (none) -> 47k; footprint (none) -> Resistor_SMD:R_0603_1608Metric_Pad1.05x0.95mm_HandSolder
- R19, R20: value (none) -> 15k; footprint (none) -> Resistor_SMD:R_0603_1608Metric_Pad1.05x0.95mm_HandSolder
- R2: value (none) -> 4k7; footprint (none) -> Resistor_SMD:R_0603_1608Metric_Pad1.05x0.95mm_HandSolder
- R4, R5, R6, R7: value (none) -> 680; footprint (none) -> Resistor_SMD:R_0603_1608Metric_Pad1.05x0.95mm_HandSolder
- SW1: value (none) -> SW_DIP_x08; footprint (none) -> Button_Switch_THT:SW_DIP_SPSTx08_Slide_9.78x22.5mm_W7.62mm_P2.54mm
- SW2: value (none) -> SW_DIP_x01; footprint (none) -> Button_Switch_THT:SW_DIP_SPSTx01_Slide_6.7x4.1mm_W7.62mm_P2.54mm_LowProfile
- TP1: value (none) -> 5V; footprint (none) -> Connector_PinSocket_2.54mm:PinSocket_1x01_P2.54mm_Vertical
- TP2: value (none) -> 3.3V; footprint (none) -> Connector_PinSocket_2.54mm:PinSocket_1x01_P2.54mm_Vertical
- U1: value (none) -> MCP2551-I/SN; footprint (none) -> Package_SO:SOIC-8_3.9x4.9mm_P1.27mm
- U2: value (none) -> ISO1050DUB; footprint (none) -> Package_SO:SOP-8_6.62x9.15mm_P2.54mm
- U3: value (none) -> STM32F072C8Tx; footprint (none) -> Package_QFP:LQFP-48_7x7mm_P0.5mm
- U4: value (none) -> LM2576; footprint (none) -> TO_SOT_Packages_THT:TO-220-5_P3.4x3.7mm_StaggerEven_Lead3.8mm_Vertical
- U5: value (none) -> LM1117-3.3; footprint (none) -> TO_SOT_Packages_SMD:SOT-223-3_TabPin2
- U6: value (none) -> IP4220CZ6; footprint (none) -> Package_SO:TSOP-6_1.65x3.05mm_P0.95mm
Connections:
- net Earth: now also JP1.2 (B)
- net GND: now also JP1.1 (A)
