File: F0:F030,F042,F072/usbcan_relay/kicad/stm32.kicad_pcb (KiCad board)
At the start: 2 copper layers, 98 x 63.5 mm, 98 parts, among them J1 +3.3V, J10 Screw_Terminal_01x02, J11 Screw_Terminal_01x03, J12 Screw_Terminal_01x03, J13 USB_B, J15 01x03, J16 Conn_01x02_Female, J17 Screw_Terminal_01x03, J18 01x05, J2 NRST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

Commit message: add simplest blink for STM32F407
Other:
- net class 0.5 removed
- net class 1 removed
- net class Default removed
