File: F0:F030,F042,F072/CANbus_stepper/kicad/stm32.kicad_sch (KiCad schematic)
At the start: 68 parts

Commit message: some code fixes, start to draw new schematic
Parts:
- C1, C10, C11, C12, C3, C5, C7, C8, C9: value (none) -> 0.1; footprint (none) -> Capacitor_SMD:C_0603_1608Metric_Pad1.05x0.95mm_HandSolder
- C2: value (none) -> 100uF; footprint (none) -> Capacitor_THT:CP_Radial_D8.0mm_P3.50mm
- C4, C6: value (none) -> 47uF, 10V; footprint (none) -> Capacitor_Tantalum_SMD:CP_EIA-6032-28_Kemet-C_Pad2.25x2.35mm_HandSolder
- D1, D2: value (none) -> MBRS130L; footprint (none) -> Diode_SMD:D_SMB_Handsoldering
- D3: value (none) -> PESD3V3L4UG; footprint (none) -> TO_SOT_Packages_SMD:SOT-363_SC-70-6_Handsoldering
- D4: value (none) -> PESD1CAN; footprint (none) -> TO_SOT_Packages_SMD:SOT-23_Handsoldering
- D5: value (none) -> MM3Z7V5; footprint (none) -> Diode_SMD:D_0805_2012Metric_Pad1.15x1.40mm_HandSolder
- D6: value (none) -> USB6B1; footprint (none) -> Package_SO:SOIC-8_3.9x4.9mm_P1.27mm
- D7, D8: value (none) -> MM3Z4V7; footprint (none) -> Diode_SMD:D_0805_2012Metric_Pad1.15x1.40mm_HandSolder
- F1: value (none) -> 1A; footprint (none) -> MyFootprints:FuseHolder
- J1: value (none) -> A; footprint (none) -> TerminalBlock_Phoenix:TerminalBlock_Phoenix_MKDS-1,5-2_1x02_P5.00mm_Horizontal
- J10: value (none) -> 12v; footprint (none) -> TerminalBlock_Phoenix:TerminalBlock_Phoenix_MKDS-1,5-2_1x02_P5.00mm_Horizontal
- J11: value (none) -> DB9_Male; footprint (none) -> Connector_Dsub:DSUB-9_Male_Horizontal_P2.77x2.84mm_EdgePinOffset4.94mm_Housed_MountingHolesOffset7.48mm
- J12: value (none) -> RS-485; footprint (none) -> TerminalBlock_Phoenix:TerminalBlock_Phoenix_MKDS-1,5-2_1x02_P5.00mm_Horizontal
- J13: value (none) -> Conn_01x06; footprint (none) -> Connector_PinSocket_2.54mm:PinSocket_1x06_P2.54mm_Vertical
- J2: value (none) -> B; footprint (none) -> TerminalBlock_Phoenix:TerminalBlock_Phoenix_MKDS-1,5-2_1x02_P5.00mm_Horizontal
- J3, J4: value (none) -> Conn_01x08_Female; footprint (none) -> Connector_PinSocket_2.54mm:PinSocket_1x08_P2.54mm_Vertical
- J5: value (none) -> +/-; footprint (none) -> TerminalBlock_Phoenix:TerminalBlock_Phoenix_MKDS-1,5-2_1x02_P5.00mm_Horizontal
- J6: value (none) -> CONN_02X03; footprint (none) -> Button_Switch_THT:SW_DIP_SPSTx04_Slide_9.78x12.34mm_W7.62mm_P2.54mm
- J7: value (none) -> 0/1; footprint (none) -> TerminalBlock_Phoenix:TerminalBlock_Phoenix_MKDS-1,5-2_1x02_P5.00mm_Horizontal
- J8: value (none) -> 2/3; footprint (none) -> TerminalBlock_Phoenix:TerminalBlock_Phoenix_MKDS-1,5-2_1x02_P5.00mm_Horizontal
- J9: value (none) -> DB9_Female; footprint (none) -> Connector_Dsub:DSUB-9_Female_Horizontal_P2.77x2.84mm_EdgePinOffset4.94mm_Housed_MountingHolesOffset7.48mm
- P1: value (none) -> USB_A; footprint (none) -> Connectors_USB:USB_B_OST_USB-B1HSxx_Horizontal
- P2, P3, P4, P5: value (none) -> Hole; footprint (none) -> MountingHole:MountingHole_3.2mm_M3
- Q1: value (none) -> SI2305; footprint (none) -> TO_SOT_Packages_SMD:SOT-23_Handsoldering
- Q2: value (none) -> AO3407; footprint (none) -> TO_SOT_Packages_SMD:SOT-23_Handsoldering
- R1, R5, R6, R7, R8: value (none) -> 330; footprint (none) -> Resistor_SMD:R_0603_1608Metric_Pad1.05x0.95mm_HandSolder
- R10, R2: value (none) -> 10k; footprint (none) -> Resistor_SMD:R_0603_1608Metric_Pad1.05x0.95mm_HandSolder
- R11, R12, R18: value (none) -> 22; footprint (none) -> Resistor_SMD:R_0603_1608Metric_Pad1.05x0.95mm_HandSolder
- R13: value (none) -> 220k; footprint (none) -> Resistor_SMD:R_0603_1608Metric_Pad1.05x0.95mm_HandSolder
- R14: value (none) -> 56k; footprint (none) -> Resistor_SMD:R_0603_1608Metric_Pad1.05x0.95mm_HandSolder
- R15, R16, R17: value (none) -> 47k; footprint (none) -> Resistor_SMD:R_0603_1608Metric_Pad1.05x0.95mm_HandSolder
- R3, R9: value (none) -> 120; footprint (none) -> Resistor_SMD:R_0603_1608Metric_Pad1.05x0.95mm_HandSolder
- R4: value (none) -> 15k; footprint (none) -> Resistor_SMD:R_0603_1608Metric_Pad1.05x0.95mm_HandSolder
- SW1: value (none) -> SW_DIP_x01; footprint (none) -> Button_Switch_THT:SW_DIP_SPSTx01_Slide_6.7x4.1mm_W7.62mm_P2.54mm_LowProfile
- TP1, TP2: value (none) -> TestPoint; footprint (none) -> Connector_PinHeader_2.54mm:PinHeader_1x01_P2.54mm_Vertical
- U1: value (none) -> ISO1050DUB; footprint (none) -> Package_SO:SOP-8_6.62x9.15mm_P2.54mm
- U2: value (none) -> LM1117-5.0; footprint (none) -> TO_SOT_Packages_SMD:SOT-223-3_TabPin2
- U3: value (none) -> LM1117-3.3; footprint (none) -> TO_SOT_Packages_SMD:SOT-223-3_TabPin2
- U4: value (none) -> MCP2551-I/SN; footprint (none) -> Package_SO:SOIC-8_3.9x4.9mm_P1.27mm
- U5: value (none) -> STM32F072CBTx; footprint (none) -> Package_QFP:LQFP-48_7x7mm_P0.5mm
- U6: value (none) -> MAX3485; footprint (none) -> Package_SO:SO-8_3.9x4.9mm_P1.27mm
