File: F0:F030,F042,F072/Socket_fans/kicad/stm32.kicad_pcb (KiCad board)
At the start: 2 copper layers, 75.5 x 52.5 mm, 89 parts, among them J1 12VIN, J10 Conn_01x02_Female, J2 thermal, J3 Buzzer, J4 cooler3, J5 FAN, J6 FAN, J7 Conn_01x02_Female, J8 MKDS, K1 SRD-12VDC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

Commit message: -> kicad 8
Other:
- net class 0.5 removed
- net class 1 removed
- net class Default removed
