File: F0:F030,F042,F072/canbus/kicad/stm32.kicad_pcb (KiCad board)
At the start: 2 copper layers, 65 x 84 mm, 67 parts, among them J1 CONN_02X03, J2 DB9_Female, J3 DB9_Male, J4 Conn_01x07, J5 12v, J6 Conn_01x01, P12 USART_BOOT, P13 USB_A, P15 Hole, P16 Hole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

Commit message: add/change README files, remove double of Canon management
Other:
- net class 0.5 removed
- net class 1 removed
- net class Default removed
