File: F0:F030,F042,F072/usbcan/kicad_new/stm32.kicad_sch (KiCad schematic)
At the start: 54 parts, among them J10 SDA, J11 PB0, J12 PB1, J13 PB4, J14 PB5, J15 PB2, J16 PB3, J17 GND, J18 GND, J19 +3.3V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

Commit message: fixed bug with usblc6 on usbcan
Parts:
- C1: value (none) -> 47u; footprint (none) -> Capacitor_Tantalum_SMD:CP_EIA-3216-18_Kemet-A_Pad1.58x1.35mm_HandSolder
- C3, C4, C5, C6, C7: value (none) -> 0.1; footprint (none) -> Capacitor_SMD:C_0603_1608Metric_Pad1.05x0.95mm_HandSolder
- C8, C9: value (none) -> 1; footprint (none) -> Capacitor_SMD:C_0805_2012Metric_Pad1.15x1.40mm_HandSolder
- D1: value (none) -> PESD1CAN; footprint (none) -> TO_SOT_Packages_SMD:SOT-23
- D3: value (none) -> LED0; footprint (none) -> LED_SMD:LED_0805_2012Metric_Pad1.15x1.40mm_HandSolder
- D4: value (none) -> LED1; footprint (none) -> LED_SMD:LED_0805_2012Metric_Pad1.15x1.40mm_HandSolder
- J1: value (none) -> Screw_Terminal_01x03; footprint (none) -> TerminalBlock_Phoenix:TerminalBlock_Phoenix_MKDS-1,5-3_1x03_P5.00mm_Horizontal
- J4: value (none) -> USB_B
- P1, P2, P3, P4: value (none) -> Hole; footprint (none) -> my_footprints:Hole_3mm
- Q1: value (none) -> B0505S; footprint (none) -> my_footprints:B0x0xS
- R1: value (none) -> 120; footprint (none) -> Resistor_SMD:R_1210_3225Metric_Pad1.42x2.65mm_HandSolder
- R3, R4, R6: value (none) -> 22; footprint (none) -> Resistor_SMD:R_0603_1608Metric_Pad1.05x0.95mm_HandSolder
- R5: value (none) -> 10k; footprint (none) -> Resistor_SMD:R_0603_1608Metric_Pad1.05x0.95mm_HandSolder
- R7, R8: value (none) -> 330; footprint (none) -> Resistor_SMD:R_0603_1608Metric_Pad1.05x0.95mm_HandSolder
- SW1: value (none) -> SW_DIP_x01; footprint (none) -> Button_Switch_THT:SW_DIP_SPSTx01_Slide_6.7x4.1mm_W7.62mm_P2.54mm_LowProfile
- U1: value (none) -> LM1117-3.3; footprint (none) -> TO_SOT_Packages_SMD:SOT-223-3_TabPin2
- U3: value (none) -> STM32F072C8Tx; footprint (none) -> Package_QFP:LQFP-48_7x7mm_P0.5mm
- U4: value (none) -> ISO1050DUB; footprint (none) -> Package_SO:SOP-8_6.62x9.15mm_P2.54mm
Connections:
- net +5V: now also U2.5 (VBUS); no longer U2.2 (GND)
- net GND: now also U2.2 (GND); no longer U2.5 (VBUS)
- net at R3.2: now also U2.4 (I/O2); no longer U2.1 (I/O1)
- net at R4.2: now also U2.6 (I/O1); no longer U2.3 (I/O2)
- net at U3.32 (PA11): now also U2.3 (I/O2); no longer U2.6 (I/O1)
- net at U3.33 (PA12): now also U2.1 (I/O1); no longer U2.4 (I/O2)
Other:
- moved on the sheet: U2
