File: F1:F103/CAR_CANbus/Lamps/kicad/l_pwrx.kicad_sch (KiCad schematic)
At the start: 7 parts, among them J7 Lamp, Q3 AO3407, Q3 IRLR7807

Commit message: start drawing PCB
Parts:
- removed D1: 1N5819, Diode_SMD:D_SOD-323_HandSoldering, symbol Device:D_Schottky
- added D6: MM3Z3V3, Diode_SMD:D_0805_2012Metric_Pad1.15x1.40mm_HandSolder, symbol Device:D_Schottky
Connections:
- net GND: now also D6.2 (A)
- net L_ctrl: now also D6.1 (K)
Other:
- moved on the sheet: Q3
Changed lines of the file:
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@@
     (stroke (width 0) (type default))
   )
-  (wire (pts (xy 103.759 45.085) (xy 101.346 45.085))
+  (wire (pts (xy 105.156 45.085) (xy 101.346 45.085))
     (stroke (width 0) (type default))
   )
@@
     (stroke (width 0) (type default))
   )
+  (wire (pts (xy 105.156 45.593) (xy 105.156 45.085))
+    (stroke (width 0) (type default))
+  )
   (wire (pts (xy 91.948 38.481) (xy 91.948 45.085))
     (stroke (width 0) (type default))
@@
     (effects (font (size 1.27 1.27)) (justify left bottom))
   )
-  (label "g" (at 100.9869 59.533 0) (fields_autoplaced)
-    (effects (font (size 1.27 1.27)) (justify left bottom))
-  )
-  (label "d" (at 108.6069 54.453 0) (fields_autoplaced)
+  (label "g" (at 84.582 70.739 0) (fields_autoplaced)
+    (effects (font (size 1.27 1.27)) (justify left bottom))
+  )
+  (label "d" (at 92.202 65.659 0) (fields_autoplaced)
     (effects (font (size 1.27 1.27)) (justify left bottom))
   )
@@
     (effects (font (size 1.27 1.27)) (justify left bottom))
   )
-  (label "s" (at 108.6069 64.613 0) (fields_autoplaced)
+  (label "s" (at 92.202 75.819 0) (fields_autoplaced)
     (effects (font (size 1.27 1.27)) (justify left bottom))
   )
@@
     (effects (font (size 1.27 1.27)) (justify left bottom))
   )
-  (hierarchical_label "L_ctrl" (shape input) (at 103.759 45.085 0) (fields_autoplaced)
+  (hierarchical_label "L_ctrl" (shape input) (at 105.156 45.085 0) (fields_autoplaced)
     (effects (font (size 1.27 1.27)) (justify left))
   )
@@
     )
   )
+  (symbol (lib_id "Device:D_Schottky") (at 105.156 49.403 270) (unit 1)
+    (in_bom yes) (on_board yes) (dnp no)
+    (property "Reference" "D6" (at 99.568 48.895 90)
+      (effects (font (size 1.27 1.27)) (justify left))
+    )
+    (property "Value" "MM3Z3V3" (at 107.569 46.101 0)
+      (effects (font (size 1.27 1.27)) (justify left))
+    )
+    (property "Footprint" "Diode_SMD:D_0805_2012Metric_Pad1.15x1.40mm_HandSolder" (at 105.156 49.403 0)
+      (effects (font (size 1.27 1.27)) hide)
+    )
+    (property "Datasheet" "~" (at 105.156 49.403 0)
+      (effects (font (size 1.27 1.27)) hide)
+    )
+    (pin "1")
+    (pin "2")
+    (instances
+      (project "lamps"
+        (path "/07322d58-7316-46ef-93d7-29583fc10978"
+          (reference "D6") (unit 1)
+        )
+        (path "/07322d58-7316-46ef-93d7-29583fc10978/e499c186-84d3-4658-851e-01ff2d40285a"
+          (reference "D15") (unit 1)
+        )
+        (path "/07322d58-7316-46ef-93d7-29583fc10978/e4a98edc-e978-4b46-ab0b-6c6f5adb40be"
+          (reference "D16") (unit 1)
+        )
+        (path "/07322d58-7316-46ef-93d7-29583fc10978/264a78a9-8249-49c8-9703-a17561438e73"
+          (reference "D17") (unit 1)
+        )
+        (path "/07322d58-7316-46ef-93d7-29583fc10978/ab52cd37-c768-42ac-8c95-dd263c06daeb"
+          (reference "D18") (unit 1)
+        )
+        (path "/07322d58-7316-46ef-93d7-29583fc10978/0a99fa1e-868d-4243-8826-7d76aec82a59"
+          (reference "D10") (unit 1)
+        )
+        (path "/07322d58-7316-46ef-93d7-29583fc10978/7e358dbb-44bb-46fa-96a3-0079855a61ff"
+          (reference "D14") (unit 1)
+        )
+      )
+    )
+  )
   (symbol (lib_id "Device:R") (at 88.138 55.88 270) (unit 1)
     (in_bom yes) (on_board yes) (dnp no)
@@
     )
   )
-  (symbol (lib_id "power:+3V3") (at 103.759 37.465 0) (unit 1)
-    (in_bom yes) (on_board yes) (dnp no) (fields_autoplaced)
-    (property "Reference" "#PWR024" (at 103.759 41.275 0)
-      (effects (font (size 1.27 1.27)) hide)
-    )
-    (property "Value" "+3V3" (at 103.759 33.52 0)
-      (effects (font (size 1.27 1.27)))
-    )
-    (property "Footprint" "" (at 103.759 37.465 0)
-      (effects (font (size 1.27 1.27)) hide)
-    )
-    (property "Datasheet" "" (at 103.759 37.465 0)
-      (effects (font (size 1.27 1.27)) hide)
-    )
-    (pin "1")
-    (instances
-      (project "lamps"
-        (path "/07322d58-7316-46ef-93d7-29583fc10978"
-          (reference "#PWR024") (unit 1)
-        )
-        (path "/07322d58-7316-46ef-93d7-29583fc10978/e499c186-84d3-4658-851e-01ff2d40285a"
-          (reference "#PWR011") (unit 1)
-        )
-        (path "/07322d58-7316-46ef-93d7-29583fc10978/0a99fa1e-868d-4243-8826-7d76aec82a59"
-          (reference "#PWR033") (unit 1)
-        )
-        (path "/07322d58-7316-46ef-93d7-29583fc10978/7e358dbb-44bb-46fa-96a3-0079855a61ff"
-          (reference "#PWR041") (unit 1)
-        )
-      )
-    )
-  )
   (symbol (lib_id "Device:R") (at 97.536 45.085 270) (unit 1)
     (in_bom yes) (on_board yes) (dnp no)
@@
     )
   )
-  (symbol (lib_id "Device:Q_NMOS_GSD") (at 106.0669 59.533 0) (unit 1)
-    (in_bom yes) (on_board yes) (dnp no) (fields_autoplaced)
-    (property "Reference" "Q3" (at 111.2739 58.509 0)
-      (effects (font (size 1.27 1.27)) (justify left))
-    )
-    (property "Value" "AO3407" (at 111.2739 60.557 0)
-      (effects (font (size 1.27 1.27)) (justify left))
-    )
-    (property "Footprint" "Package_TO_SOT_SMD:SOT-23_Handsoldering" (at 111.1469 56.993 0)
-      (effects (font (size 1.27 1.27)) hide)
-    )
-    (property "Datasheet" "~" (at 106.0669 59.533 0)
+  (symbol (lib_id "Device:Q_NMOS_GSD") (at 89.662 70.739 0) (unit 1)
+    (in_bom yes) (on_board yes) (dnp no)
+    (property "Reference" "Q3" (at 94.869 69.715 0)
+      (effects (font (size 1.27 1.27)) (justify left))
+    )
+    (property "Value" "AO3407" (at 94.869 71.763 0)
+      (effects (font (size 1.27 1.27)) (justify left))
+    )
+    (property "Footprint" "Package_TO_SOT_SMD:SOT-23_Handsoldering" (at 94.742 68.199 0)
+      (effects (font (size 1.27 1.27)) hide)
+    )
+    (property "Datasheet" "~" (at 89.662 70.739 0)
       (effects (font (size 1.27 1.27)) hide)
     )
@@
         (path "/07322d58-7316-46ef-93d7-29583fc10978/7e358dbb-44bb-46fa-96a3-0079855a61ff"
           (reference "Q8") (unit 1)
+        )
+      )
+    )
+  )
+  (symbol (lib_name "GND_3") (lib_id "power:GND") (at 105.156 53.213 0) (mirror y) (unit 1)
+    (in_bom yes) (on_board yes) (dnp no)
+    (property "Reference" "#PWR032" (at 105.156 59.563 0)
+      (effects (font (size 1.27 1.27)) hide)
+    )
+    (property "Value" "GND" (at 105.156 57.158 0)
+      (effects (font (size 1.27 1.27)) hide)
+    )
+    (property "Footprint" "" (at 105.156 53.213 0)
+      (effects (font (size 1.27 1.27)) hide)
+    )
+    (property "Datasheet" "" (at 105.156 53.213 0)
+      (effects (font (size 1.27 1.27)) hide)
+    )
+    (pin "1")
+    (instances
+      (project "lamps"
+        (path "/07322d58-7316-46ef-93d7-29583fc10978"
+          (reference "#PWR032") (unit 1)
+        )
+        (path "/07322d58-7316-46ef-93d7-29583fc10978/e499c186-84d3-4658-851e-01ff2d40285a"
+          (reference "#PWR010") (unit 1)
+        )
+        (path "/07322d58-7316-46ef-93d7-29583fc10978/0a99fa1e-868d-4243-8826-7d76aec82a59"
+          (reference "#PWR033") (unit 1)
+        )
+        (path "/07322d58-7316-46ef-93d7-29583fc10978/7e358dbb-44bb-46fa-96a3-0079855a61ff"
+          (reference "#PWR041") (unit 1)
         )
       )
@@
         )
       )
-    )
-  )
-  (symbol (lib_id "Device:D_Schottky") (at 103.759 41.275 270) (unit 1)
-    (in_bom yes) (on_board yes) (dnp no) (fields_autoplaced)
-    (property "Reference" "D1" (at 105.791 39.9335 90)
-      (effects (font (size 1.27 1.27)) (justify left))
-    )
-    (property "Value" "1N5819" (at 105.791 41.9815 90)
-      (effects (font (size 1.27 1.27)) (justify left))
-    )
-    (property "Footprint" "Diode_SMD:D_SOD-323_HandSoldering" (at 103.759 41.275 0)
-      (effects (font (size 1.27 1.27)) hide)
-    )
-    (property "Datasheet" "~" (at 103.759 41.275 0)
-      (effects (font (size 1.27 1.27)) hide)
-    )
-    (pin "1")
-    (pin "2")
-    (instances
-      (project "lamps"
-        (path "/07322d58-7316-46ef-93d7-29583fc10978"
-          (reference "D1") (unit 1)
-        )
-        (path "/07322d58-7316-46ef-93d7-29583fc10978/e499c186-84d3-4658-851e-01ff2d40285a"
-          (reference "D1") (unit 1)
-        )
-        (path "/07322d58-7316-46ef-93d7-29583fc10978/0a99fa1e-868d-4243-8826-7d76aec82a59"
-          (reference "D10") (unit 1)
-        )
-        (path "/07322d58-7316-46ef-93d7-29583fc10978/7e358dbb-44bb-46fa-96a3-0079855a61ff"
-          (reference "D14") (unit 1)
-        )
-      )

Commit message: finished PCB
Parts:
- removed J7: Lamp, TerminalBlock_Phoenix:TerminalBlock_Phoenix_MKDS-1,5-2_1x02_P5.00mm_Horizontal, symbol Connector:Screw_Terminal_01x02
Connections:
- net d renamed L_minus
Changed lines of the file:
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@@
 (kicad_sch (version 20230121) (generator eeschema)
   (paper "A4")
-  (junction (at 91.948 45.085) (diameter 0) (color 0 0 0 0)
-  )
   (junction (at 91.948 55.88) (diameter 0) (color 0 0 0 0)
   )
@@
     (stroke (width 0) (type default))
   )
-  (wire (pts (xy 91.948 38.481) (xy 91.948 45.085))
-    (stroke (width 0) (type default))
-  )
-  (wire (pts (xy 92.075 38.481) (xy 91.948 38.481))
-    (stroke (width 0) (type default))
-  )
   (text "Solder one of MOSFETs" (at 84.963 29.337 0)
     (effects (font (size 1.27 1.27)) (justify left bottom))
@@
     (effects (font (size 1.27 1.27)) (justify left bottom))
   )
-  (label "d" (at 91.948 44.958 0) (fields_autoplaced)
+  (label "d" (at 92.3121 45.085 0) (fields_autoplaced)
     (effects (font (size 1.27 1.27)) (justify left bottom))
   )
@@
     (effects (font (size 1.27 1.27)) (justify left))
   )
-  (hierarchical_label "Pwr" (shape input) (at 92.075 35.941 180) (fields_autoplaced)
+  (hierarchical_label "L_minus" (shape input) (at 91.948 45.6549 180) (fields_autoplaced)
     (effects (font (size 1.27 1.27)) (justify right))
   )
@@
     (effects (font (size 1.27 1.27)) (justify right))
   )
-  (symbol (lib_id "Connector:Screw_Terminal_01x02") (at 97.155 35.941 0) (unit 1)
-    (in_bom yes) (on_board yes) (dnp no)
-    (property "Reference" "J7" (at 99.568 35.687 90)
-      (effects (font (size 1.27 1.27)))
-    )
-    (property "Value" "Lamp" (at 99.187 38.4556 0)
-      (effects (font (size 1.27 1.27)) (justify left) hide)
-    )
-    (property "Footprint" "TerminalBlock_Phoenix:TerminalBlock_Phoenix_MKDS-1,5-2_1x02_P5.00mm_Horizontal" (at 97.155 35.941 0)
-      (effects (font (size 1.27 1.27)) hide)
-    )
-    (property "Datasheet" "~" (at 97.155 35.941 0)
-      (effects (font (size 1.27 1.27)) hide)
-    )
-    (pin "1")
-    (pin "2")
-    (instances
-      (project "lamps"
-        (path "/07322d58-7316-46ef-93d7-29583fc10978"
-          (reference "J7") (unit 1)
-        )
-        (path "/07322d58-7316-46ef-93d7-29583fc10978/e499c186-84d3-4658-851e-01ff2d40285a"
-          (reference "J2") (unit 1)
-        )
-        (path "/07322d58-7316-46ef-93d7-29583fc10978/0a99fa1e-868d-4243-8826-7d76aec82a59"
-          (reference "J7") (unit 1)
-        )
-        (path "/07322d58-7316-46ef-93d7-29583fc10978/7e358dbb-44bb-46fa-96a3-0079855a61ff"
-          (reference "J11") (unit 1)
-        )
-      )
-      (project "stm32"
-        (path "/f40cbe7e-cd25-45e5-a6cb-d92457495048"
-          (reference "J12") (unit 1)
-        )
-      )
-    )
-  )
   (symbol (lib_name "GND_3") (lib_id "power:GND") (at 91.948 55.88 0) (mirror y) (unit 1)

Commit message: -> kicad 8
Parts:
- renumbered D6 to D10, Q3 to Q2, R16 to R11, R26 to R12, R26 to R13
