File: F1:F103/CAR_CANbus/Lamps/kicad/lamps.kicad_pcb (KiCad board)
At the start: 2 copper layers, 100 x 100 mm, 84 parts, among them J1 Power, J10 Lamp, J11 Lamp, J2 UART, J3 Prog, J4 CAN, J5 ESW, J6 Lamp, J7 Lamp, J8 Lamp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

Commit message: continue
Parts:
- removed TP1, TP2, TP3: Gnd, TestPoint:TestPoint_Loop_D1.80mm_Drill1.0mm_Beaded
- removed TP4: 12V, TestPoint:TestPoint_Loop_D1.80mm_Drill1.0mm_Beaded
- removed TP5: 5V, TestPoint:TestPoint_Loop_D1.80mm_Drill1.0mm_Beaded
- removed TP6: 3V3, TestPoint:TestPoint_Loop_D1.80mm_Drill1.0mm_Beaded
- C1, C2, C3, C6, D1, D12, D14, D2, JP1, L1, Q5, Q7, R17, R18, R19, R25, R3, R4, R7, U2, U4: moved to B.Cu
- moved Q7 244.1 mm to (92.6, 96.7), turned to 180 degrees
- moved J11 240.2 mm to (85.2, 101.8), turned to 90 degrees
- moved D14 238.1 mm to (100.9, 100.7), turned to 180 degrees
- moved R25 236.5 mm to (101.0, 96.7), turned to 180 degrees
- moved R18 232.8 mm to (94.1, 89.0)
- moved Q5 231.2 mm to (89.5, 88.0), turned to 180 degrees
- moved R17 230.5 mm to (94.4, 85.7), turned to 180 degrees
- moved J7 229.6 mm to (150.6, 33.4)
- moved D10 229.6 mm to (141.8, 23.0)
- moved Q2 229.6 mm to (173.1, 33.8)
- moved Q3 229.6 mm to (156.0, 45.0)
- moved R12 229.6 mm to (143.2, 39.1)
- moved R13 229.6 mm to (150.2, 21.8)
- moved R11 229.6 mm to (162.3, 23.5)
- moved J9 226.8 mm to (85.2, 90.2), turned to 90 degrees
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Connections:
- D11 pad 1: /adc1 -> /adc5
- D12 pad 1: /adc2 -> /adc0
- D14 pad 1: /adc5 -> /adc1
- D9 pad 1: /adc0 -> /adc2
- R10 pad 1: /adc0 -> /adc2
- R11 pad 1: /T2_Ch3 -> /T2_Ch4
- R12 pad 2: /T2_Ch3 -> /T2_Ch4
- R16 pad 1: /adc1 -> /adc5
- R19 pad 1: /adc2 -> /adc0
- R23 pad 1: /T2_Ch4 -> /T2_Ch3
- R24 pad 2: /T2_Ch4 -> /T2_Ch3
- R25 pad 1: /adc5 -> /adc1
Routing:
- net GND: track 16.3 -> 201.2 mm, vias 0 -> 9
- net +12V: track 0.00 -> 62.0 mm, vias 0 -> 1
- net /HOT@Always: track 0.00 -> 61.2 mm
- net +5V: track 0.00 -> 59.8 mm, vias 0 -> 3
- net /adc1: track 2.03 -> 40.0 mm, vias 0 -> 1
- net /T3_Ch3: track 0.00 -> 35.7 mm, vias 0 -> 1
- net /T2_Ch3: track 0.00 -> 33.7 mm
- net /adc0: track 2.86 -> 34.1 mm, vias 0 -> 1
- net /L_pwrX1/d: track 0.00 -> 22.7 mm, vias 0 -> 1
- net /CANL: track 0.00 -> 20.8 mm
- net +3V3: track 36.4 -> 55.8 mm
- net Net-(U2-FB): track 0.00 -> 16.2 mm
- net /CANH: track 0.00 -> 13.4 mm
- net /VEN: track 0.00 -> 8.52 mm, vias 0 -> 1
- net /CAN_Rx: track 4.16 -> 12.2 mm
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
Commit message: finished PCB
Parts:
- D10, D11, D13, Q2, Q4, R13, R14, R16, R22: moved to B.Cu
- D14, R25: moved to F.Cu
- J6, J7: value Lamp -> ACC
- J8: value Lamp -> Reserved
- moved J6 137.0 mm to (71.5, 63.8)
- moved R9 125.5 mm to (85.3, 76.2)
- moved R8 123.1 mm to (85.2, 78.0), turned to 180 degrees
- moved D9 122.0 mm to (87.8, 81.2), turned to 90 degrees
- moved R10 121.1 mm to (86.9, 84.0), turned to 180 degrees
- moved Q1 120.8 mm to (83.3, 82.5), turned to -90 degrees
- moved J10 108.5 mm to (128.2, 84.0), turned to -90 degrees
- moved R22 101.3 mm to (109.8, 91.7), turned to -90 degrees
- moved R20 99.2 mm to (110.8, 86.5), turned to -90 degrees
- moved D13 98.8 mm to (110.8, 88.9)
- moved R21 95.2 mm to (112.4, 86.5), turned to 90 degrees
- moved J7 87.9 mm to (74.2, 77.0), turned to 90 degrees
- moved Q6 85.7 mm to (109.8, 91.0), turned to -90 degrees
- moved J8 79.0 mm to (74.2, 89.0), turned to 90 degrees
- moved R11 73.1 mm to (118.0, 81.7), turned to -90 degrees
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Connections:
- D10 pad 1: /adc4 -> /adc5
- D11 pad 1: /adc5 -> /adc2
- D12 pad 1: /adc0 -> /adc1
- D14 pad 1: /adc1 -> /adc4
- D9 pad 1: /adc2 -> /adc0
- J10 pad 1: /HOT@Always -> /L5
- J10 pad 2: Net-(J10-Pin_2) -> /L6
- J11 pad 1: /HOT@Always -> /L4
- J11 pad 2: /L_pwrX1/d -> /L3
- J6 pad 1: +12V -> /HOT@Always
- J6 pad 2: Net-(J6-Pin_2) -> /HOT@Always
- J7 pad 2: /L_pwrX/d -> /HOT@Always
- J8 pad 2: Net-(J8-Pin_2) -> +12V
- J9 pad 1: /HOT@Always -> /L2
- J9 pad 2: Net-(J9-Pin_2) -> /L1
- Q1 pad 3: Net-(J6-Pin_2) -> /L1
- Q2 pad 2: /L_pwrX/d -> /L5
- Q3 pad 3: /L_pwrX/d -> /L5
- Q4 pad 3: Net-(J8-Pin_2) -> /L3
- Q5 pad 3: Net-(J9-Pin_2) -> /L2
- Q6 pad 3: Net-(J10-Pin_2) -> /L4
- Q7 pad 2: /L_pwrX1/d -> /L6
- Q8 pad 3: /L_pwrX1/d -> /L6
- R10 pad 1: /adc2 -> /adc0
- R10 pad 2: Net-(J6-Pin_2) -> /L1
- R13 pad 1: /adc4 -> /adc5
- R13 pad 2: /L_pwrX/d -> /L5
- R14 pad 1: /T3_Ch2 -> /T3_Ch3
- R15 pad 2: /T3_Ch2 -> /T3_Ch3
- R16 pad 1: /adc5 -> /adc2
- R16 pad 2: Net-(J8-Pin_2) -> /L3
- R17 pad 1: /T3_Ch3 -> /T3_Ch2
- R18 pad 2: /T3_Ch3 -> /T3_Ch2
- R19 pad 1: /adc0 -> /adc1
- R19 pad 2: Net-(J9-Pin_2) -> /L2
- R22 pad 2: Net-(J10-Pin_2) -> /L4
- R25 pad 1: /adc1 -> /adc4
- R25 pad 2: /L_pwrX1/d -> /L6
- U3 pad 16: unconnected-(U3-PA6-Pad16) -> /T3_Ch1
- U3 pad 17: unconnected-(U3-PA7-Pad17) -> /T3_Ch2
Routing:
- net GND: track 201.2 -> 404.4 mm, vias 9 -> 13
- net /T3_Ch1: track 0.00 -> 38.8 mm, vias 0 -> 2
- net /HOT@Always: track 61.2 -> 25.5 mm
- net /T3_Ch2: track 0.00 -> 34.9 mm, vias 0 -> 1
- net +12V: track 62.0 -> 94.0 mm
- net /L6: track 0.00 -> 29.8 mm, vias 0 -> 1
- net /adc2: track 0.00 -> 23.7 mm, vias 0 -> 1
- net /L_pwrX1/d: track 22.7 -> 0.00 mm, vias 1 -> 0
- net /adc4: track 0.00 -> 21.5 mm, vias 0 -> 2
- net /adc3: track 0.00 -> 20.6 mm, vias 0 -> 1
- net /L5: track 0.00 -> 18.7 mm, vias 0 -> 1
- net /T3_Ch4: track 2.10 -> 16.3 mm, vias 1 -> 0
- net /L1: track 0.00 -> 11.2 mm, vias 0 -> 1
- net /T3_Ch3: track 35.7 -> 24.9 mm
- net /T2_Ch4: track 0.00 -> 10.7 mm
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- added copper zone on B.Cu, net GND
- added copper zone on F.Cu, net GND
Other:
- board size 100 x 100 mm -> 65.5 x 41 mm
