File: testboard/F0_F1_F3-LQFP48_testboard/stm32.kicad_sch (KiCad schematic)
At the start: 54 parts

Commit message: save under new kicad
Parts:
- C1, C10, C2, C3, C7, C8, C9: value (none) -> 0.1; footprint (none) -> Capacitor_SMD:C_0603_1608Metric_Pad1.05x0.95mm_HandSolder
- C4: value (none) -> 47u; footprint (none) -> Capacitor_Tantalum_SMD:CP_EIA-6032-28_Kemet-C_Pad2.25x2.35mm_HandSolder
- C5, C6: value (none) -> 12; footprint (none) -> Capacitor_SMD:C_0603_1608Metric_Pad1.05x0.95mm_HandSolder
- D1, D2, D3, D4, D5, D6: value (none) -> LED; footprint (none) -> LED_THT:LED_D3.0mm
- J1, J11, J5, J6, J7, J8, J9: value (none) -> Conn_01x04_Female; footprint (none) -> Connector_PinSocket_2.54mm:PinSocket_1x04_P2.54mm_Vertical
- J10, J12, J2, J4: value (none) -> Conn_01x01_Female; footprint (none) -> Connector_PinSocket_2.54mm:PinSocket_1x01_P2.54mm_Vertical
- J3: value (none) -> Conn_01x02_Female; footprint (none) -> Connector_PinSocket_2.54mm:PinSocket_1x02_P2.54mm_Vertical
- P1: value (none) -> USART1; footprint (none) -> Connector_PinSocket_2.54mm:PinSocket_1x03_P2.54mm_Vertical
- P2: value (none) -> USART2/3; footprint (none) -> Connector_PinSocket_2.54mm:PinSocket_1x03_P2.54mm_Vertical
- P3: value (none) -> USB_B; footprint (none) -> Connector_USB:USB_B_OST_USB-B1HSxx_Horizontal
- Q1: value (none) -> DTA114Y; footprint (none) -> Package_TO_SOT_SMD:SOT-323_SC-70_Handsoldering
- R1, R14, R15, R2: value (none) -> 4k7; footprint (none) -> Resistor_SMD:R_0805_2012Metric_Pad1.15x1.40mm_HandSolder
- R10, R11, R6, R7, R8, R9: value (none) -> 220; footprint (none) -> Resistor_SMD:R_0805_2012Metric_Pad1.15x1.40mm_HandSolder
- R12, R13: value (none) -> 22; footprint (none) -> Resistor_SMD:R_0603_1608Metric_Pad1.05x0.95mm_HandSolder
- R16: value (none) -> 1k5; footprint (none) -> Resistor_SMD:R_0603_1608Metric_Pad1.05x0.95mm_HandSolder
- R3: value (none) -> 10k; footprint (none) -> Resistor_SMD:R_0603_1608Metric_Pad1.05x0.95mm_HandSolder
- R5: value (none) -> 100k; footprint (none) -> Resistor_SMD:R_0603_1608Metric_Pad1.05x0.95mm_HandSolder
- SW1: value (none) -> Reset; footprint (none) -> Button_Switch_THT:SW_PUSH_6mm
- SW2: value (none) -> Boot; footprint (none) -> Button_Switch_THT:SW_PUSH_6mm
- U1: value (none) -> LM1117-3.3; footprint (none) -> Package_TO_SOT_SMD:SOT-223
- U2: value (none) -> STM32LQFP48; footprint (none) -> Package_DIP:DIP-48_W15.24mm_Socket_LongPads
- U3: value (none) -> USBLC6-2SC6; footprint (none) -> Package_TO_SOT_SMD:SOT-23-6_Handsoldering
- Y1: value (none) -> 8MHz; footprint (none) -> Crystal:Crystal_HC49-U_Vertical
