File: F1:F103/shutter/UNISTABLE/kicad/shutter.kicad_pcb (KiCad board)
At the start: 2 copper layers, 61 x 42.5 mm, 49 parts, among them J1 ccd, J10 shutter, J11 USB_B, J2 hall, J3 ShtrPower, J4 SWD, J5 5Vext, J6 5v, J7 GND, J8 3v3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

Commit message: Unistable shutter
Routing:
- net GND: track 285.1 -> 286.8 mm
