File: F1:F103/Hall_linear/kicad/Hall.kicad_pcb (KiCad board)
At the start: 2 copper layers, 45.3 x 46.8 mm, 35 parts, among them J1 SWD, J2 5v, J3 Sensor, J4 GND, J5 3v3, J6 USB_C_Receptacle_USB2.0_16P, Q1 DTA114Y, U1 STM32F103C6Tx, U2 LM1117-3.3, U3 USBLC6-2SC6, U4 MCP2551-I-SN, Y1 NX5032GA-8MHz

Commit message: fixed PCB, add pre-alpha code
Parts:
- removed JP1: CANbus, Jumper:SolderJumper-2_P1.3mm_Open_TrianglePad1.0x1.5mm
- added D1: SS14, Diode_SMD:D_SOD-323_HandSoldering, F.Cu at (64.3, 41.6)
- added R2: 10k, Resistor_SMD:R_0603_1608Metric_Pad0.98x0.95mm_HandSolder, F.Cu at (64.3, 45.6)
- added R3: 10k, Resistor_SMD:R_0603_1608Metric_Pad0.98x0.95mm_HandSolder, F.Cu at (66.2, 45.6)
- moved C3 6.61 mm to (64.6, 56.7)
- moved J2 0.82 mm to (63.6, 61.5)
- moved J5 0.25 mm to (65.4, 28.3)
- moved R8 0.23 mm to (86.5, 61.3)
- renumbered D1 to D2, D2 to D3, R9 to R10, R3 to R4, R4 to R5, R5 to R6, R6 to R7, R7 to R8, R8 to R9
Connections:
- U1 pad 13: Net-(JP1-B) -> unconnected-(U1-PA3-Pad13)
- U1 pad 17: /ADCin -> Net-(D1-A)
Routing:
- net GND: track 281.1 -> 403.7 mm, vias 12 -> 21
- net Net-(D1-A): track 0.00 -> 6.63 mm
- net Net-(JP1-B): track 6.32 -> 0.00 mm
- net /ADCin: track 7.19 -> 2.76 mm
- net /CANL: track 37.3 -> 34.7 mm
- net +3V3: track 85.9 -> 88.3 mm
- net /VBUS: track 91.2 -> 93.5 mm
- net /CANH: track 39.6 -> 38.4 mm, vias 3 -> 2
Other:
- board text removed: "Solder this for CAN instead of USB"
