File: F1:F103/Hall_linear/kicad/Hall.kicad_sch (KiCad schematic)
At the start: 35 parts, among them J1 SWD, J2 5v, J3 Sensor, J4 GND, J5 3v3, J6 USB_C_Receptacle_USB2.0_16P, Q1 DTA114Y, U1 STM32F103C6Tx, U2 LM1117-3.3, U3 USBLC6-2SC6, U4 MCP2551-I-SN, Y1 NX5032GA-8MHz

Commit message: fixed PCB, add pre-alpha code
Parts:
- removed JP1: CANbus, Jumper:SolderJumper-2_P1.3mm_Open_TrianglePad1.0x1.5mm, symbol Jumper:SolderJumper_2_Bridged
- added D1: SS14, Diode_SMD:D_SOD-323_HandSoldering, symbol Diode:SS14
- added R2, R3: 10k, Resistor_SMD:R_0603_1608Metric_Pad0.98x0.95mm_HandSolder, symbol Device:R
- renumbered D1 to D2, D2 to D3, R9 to R10, R3 to R4, R4 to R5, R5 to R6, R6 to R7, R7 to R8, R8 to R9
Connections:
- net +3V3: now also D1.1 (K)
- net ADCin: now also R2.1; no longer U1.17 (PA7)
- net GND: now also R3.2
- new net: D1.2 (A), R2.2, R3.1, U1.17 (PA7)
- no-connect marks 27 -> 28
Other:
- moved on the sheet: C1, C2, J1, R1, U1, Y1
