File: F3:F303/InterfaceBoard/kicad/iso485.kicad_sch (KiCad schematic)
At the start: 7 parts, among them J9 Term_3, Q3 B0505S-1W, U5 ISO3088DW

Commit message: finish, add gerbers
Parts:
- renumbered C15 to C26, C16 to C31, D4 to D11, F2 to F5, J9 to J13, Q3 to Q6, U5 to U8
Changed lines of the file:
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@@
 			)
 		)
-		(property "Reference" "Q3"
+		(property "Reference" "Q6"
 			(at 87.63 32.004 0)
 			(effects
@@
 			(project "many485"
 				(path "/8d999898-5824-4200-a5bb-e5cd72e34b91/b5d3972e-2956-484f-8514-69dcc9a48328"
-					(reference "Q3")
+					(reference "Q6")
 					(unit 1)
 				)
@@
 				)
 				(path "/8d999898-5824-4200-a5bb-e5cd72e34b91/fffbe808-9aec-4c0c-a1ae-7f856729924e"
-					(reference "Q4")
+					(reference "Q7")
 					(unit 1)
 				)
@@
 			)
 		)
-		(property "Reference" "J9"
+		(property "Reference" "J13"
 			(at 112.522 54.737 0)
 			(hide yes)
@@
 			(project "many485"
 				(path "/8d999898-5824-4200-a5bb-e5cd72e34b91/b5d3972e-2956-484f-8514-69dcc9a48328"
-					(reference "J9")
-					(unit 1)
-				)
-				(path "/8d999898-5824-4200-a5bb-e5cd72e34b91/bfb47038-e30b-4456-8a3f-910a2a85c045"
-					(reference "J11")
-					(unit 1)
-				)
-				(path "/8d999898-5824-4200-a5bb-e5cd72e34b91/fffbe808-9aec-4c0c-a1ae-7f856729924e"
-					(reference "J10")
+					(reference "J13")
+					(unit 1)
+				)
+				(path "/8d999898-5824-4200-a5bb-e5cd72e34b91/bfb47038-e30b-4456-8a3f-910a2a85c045"
+					(reference "J12")
+					(unit 1)
+				)
+				(path "/8d999898-5824-4200-a5bb-e5cd72e34b91/fffbe808-9aec-4c0c-a1ae-7f856729924e"
+					(reference "J14")
 					(unit 1)
 				)
@@
 			)
 		)
-		(property "Reference" "D4"
+		(property "Reference" "D11"
 			(at 106.68 68.9059 0)
 			(effects
@@
 			(project "many485"
 				(path "/8d999898-5824-4200-a5bb-e5cd72e34b91/b5d3972e-2956-484f-8514-69dcc9a48328"
-					(reference "D4")
-					(unit 1)
-				)
-				(path "/8d999898-5824-4200-a5bb-e5cd72e34b91/bfb47038-e30b-4456-8a3f-910a2a85c045"
-					(reference "D6")
-					(unit 1)
-				)
-				(path "/8d999898-5824-4200-a5bb-e5cd72e34b91/fffbe808-9aec-4c0c-a1ae-7f856729924e"
-					(reference "D5")
+					(reference "D11")
+					(unit 1)
+				)
+				(path "/8d999898-5824-4200-a5bb-e5cd72e34b91/bfb47038-e30b-4456-8a3f-910a2a85c045"
+					(reference "D12")
+					(unit 1)
+				)
+				(path "/8d999898-5824-4200-a5bb-e5cd72e34b91/fffbe808-9aec-4c0c-a1ae-7f856729924e"
+					(reference "D10")
 					(unit 1)
 				)
@@
 			)
 		)
-		(property "Reference" "C15"
+		(property "Reference" "C26"
 			(at 71.882 42.926 90)
 			(effects
@@
 			(project "many485"
 				(path "/8d999898-5824-4200-a5bb-e5cd72e34b91/b5d3972e-2956-484f-8514-69dcc9a48328"
-					(reference "C15")
-					(unit 1)
-				)
-				(path "/8d999898-5824-4200-a5bb-e5cd72e34b91/bfb47038-e30b-4456-8a3f-910a2a85c045"
-					(reference "C19")
-					(unit 1)
-				)
-				(path "/8d999898-5824-4200-a5bb-e5cd72e34b91/fffbe808-9aec-4c0c-a1ae-7f856729924e"
-					(reference "C17")
+					(reference "C26")
+					(unit 1)
+				)
+				(path "/8d999898-5824-4200-a5bb-e5cd72e34b91/bfb47038-e30b-4456-8a3f-910a2a85c045"
+					(reference "C27")
+					(unit 1)
+				)
+				(path "/8d999898-5824-4200-a5bb-e5cd72e34b91/fffbe808-9aec-4c0c-a1ae-7f856729924e"
+					(reference "C25")
 					(unit 1)
 				)
@@
 			)
 		)
-		(property "Reference" "C16"
+		(property "Reference" "C31"
 			(at 92.71 42.672 90)
 			(effects
@@
 			(project "many485"
 				(path "/8d999898-5824-4200-a5bb-e5cd72e34b91/b5d3972e-2956-484f-8514-69dcc9a48328"
-					(reference "C16")
-					(unit 1)
-				)
-				(path "/8d999898-5824-4200-a5bb-e5cd72e34b91/bfb47038-e30b-4456-8a3f-910a2a85c045"
-					(reference "C20")
-					(unit 1)
-				)
-				(path "/8d999898-5824-4200-a5bb-e5cd72e34b91/fffbe808-9aec-4c0c-a1ae-7f856729924e"
-					(reference "C18")
+					(reference "C31")
+					(unit 1)
+				)
+				(path "/8d999898-5824-4200-a5bb-e5cd72e34b91/bfb47038-e30b-4456-8a3f-910a2a85c045"
+					(reference "C32")
+					(unit 1)
+				)
+				(path "/8d999898-5824-4200-a5bb-e5cd72e34b91/fffbe808-9aec-4c0c-a1ae-7f856729924e"
+					(reference "C30")
 					(unit 1)
 				)
@@
 			)
 		)
-		(property "Reference" "F2"
+		(property "Reference" "F5"
 			(at 66.04 24.638 90)
 			(effects
@@
 			(project "many485"
 				(path "/8d999898-5824-4200-a5bb-e5cd72e34b91/b5d3972e-2956-484f-8514-69dcc9a48328"
-					(reference "F2")
+					(reference "F5")
 					(unit 1)
 				)
@@
 				)
 				(path "/8d999898-5824-4200-a5bb-e5cd72e34b91/fffbe808-9aec-4c0c-a1ae-7f856729924e"
-					(reference "F3")
+					(reference "F6")
 					(unit 1)
 				)
@@
 			)
 		)
-		(property "Reference" "U5"
+		(property "Reference" "U8"
 			(at 82.55 81.026 0)
 			(effects
@@
 			(project "many485"
 				(path "/8d999898-5824-4200-a5bb-e5cd72e34b91/b5d3972e-2956-484f-8514-69dcc9a48328"
-					(reference "U5")
-					(unit 1)
-				)
-				(path "/8d999898-5824-4200-a5bb-e5cd72e34b91/bfb47038-e30b-4456-8a3f-910a2a85c045"
+					(reference "U8")
+					(unit 1)
+				)
+				(path "/8d999898-5824-4200-a5bb-e5cd72e34b91/bfb47038-e30b-4456-8a3f-910a2a85c045"
+					(reference "U9")
+					(unit 1)
+				)
+				(path "/8d999898-5824-4200-a5bb-e5cd72e34b91/fffbe808-9aec-4c0c-a1ae-7f856729924e"
 					(reference "U7")
 					(unit 1)
 				)
-				(path "/8d999898-5824-4200-a5bb-e5cd72e34b91/fffbe808-9aec-4c0c-a1ae-7f856729924e"
-					(reference "U6")
-					(unit 1)
-				)
