File: F3:F303/InterfaceBoard/kicad/many485.kicad_pcb (KiCad board)
At the start: 2 copper layers, 79.5 x 84 mm, 116 parts, among them J1 Screw_Terminal_01x02, J10 Term_3, J11 Term_3, J12 Term_3, J13 Term_3, J14 SSI/422, J2 USB_B, J3 Prog, J4 HOLE, J5 HOLE, J6 HOLE, J7 HOLE, J8 Term_3, J9 Term_3, Q1 AO3401, Q2 B0505S-1W, Q3 B0505S-1W, Q4 B0505S-1W, Q5 B0505S-1W, Q6 B0505S-1W, Q7 B0505S-2W, SW1 SW_Push, SW2 SW_Push, SW3 SW_DIP_x01, SW4 SW_Push, U1 LM1117MP-3.3, U10 H11L1, U11 H11L1, U12 MAX3232, U13 ISO3086, U2 USBLC6-2SC6, U3 STM32F303RBT6, U4 ISO1050DUB, U5 ISO3088DW, U6 ISO3088DW, U7 ISO3088DW, U8 H11L1, U9 H11L1, Y1 8MHz

Commit message: finish, add gerbers
Parts:
- added G***: LOGO, my_footprints:QR, B.Cu at (108.2, 81.5)
- TP1: renamed from TP3; footprint Connector_PinSocket_2.54mm:PinSocket_1x01_P2.54mm_Vertical -> TestPoint:TestPoint_Loop_D2.54mm_Drill1.5mm_Beaded
- TP2: renamed from TP1; footprint Connector_PinSocket_2.54mm:PinSocket_1x01_P2.54mm_Vertical -> TestPoint:TestPoint_Loop_D2.54mm_Drill1.5mm_Beaded
- TP3: renamed from TP2; footprint Connector_PinSocket_2.54mm:PinSocket_1x01_P2.54mm_Vertical -> TestPoint:TestPoint_Loop_D2.54mm_Drill1.5mm_Beaded
- moved R7 0.59 mm to (145.5, 57.8)
- moved J1 0.50 mm to (74.0, 37.5)
- moved J4 0.50 mm to (74.0, 114.5)
- moved R6 0.41 mm to (112.6, 57.3)
- moved C7 0.35 mm to (145.7, 50.0)
- moved R3 0.35 mm to (145.7, 46.4)
- renumbered C28 to C1, C22 to C10, C23 to C11, C3 to C12, C1 to C13, C33 to C14, C32 to C15, C2 to C16, C7 to C17, C10 to C18, C5 to C19, C14 to C2, C8 to C20, C12 to C21, C9 to C22, C6 to C23, C11 to C24, C17 to C25, C15 to C26, C19 to C27, C30 to C28, C31 to C29, C25 to C3, C18 to C30, C16 to C31, C20 to C32, C26 to C4, C24 to C5, C27 to C6, C21 to C7, C29 to C8, C13 to C9, D3 to D1, D5 to D10, D4 to D11, D6 to D12, D10 to D2, D8 to D3, D9 to D4, D7 to D5, D12 to D6, D2 to D7, D11 to D8, D1 to D9, F5 to F2, F6 to F3, F2 to F5, F3 to F6, J5 to J1, J14 to J10, J2 to J11, J11 to J12, J9 to J13, J10 to J14, J4 to J2, J6 to J4, J7 to J5, J12 to J6, J13 to J7, J1 to J9, JP3 to JP1, JP1 to JP3, JP5 to JP4, JP4 to JP5, Q6 to Q3, Q7 to Q4, Q3 to Q6, Q4 to Q7, R9 to R1, R7 to R10, R8 to R11, R3 to R12, R1 to R13, R18 to R14, R2 to R15, R5 to R16, R4 to R17, R6 to R18, R17 to R2, R12 to R3, R11 to R4, R14 to R5, R15 to R6, R10 to R7, R13 to R8, R16 to R9, SW3 to SW1, SW4 to SW2, SW2 to SW3, SW1 to SW4, U4 to U1, U9 to U10, U10 to U11, U8 to U12, U11 to U13, U12 to U2, U13 to U3, U1 to U4, U2 to U5, U3 to U6, U6 to U7, U5 to U8, U7 to U9
Routing:
- net GND: track 851.1 -> 888.7 mm, vias 24 -> 25
- net /Isolated_485_2/gndi2: track 30.3 -> 40.6 mm
- net /Isolated_485_3/gndi2: track 30.3 -> 40.4 mm
- net /Isolated_485_01/gndi2: track 30.3 -> 40.4 mm
- net Net-(D2-A1): track 38.5 -> 37.2 mm
- net /Isolated_232/5Vloc5: track 77.7 -> 76.4 mm
- net /Isolated_232/5viso5: track 60.7 -> 59.9 mm
- net /232Rx1: track 67.7 -> 68.5 mm
- net /SSI_422/SSI_VR: track 33.7 -> 33.0 mm
- added copper zone on B.Cu, net GND
- added copper zone on F.Cu, net GND
Other:
- board size 79.5 x 84 mm -> 80 x 84 mm
- board text added: "232(1)"
- board text added: "232(2)"
- board text added: "3V3"
- board text added: "422"
- board text added: "485(1)"
- board text added: "485(2)"
- board text added: "485(3)"
- board text added: "5V"
- board text added: "B Gnd A"
- board text added: "B(-) Gnd A(+)"
- board text added: "Boot"
- board text added: "CAN"
- board text added: "CANL Gnd CANH"
- board text added: "Config mode"
- board text added: "Gnd"
- board text added: "Gnd +5V"
- board text added: "IF1"
- board text added: "IF2"
- board text added: "IF3"
- board text added: "IF4"
- board text added: "IF5"
- board text added: "IF6 CAN"
- board text added: "IF7"
- board text added: "RS- 232"
- board text added: "RS-232"
- board text added: "RS-422"
- board text added: "RS-485 (1)"
- board text added: "RS-485 (2)"
- board text added: "RS-485 (3)"
- board text added: "Reset"
- board text added: "Reset encoder on connect"
- board text added: "Rx"
- board text added: "SSI"
- board text added: "SSI/485 pinout: 1 - Gnd 2 - Y (R-) 3 - Z (R+) 4 - SSI_VR 5 - 5V 6 - A (T-) 7 - B (T+) 8 - SSI_Z 9 - Gnd"
- board text added: "SSI/RS-422"
- board text added: "SWCLK SWDIO GND 3V3 BOOT RESET"
- board text added: "Tx"
- board text added: "Tx Gnd Rx"
- board text added: "VR"
