File: F3:F303/InterfaceBoard/kicad/many485.kicad_sch (KiCad schematic)
At the start: 52 parts, among them J1 Screw_Terminal_01x02, J2 USB_B, J3 Prog, J4 HOLE, J5 HOLE, J6 HOLE, J7 HOLE, J8 Term_3, Q1 AO3401, Q2 B0505S-1W, SW1 SW_Push, SW2 SW_Push, SW3 SW_DIP_x01, U1 LM1117MP-3.3, U2 USBLC6-2SC6, U3 STM32F303RBT6, U4 ISO1050DUB, Y1 8MHz

Commit message: finish, add gerbers
Parts:
- TP1: renamed from TP3; footprint Connector_PinSocket_2.54mm:PinSocket_1x01_P2.54mm_Vertical -> TestPoint:TestPoint_Loop_D2.54mm_Drill1.5mm_Beaded
- TP2: renamed from TP1; footprint Connector_PinSocket_2.54mm:PinSocket_1x01_P2.54mm_Vertical -> TestPoint:TestPoint_Loop_D2.54mm_Drill1.5mm_Beaded
- TP3: renamed from TP2; footprint Connector_PinSocket_2.54mm:PinSocket_1x01_P2.54mm_Vertical -> TestPoint:TestPoint_Loop_D2.54mm_Drill1.5mm_Beaded
- renumbered C3 to C12, C1 to C13, C2 to C16, C7 to C17, C10 to C18, C5 to C19, C14 to C2, C8 to C20, C12 to C21, C9 to C22, C6 to C23, C11 to C24, C13 to C9, D3 to D1, D2 to D7, D1 to D9, J5 to J1, J2 to J11, J4 to J2, J6 to J4, J7 to J5, J1 to J9, JP3 to JP1, JP1 to JP3, JP5 to JP4, JP4 to JP5, R9 to R1, R7 to R10, R8 to R11, R3 to R12, R1 to R13, R2 to R15, R5 to R16, R4 to R17, R6 to R18, SW3 to SW1, SW2 to SW3, SW1 to SW4, U4 to U1, U1 to U4, U2 to U5, U3 to U6
Other:
- note added: "485-1"
- note added: "485-2"
- note added: "485-3"
