File: F3:F303/InterfaceBoard/kicad/ssi_422.kicad_sch (KiCad schematic)
At the start: 13 parts, among them J14 SSI{slash}422, Q7 B0505S-2W, SW4 SW_Push, U13 ISO3086

Commit message: finish, add gerbers
Parts:
- J10: renamed from J14; value SSI/422 -> SSI/422
- renumbered C33 to C14, C32 to C15, C30 to C28, C31 to C29, D12 to D6, D11 to D8, F6 to F3, Q7 to Q4, R18 to R14, SW4 to SW2, U13 to U3
Changed lines of the file:
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@@
 			)
 		)
-		(property "Reference" "C30"
+		(property "Reference" "C28"
 			(at 101.6 63.754 90)
 			(effects
@@
 			(project "many485"
 				(path "/8d999898-5824-4200-a5bb-e5cd72e34b91/80264a45-619f-4fbb-976c-6c15dcb432b8"
-					(reference "C30")
+					(reference "C28")
 					(unit 1)
 				)
@@
 			)
 		)
-		(property "Reference" "U13"
+		(property "Reference" "U3"
 			(at 117.094 56.896 0)
 			(effects
@@
 			(project "many485"
 				(path "/8d999898-5824-4200-a5bb-e5cd72e34b91/80264a45-619f-4fbb-976c-6c15dcb432b8"
-					(reference "U13")
+					(reference "U3")
 					(unit 1)
 				)
@@
 			)
 		)
-		(property "Reference" "R18"
+		(property "Reference" "R14"
 			(at 142.748 52.324 90)
 			(effects
@@
 			(project "many485"
 				(path "/8d999898-5824-4200-a5bb-e5cd72e34b91/80264a45-619f-4fbb-976c-6c15dcb432b8"
-					(reference "R18")
+					(reference "R14")
 					(unit 1)
 				)
@@
 			)
 		)
-		(property "Reference" "C33"
+		(property "Reference" "C14"
 			(at 194.31 48.26 0)
 			(effects
@@
 			(project "many485"
 				(path "/8d999898-5824-4200-a5bb-e5cd72e34b91/80264a45-619f-4fbb-976c-6c15dcb432b8"
-					(reference "C33")
+					(reference "C14")
 					(unit 1)
 				)
@@
 			)
 		)
-		(property "Reference" "D12"
+		(property "Reference" "D6"
 			(at 148.59 75.8909 0)
 			(effects
@@
 			(project "many485"
 				(path "/8d999898-5824-4200-a5bb-e5cd72e34b91/80264a45-619f-4fbb-976c-6c15dcb432b8"
-					(reference "D12")
+					(reference "D6")
 					(unit 1)
 				)
@@
 			)
 		)
-		(property "Reference" "C32"
+		(property "Reference" "C15"
 			(at 173.736 48.006 0)
 			(effects
@@
 			(project "many485"
 				(path "/8d999898-5824-4200-a5bb-e5cd72e34b91/80264a45-619f-4fbb-976c-6c15dcb432b8"
-					(reference "C32")
+					(reference "C15")
 					(unit 1)
 				)
@@
 			)
 		)
-		(property "Reference" "F6"
+		(property "Reference" "F3"
 			(at 168.91 53.848 90)
 			(effects
@@
 			(project "many485"
 				(path "/8d999898-5824-4200-a5bb-e5cd72e34b91/80264a45-619f-4fbb-976c-6c15dcb432b8"
-					(reference "F6")
+					(reference "F3")
 					(unit 1)
 				)
@@
 			)
 		)
-		(property "Reference" "C31"
+		(property "Reference" "C29"
 			(at 130.81 96.52 0)
 			(effects
@@
 			(project "many485"
 				(path "/8d999898-5824-4200-a5bb-e5cd72e34b91/80264a45-619f-4fbb-976c-6c15dcb432b8"
-					(reference "C31")
+					(reference "C29")
 					(unit 1)
 				)
@@
 			)
 		)
-		(property "Reference" "Q7"
+		(property "Reference" "Q4"
 			(at 182.88 40.4325 0)
 			(effects
@@
 			(project "many485"
 				(path "/8d999898-5824-4200-a5bb-e5cd72e34b91/80264a45-619f-4fbb-976c-6c15dcb432b8"
-					(reference "Q7")
+					(reference "Q4")
 					(unit 1)
 				)
@@
 			)
 		)
-		(property "Reference" "D11"
+		(property "Reference" "D8"
 			(at 148.59 61.9209 0)
 			(effects
@@
 			(project "many485"
 				(path "/8d999898-5824-4200-a5bb-e5cd72e34b91/80264a45-619f-4fbb-976c-6c15dcb432b8"
-					(reference "D11")
+					(reference "D8")
 					(unit 1)
 				)
@@
 			)
 		)
-		(property "Reference" "SW4"
+		(property "Reference" "SW2"
 			(at 139.7 54.3362 0)
 			(effects
@@
 			(project "many485"
 				(path "/8d999898-5824-4200-a5bb-e5cd72e34b91/80264a45-619f-4fbb-976c-6c15dcb432b8"
-					(reference "SW4")
+					(reference "SW2")
 					(unit 1)
 				)
@@
 			)
 		)
-		(property "Reference" "J14"
+		(property "Reference" "J10"
 			(at 196.85 67.31 0)
 			(effects
@@
 			)
 		)
-		(property "Value" "SSI{slash}422"
+		(property "Value" "SSI/422"
 			(at 191.516 94.869 0)
 			(effects
@@
 			(project "many485"
 				(path "/8d999898-5824-4200-a5bb-e5cd72e34b91/80264a45-619f-4fbb-976c-6c15dcb432b8"
-					(reference "J14")
-					(unit 1)
-				)
+					(reference "J10")
+					(unit 1)
+				)
