File: F3:F303/MLX90640-allsky/kicad/mainboard.kicad_pcb (KiCad board)
At the start: 2 copper layers, 388.5 x 80.5 mm, 93 parts, among them J1 Conn_01x03_Pin, J10 Conn_01x04_Socket, J11 Conn_01x04_Socket, J12 Conn_01x04_Socket, J13 Conn_01x04_Socket, J14 Conn_01x04_Socket, J15 Conn_01x04_Socket, J16 Prog, J17 hole, J18 hole, J19 hole, J2 Conn_01x03_Pin, J20 hole, J21 hole, J22 hole, J23 hole, J24 hole, J3 Conn_01x04_Pin, J4 Conn_01x02, J5 Conn_01x04_Socket, J8 Conn_01x04_Socket, J9 Conn_01x04_Socket, Q1 B1203S-1W, Q2 B1212S-1W, Q3 SI2300, U1 PC817, U2 PC817, U3 IP4220CZ6, U4 USBLC6-2SC6, U5 STM32F303CBTx, Y1 8MHz

Commit message: Almost finish PCB
Parts:
- removed the J4 at (70.7, 153.3)
- removed JP1, JP2, JP3, JP4: Jumper_2_Small_Open, Jumper:SolderJumper-2_P1.3mm_Open_TrianglePad1.0x1.5mm
- removed the R4 at (70.7, 144.9)
- removed the R8 at (87.6, 151.0)
- removed the U2 at (87.0, 155.5)
- added C11: 1u, Capacitor_SMD:C_0805_2012Metric_Pad1.18x1.45mm_HandSolder, F.Cu at (150.8, 116.5)
- added C14: 1u, Capacitor_SMD:C_0805_2012Metric_Pad1.18x1.45mm_HandSolder, B.Cu at (141.2, 104.6)
- added R1: x, Resistor_SMD:R_2010_5025Metric_Pad1.40x2.65mm_HandSolder, B.Cu at (119.2, 87.6)
- added R11: 330, Resistor_SMD:R_0603_1608Metric_Pad0.98x0.95mm_HandSolder, B.Cu at (145.3, 94.1)
- added R3: x, Resistor_SMD:R_2010_5025Metric_Pad1.40x2.65mm_HandSolder, B.Cu at (115.9, 87.6)
- added R5: x, Resistor_SMD:R_2010_5025Metric_Pad1.40x2.65mm_HandSolder, B.Cu at (112.6, 87.6)
- added R7: 20k, Resistor_SMD:R_0805_2012Metric_Pad1.20x1.40mm_HandSolder, B.Cu at (136.4, 94.6)
- added R9: 100k, Resistor_SMD:R_0805_2012Metric_Pad1.20x1.40mm_HandSolder, B.Cu at (136.4, 92.4)
- added U1: PC817, Package_DIP:DIP-4_W7.62mm, F.Cu at (147.3, 95.0)
- C10, C7, C8, C9: moved to F.Cu
- C13: renamed from C12; value 12 -> 6
- C16: renamed from C14; value 12 -> 6
- J2: footprint TerminalBlock_Phoenix:TerminalBlock_Phoenix_MKDS-1,5-3_1x03_P5.00mm_Horizontal -> TerminalBlock_Phoenix:TerminalBlock_Phoenix_MKDS-1,5-4_1x04_P5.00mm_Horizontal
- J3: footprint Connector_PinHeader_2.54mm:PinHeader_1x04_P2.54mm_Vertical -> Connector_PinHeader_2.54mm:PinHeader_1x06_P2.54mm_Vertical
- J4: renamed from J5; footprint Connector_PinHeader_2.54mm:PinHeader_1x04_P2.54mm_Vertical -> Connector_PinHeader_2.54mm:PinHeader_1x06_P2.54mm_Vertical
- R19: renamed from R15; moved to F.Cu
- R20: renamed from R16; moved to F.Cu
- R22: renamed from R18; moved to F.Cu
- R24: renamed from R20; moved to F.Cu
- R25: renamed from R21; moved to F.Cu
- R26: renamed from R22; moved to F.Cu
- R27: renamed from R23; moved to F.Cu
- Y1: value 8MHz -> NX5032GA-8MHz; footprint Crystal:Crystal_HC49-U_Vertical -> Crystal:Crystal_SMD_5032-2Pin_5.0x3.2mm; moved to B.Cu
- moved C13 372.5 mm to (124.5, 102.9), turned to -90 degrees
- moved C16 364.0 mm to (132.7, 102.9), turned to -90 degrees
- moved Y1 362.7 mm to (128.7, 102.0)
- moved R33 359.0 mm to (138.1, 103.7), turned to -90 degrees
- moved R31 358.0 mm to (121.9, 110.8), turned to 90 degrees
- moved J15 356.0 mm to (134.2, 100.7), turned to 90 degrees
- moved R32 353.8 mm to (130.8, 106.1)
- moved C18 353.4 mm to (124.9, 120.6)
- moved C15 343.9 mm to (135.3, 118.1), turned to 90 degrees
- moved C17 343.8 mm to (124.1, 108.2), turned to 180 degrees
- moved C12 334.6 mm to (134.2, 106.1)
- moved C6 294.7 mm to (152.2, 114.5), turned to 90 degrees
- moved RN1 292.0 mm to (151.6, 122.3), turned to 180 degrees
- moved Q3 279.2 mm to (129.1, 113.8), turned to 90 degrees
- moved R29 279.1 mm to (143.3, 127.3)
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- renumbered C11 to C12, C13 to C15, C15 to C17, C16 to C18, J11 to J10, J12 to J11, J13 to J12, J14 to J13, J15 to J14, J16 to J15, J17 to J16, J18 to J17, J19 to J18, J20 to J19, J21 to J20, J22 to J21, J23 to J22, J24 to J23, J6 to J5, J7 to J6, J8 to J7, J9 to J8, J10 to J9, R6 to R10, R7 to R12, R9 to R13, R10 to R14, R11 to R15, R12 to R16, R13 to R17, R14 to R18, R1 to R2, R17 to R21, R19 to R23, R24 to R28, R25 to R29, R26 to R30, R27 to R31, R28 to R32, R29 to R33, R2 to R4, R3 to R6, R5 to R8, U1 to U2
Connections:
- D3 pad 1: /MOSI -> /MISO
- D3 pad 4: /CS -> /MOSI
- D3 pad 5: /MISO -> /CS
- GD1 pad 1: Net-(J1-Pin_1) -> /12Vin
- GD1 pad 3: Net-(J1-Pin_3) -> /GNDin
- J1 pad 1: Net-(J1-Pin_1) -> /12Vin
- J1 pad 3: Net-(J1-Pin_3) -> /GNDin
- J2 pad 3: +12V -> Net-(J2-Pin_3)
- L1 pad 1: Net-(J1-Pin_1) -> /12Vin
- L1 pad 4: Net-(J1-Pin_3) -> /GNDin
- R10 pad 1: Net-(J2-Pin_2) -> Net-(J2-Pin_4)
- R2 pad 1: Net-(J2-Pin_1) -> Net-(J2-Pin_3)
- R2 pad 2: Net-(JP2-A) -> /GNDin
- R4 pad 1: Net-(J2-Pin_1) -> Net-(J2-Pin_3)
- R4 pad 2: Net-(JP2-A) -> /GNDin
- R6 pad 1: Net-(JP1-B) -> Net-(J2-Pin_3)
- R6 pad 2: Net-(JP2-B) -> /GNDin
- R8 pad 1: Net-(J2-Pin_2) -> Net-(J2-Pin_4)
- R8 pad 2: GND1 -> /GNDin
- RV1 pad 1: Net-(J1-Pin_3) -> /GNDin
- RV1 pad 2: Net-(J1-Pin_1) -> /12Vin
- U2 pad 4: +12V -> /12Vin
- U3 pad 1: /AIN1 -> /AIN2
- U3 pad 3: /AIN2 -> /AIN1
- U3 pad 4: /AIN4 -> /AIN3
- U3 pad 6: /AIN3 -> /AIN4
- U5 pad 20: /CS -> unconnected-(U5-PB2-Pad20)
- U5 pad 46: unconnected-(U5-PB9-Pad46) -> /CS
Routing:
- net GND: track 0.00 -> 422.3 mm, vias 0 -> 25
- net +3.3V: track 0.00 -> 197.6 mm, vias 0 -> 9
- net +12VA: track 0.00 -> 92.4 mm, vias 0 -> 2
- net /GNDin: track 0.00 -> 92.0 mm
- net /12Vin: track 0.00 -> 80.3 mm
- net /PWM2: track 0.00 -> 62.1 mm, vias 0 -> 3
- net /PWM1: track 0.00 -> 59.0 mm, vias 0 -> 3
- net /SCL: track 0.00 -> 35.1 mm, vias 0 -> 4
- net /SDA: track 0.00 -> 33.7 mm, vias 0 -> 4
- net /TX: track 0.00 -> 32.7 mm, vias 0 -> 2
- net /AIN1: track 0.00 -> 31.2 mm, vias 0 -> 3
- net /dio: track 0.00 -> 30.4 mm, vias 0 -> 1
- net /AIN2: track 0.00 -> 29.5 mm, vias 0 -> 3
- net /PWM4: track 0.00 -> 28.8 mm
- net /PWM3: track 0.00 -> 28.1 mm, vias 0 -> 2
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- added copper zone on B.Cu, net GND
- added copper zone on F.Cu, net GND
Other:
- board size 388.5 x 80.5 mm -> 58 x 71 mm
- board text added: "+12V"
- board text added: "1"
- board text added: "12V"
- board text added: "3V3 SCL SDA Gnd"
- board text added: "3v3"
- board text added: "6"
- board text added: "BME280"
- board text added: "Earth"
- board text added: "G1"
- board text added: "G2"
- board text added: "Gnd"
- board text added: "Gnd USBDP USBDM 5V"
- board text added: "I2C bus to sensors"
- board text added: "NTC1 NTC2"
- board text added: "NTC4 NTC3"
- board text added: "NTC: 1,2 NTC1/4 3,4 NTC2/3"
- board text added: "PWM1"
- board text added: "PWM2"
- board text added: "Prog"
- board text added: "S1"
- board text added: "S2"
- board text added: "SWCLK SWDIO Gnd +3V3 NC NC"
- board text added: "UART"
- board text added: "UART: 1 Gnd 2 +12V 3 Video1 4 Video2 5 Tx 6 Rx"
- board text added: "Vcc Gnd SDI SCK CSB SDO"
