File: F3:F303/MLX90640-allsky/kicad/mainboard.kicad_sch (KiCad schematic)
At the start: 93 parts, among them J1 Conn_01x03_Pin, J10 Conn_01x04_Socket, J11 Conn_01x04_Socket, J12 Conn_01x04_Socket, J13 Conn_01x04_Socket, J14 Conn_01x04_Socket, J15 Conn_01x04_Socket, J16 Prog, J17 hole, J18 hole, J19 hole, J2 Conn_01x03_Pin, J20 hole, J21 hole, J22 hole, J23 hole, J24 hole, J3 Conn_01x04_Pin, J4 Conn_01x02, J5 Conn_01x04_Socket, J8 Conn_01x04_Socket, J9 Conn_01x04_Socket, Q1 B1203S-1W, Q2 B1212S-1W, Q3 SI2300, U1 PC817, U2 PC817, U3 IP4220CZ6, U4 USBLC6-2SC6, U5 STM32F303CBTx, Y1 8MHz

Commit message: Almost finish PCB
Parts:
- removed J4: Conn_01x02, Connector_PinHeader_2.54mm:PinHeader_1x02_P2.54mm_Vertical, symbol Connector_Generic:Conn_01x02
- removed JP1, JP2, JP3, JP4: Jumper_2_Small_Open, Jumper:SolderJumper-2_P1.3mm_Open_TrianglePad1.0x1.5mm, symbol Jumper:Jumper_2_Small_Open
- removed R4: x, Resistor_SMD:R_2010_5025Metric_Pad1.40x2.65mm_HandSolder, symbol Device:R
- removed R8: 330, Resistor_SMD:R_0603_1608Metric_Pad0.98x0.95mm_HandSolder, symbol Device:R
- removed U2: PC817, Package_DIP:DIP-4_W7.62mm, symbol Isolator:PC817
- added C11, C14: 1u, Capacitor_SMD:C_0805_2012Metric_Pad1.18x1.45mm_HandSolder, symbol Device:C
- added R1, R3, R5: x, Resistor_SMD:R_2010_5025Metric_Pad1.40x2.65mm_HandSolder, symbol Device:R
- added R11: 330, Resistor_SMD:R_0603_1608Metric_Pad0.98x0.95mm_HandSolder, symbol Device:R
- added R7: 20k, Resistor_SMD:R_0805_2012Metric_Pad1.20x1.40mm_HandSolder, symbol Device:R
- added R9: 100k, Resistor_SMD:R_0805_2012Metric_Pad1.20x1.40mm_HandSolder, symbol Device:R
- added U1: PC817, Package_DIP:DIP-4_W7.62mm, symbol Isolator:PC817
- C13: renamed from C12; value 12 -> 6
- C16: renamed from C14; value 12 -> 6
- J2: footprint TerminalBlock_Phoenix:TerminalBlock_Phoenix_MKDS-1,5-3_1x03_P5.00mm_Horizontal -> TerminalBlock_Phoenix:TerminalBlock_Phoenix_MKDS-1,5-4_1x04_P5.00mm_Horizontal; symbol Connector:Screw_Terminal_01x03 -> Connector:Screw_Terminal_01x04
- J3: footprint Connector_PinHeader_2.54mm:PinHeader_1x04_P2.54mm_Vertical -> Connector_PinHeader_2.54mm:PinHeader_1x06_P2.54mm_Vertical; symbol Connector:Conn_01x04_Pin -> Connector:Conn_01x06_Pin
- J4: renamed from J5; footprint Connector_PinHeader_2.54mm:PinHeader_1x04_P2.54mm_Vertical -> Connector_PinHeader_2.54mm:PinHeader_1x06_P2.54mm_Vertical; symbol Connector:Conn_01x04_Socket -> Connector:Conn_01x06_Pin
- Y1: value 8MHz -> NX5032GA-8MHz; footprint Crystal:Crystal_HC49-U_Vertical -> Crystal:Crystal_SMD_5032-2Pin_5.0x3.2mm
- renumbered C11 to C12, C13 to C15, C15 to C17, C16 to C18, J11 to J10, J12 to J11, J13 to J12, J14 to J13, J15 to J14, J16 to J15, J17 to J16, J18 to J17, J19 to J18, J20 to J19, J21 to J20, J22 to J21, J23 to J22, J24 to J23, J6 to J5, J7 to J6, J8 to J7, J9 to J8, J10 to J9, R6 to R10, R7 to R12, R9 to R13, R10 to R14, R11 to R15, R12 to R16, R13 to R17, R14 to R18, R15 to R19, R1 to R2, R16 to R20, R17 to R21, R18 to R22, R19 to R23, R20 to R24, R21 to R25, R22 to R26, R23 to R27, R24 to R28, R25 to R29, R26 to R30, R27 to R31, R28 to R32, R29 to R33, R2 to R4, R3 to R6, R5 to R8, U1 to U2
Connections:
- net +12V: no longer J2.3 (Pin_3), U2.4
- net +3.3V: now also C11.1, C14.1, R11.2
- net AIN1: now also U3.3 (I/O2); no longer U3.1 (I/O1)
- net AIN2: now also U3.1 (I/O1); no longer U3.3 (I/O2)
- net AIN3: now also U3.4 (I/O2); no longer U3.6 (I/O1)
- net AIN4: now also U3.6 (I/O1); no longer U3.4 (I/O2)
- net CS: now also D3.5 (K), U5.46 (PB9); no longer D3.4 (K), U5.20 (PB2)
- net GND: now also C11.2, C14.2
- net GND1: no longer R8.2
- net MISO: now also D3.1 (K); no longer D3.5 (K)
- net MOSI: now also D3.4 (K); no longer D3.1 (K)
- net PWM1: now also J3.5 (Pin_5), J4.5 (Pin_5)
- net PWM2: now also J3.6 (Pin_6), J4.6 (Pin_6), U1.2
- net at R6.1: now also J2.3 (Pin_3), R2.1, R4.1
- net 12Vin: now reaches GD1.1, J1.1 (Pin_1), L1.1, RV1.2
- net 12Vin: now also U2.4, U1.4
- net GNDin: now reaches GD1.3, J1.3 (Pin_3), L1.4, RV1.1
- net GNDin: now also R2.2, R4.2, R6.2, R8.2, R1.2, R3.2, R5.2, R7.2
- net at R10.1, R8.1: now also J2.4 (Pin_4); no longer J2.2 (Pin_2)
- new net: R11.1, U1.1
- new net: R9.2, U1.3
- new net: J2.1 (Pin_1), R1.1, R3.1, R5.1
- new net: J2.2 (Pin_2), R7.1, R9.1
Other:
- note added: "Gate1 Source1 Gate2 Source2"
- note added: "NTC3 gnd3 NTC4 gnd4"
- note removed: "Drain Gate Source"
- note removed: "NTC4 gnd4 NTC3 gnd3"
- note removed: "Optional PWM output"
- moved on the sheet: D3, R2, R4, R6, R8
