File: F1:F103/FX3U/kicad/fx3u_24mr.kicad_sch (KiCad schematic)
At the start: 14 parts, among them J1 Conn_01x05_Pin, SW1 SW_SPDT, U1 STM32F103VCTx, U2 SP3485CN, U3 ULN2003, U4 ULN2003

Commit message: Almost finish schematics
Parts:
- removed R3, R4: 2k, Resistor_SMD:R_0603_1608Metric_Pad0.98x0.95mm_HandSolder, symbol Device:R
- removed SW1: SW_SPDT, symbol Switch:SW_SPDT
- added C1, C2, C3, C4: 1000u, Capacitor_THT:CP_Radial_D14.0mm_P7.50mm, symbol Device:C_Polarized
- added C10, C14, C17, C20, C21, C22, C23, C24, C25, C31, C32, C33, C5, C6, C8: 0.1, Capacitor_SMD:C_0603_1608Metric_Pad1.08x0.95mm_HandSolder, symbol Device:C
- added C11, C7, C9: 10u, Capacitor_SMD:C_0805_2012Metric_Pad1.18x1.45mm_HandSolder, symbol Device:C
- added C12: 100u, Capacitor_Tantalum_SMD:CP_EIA-3528-12_Kemet-T_Pad1.50x2.35mm_HandSolder, symbol Device:C_Polarized
- added C13, C15, C16, C18, C19: 1u, Capacitor_SMD:C_0805_2012Metric_Pad1.18x1.45mm_HandSolder, symbol Device:C
- added C26, C27, C28, C29, C30: 6?, Capacitor_SMD:C_0805_2012Metric_Pad1.18x1.45mm_HandSolder, symbol Device:C
- added D17: Power, LED_SMD:LED_0805_2012Metric_Pad1.15x1.40mm_HandSolder, symbol Device:LED
- added D18, D19: M7, Diode_SMD:D_SMA_Handsoldering, symbol Device:D_Zener
- added D20: SMBJ30A, Diode_SMD:D_SMB, symbol Diode:SMAJ30A
- added D21: SS24, Diode_SMD:D_SMA_Handsoldering, symbol Device:D_Schottky
- added D22: SS14, Diode_SMD:D_SMA_Handsoldering, symbol Device:D_Schottky
- added D23, D24: SM6T6V8A, Diode_SMD:D_SMB, symbol Diode:SM6T6V8A
- added F1: U110-TAER, symbol Device:Fuse
- added J2: DC, symbol Connector:Conn_01x02_Socket
- added J3: DE9_Receptacle, Connector_Dsub:DSUB-9_Female_Vertical_P2.77x2.84mm, symbol Connector:DE9_Receptacle
- added J4: RS485, symbol Connector:Conn_01x02_Socket
- added L1: JY_B32, symbol Device:L_Coupled_1243
- added L2: 68, Inductor_SMD:L_10.4x10.4_H4.8, symbol Device:L_Ferrite
- added R47: 510, Resistor_SMD:R_0603_1608Metric_Pad0.98x0.95mm_HandSolder, symbol Device:R
- added R48, R49, R50, R57: 4.7k, Resistor_SMD:R_0603_1608Metric_Pad0.98x0.95mm_HandSolder, symbol Device:R
- added R51, R52, R53: 10k, Resistor_SMD:R_0603_1608Metric_Pad0.98x0.95mm_HandSolder, symbol Device:R
- added R54: 0, Resistor_SMD:R_0603_1608Metric_Pad0.98x0.95mm_HandSolder, symbol Device:R
- added R55: 470, Resistor_SMD:R_0603_1608Metric_Pad0.98x0.95mm_HandSolder, symbol Device:R
- added R56: 6.2k, Resistor_SMD:R_0603_1608Metric_Pad0.98x0.95mm_HandSolder, symbol Device:R
- added SW3: SW_DPDT_x2, Button_Switch_THT:SW_CK_JS202011CQN_DPDT_Straight, symbol Switch:SW_DPDT_x2
- added U19: AMS1117-3.3, Package_TO_SOT_SMD:SOT-223-3_TabPin2, symbol Regulator_Linear:AMS1117-3.3
- added U20: SP3232, Package_SO:SOIC-16_3.9x9.9mm_P1.27mm, symbol Interface_UART:MAX3232
- added U21: BL3085, Package_SO:SOIC-8_3.9x4.9mm_P1.27mm, symbol Interface_UART:SSP3085
- added U22: ATMLH202-64DM, Package_SO:SOIC-8_3.9x4.9mm_P1.27mm, symbol Memory_EEPROM:AT24CS64-SSHM
- added U23: EL817, Package_DIP:DIP-4_W7.62mm, symbol Isolator:EL817
- added U5: XL1509-5.0, Package_SO:SOIC-8_3.9x4.9mm_P1.27mm, symbol Regulator_Switching:XL1509-5.0
- added Y1: 8MHz, Crystal:Crystal_HC49-U_Vertical, symbol Device:Crystal
- added Y2: 32768, Crystal:Crystal_HC49-U_Vertical, symbol Device:Crystal
- D2: value 15V -> M7; footprint (none) -> Diode_SMD:D_SMA_Handsoldering
- R2: value 2k -> 510
- RV1, RV2: value pot -> 10k; footprint (none) -> Potentiometer_THT:Potentiometer_Bourns_3386F_Vertical
Connections:
- net +3.3V: now also C12.1, C13.2, C17.2, C20.1, C21.1, C22.1, C23.1, C24.1, C25.1, C8.1, C9.1, R47.2, R51.1, R52.1, R53.2, SW3.1 (A), SW3.4 (A), U19.2 (VO), U20.16 (VCC), U22.8 (VCC), U23.4
- net +5V: now also C10.1, C11.1, C14.2, D22.1 (K), R48.1, R50.1, U19.3 (VI), U21.8 (VCC)
- net DE_485: now also R48.2, U21.2 (~{RE}), U21.3 (DE)
- net GND: now also U3.8 (GND), U4.8 (GND), C1.2, C10.2, C11.2, C12.2, C13.1, C14.1, C17.1, C18.2, C19.2, C2.2, C20.2, C21.2, C22.2, C23.2, C24.2, C25.2, C26.2, C27.2, C28.1, C29.1, C3.2, C30.2, C31.2, C32.2, C33.2, C4.2, C5.2, C6.2, C7.2, C8.2, C9.2, D17.1 (K), D20.2 (A2), D21.2 (A), D23.2 (A2), D24.2 (A2), J3.5, L1.3, R49.2, R54.1, R55.1, R57.2, SW3.3 (C), SW3.6 (C), U19.1 (GND), U20.15 (GND), U22.1 (A0), U22.2 (A1), U22.3 (A2), U22.4 (GND), U22.7 (WP), U23.2, U5.4 (~{EN}), U5.5 (GND), U5.6 (GND), U5.7 (GND), U5.8 (GND); no longer U1.61 (PD14)
- net NRST: now also C30.1, R53.1
- net POW_DET: now also C31.1, R57.1, U23.3
- net PROG_SW: now also SW3.2 (B)
- net Rx_232: now also U20.9 (R2OUT)
- net Rx_485: now also U21.1 (RO)
- net SWDIO: now also R52.2, U22.5 (SDA)
- net Tx_232: now also U20.10 (T2IN)
- net Tx_485: now also U21.4 (DI)
- net Y0: now also U4.7 (I7)
- net Y1: now also U4.6 (I6)
- net Y10: now also U3.6 (I6)
- net Y11: now also U3.5 (I5)
- net Y2: now also U4.5 (I5)
- net Y3: now also U4.4 (I4)
- net Y4: now also U4.3 (I3)
- net Y5: now also U4.2 (I2)
- net Y6: now also U4.1 (I1)
- net Y7: now also U3.7 (I7)
- net R7: now reaches U3.10 (O7)
- net R10: now reaches U3.11 (O6)
- net R11: now reaches U3.12 (O5)
- net relay_24: now reaches U3.9 (COM)
- net relay_24: now also D2.1 (K), U4.9 (COM), C32.1, C33.1
- net R0: now reaches U4.10 (O7)
- net R1: now reaches U4.11 (O6)
- net R2: now reaches U4.12 (O5)
- net R3: now reaches U4.13 (O4)
- net R4: now reaches U4.14 (O3)
- net R5: now reaches U4.15 (O2)
- net R6: now reaches U4.16 (O1)
- net 24O: now reaches D2.2 (A)
- net 24O: now also D18.2 (A), D19.1 (K), D20.1 (A1), R56.2
- net at U1.12 (OSC_IN): now also C29.2, Y1.1
- net at U1.13 (OSC_OUT): now also C28.2, Y1.2
- net EEPROM_SCL: now reaches U1.77 (PA15)
- net EEPROM_SCL: now also R51.2, U22.6 (SCL)
- net at U1.8 (PC14): now also C26.1, Y2.1
- net at U1.9 (PC15): now also C27.1, Y2.2
- new net: C15.1, U20.1 (C1+)
- new net: C15.2, U20.3 (C1-)
- new net: R55.2, R56.1, U23.1
- new net: D17.2 (A), R47.1
- new net: C18.1, U20.2 (VS+)
- new net: C16.1, U20.4 (C2+)
- new net: C16.2, U20.5 (C2-)
- new net: C19.1, U20.6 (VS-)
- new net: J3.2, U20.7 (T2OUT)
- new net: J3.3, U20.8 (R2IN)
- new net: C2.1, C5.1, D21.1 (K), D22.2 (A), L2.1, U5.2 (OUT)
- new net: F1.1, J2.2 (Pin_2)
- new net: F1.2, L1.1
- new net: D23.1 (A1), J4.1 (Pin_1), R49.1, U21.6 (A)
- new net: D24.1 (A1), J4.2 (Pin_2), R50.2, U21.7 (B)
- new net: D19.2 (A), L1.2
- new net: J2.1 (Pin_1), L1.4
- new net: L2.2, U5.3 (FB)
- new net: R54.2, U1.61 (PD14)
- new net +24V: C1.1, C3.1, C4.1, C6.1, C7.1, D18.1 (K), U5.1 (VIN)
- no-connect marks 0 -> 18
Other:
- added sheet Y_relay (Y_relay.kicad_sch)
- added sheet Y_relay1 (Y_relay.kicad_sch)
- added sheet Y_relay2 (Y_relay.kicad_sch)
- added sheet Y_relay3 (Y_relay.kicad_sch)
- added sheet Y_relay4 (Y_relay.kicad_sch)
- added sheet Y_relay5 (Y_relay.kicad_sch)
- added sheet Y_relay6 (Y_relay.kicad_sch)
- added sheet Y_relay7 (Y_relay.kicad_sch)
- added sheet Y_relay8 (Y_relay.kicad_sch)
- added sheet Y_relay9 (Y_relay.kicad_sch)
- note added: "24O is power for EL817 inputs"
- note added: "38400/9600"
- moved on the sheet: D1, R2, U3

Commit message: End schematics
Parts:
- removed U2: SP3485CN, Package_SO:SOIC-8_3.9x4.9mm_P1.27mm, symbol Interface_UART:SP3485CN
- added BT1: CR1220, symbol Device:Battery_Cell
- added C34, C35, C36, C39, C40: 0.1, Capacitor_SMD:C_0603_1608Metric_Pad1.08x0.95mm_HandSolder, symbol Device:C
- added C37, C38, C41: 10u, Capacitor_SMD:C_1210_3225Metric_Pad1.33x2.70mm_HandSolder, symbol Device:C
- added D35, D36: schottky, Diode_SMD:D_1206_3216Metric_Pad1.42x1.75mm_HandSolder, symbol Device:D_Schottky
- added D37, D38: SM6T6V8A, Diode_SMD:D_SMB, symbol Diode:SM6T6V8A
- added J5: CAN, symbol Connector:Conn_01x02_Socket
- added J6: Xin, symbol Connector:Conn_01x15_Socket
- added J7: Yout, symbol Connector:Conn_01x13_Socket
- added J8: Analog, symbol Connector:Conn_01x10_Socket
- added R100, R103, R85, R86, R90, R92, R95, R97: 4.7k, Resistor_SMD:R_0603_1608Metric_Pad0.98x0.95mm_HandSolder, symbol Device:R
- added R101, R93, R98: 499, Resistor_SMD:R_1210_3225Metric_Pad1.30x2.65mm_HandSolder, symbol Device:R
- added R102, R81, R82, R83, R84, R89, R91, R94, R96, R99: 10k, Resistor_SMD:R_0603_1608Metric_Pad0.98x0.95mm_HandSolder, symbol Device:R
- added R80: 120, Resistor_SMD:R_0805_2012Metric_Pad1.20x1.40mm_HandSolder, symbol Device:R
- added R87, R88: 120, Resistor_SMD:R_0603_1608Metric_Pad0.98x0.95mm_HandSolder, symbol Device:R
- added U24: TJA1050, Package_SO:SOIC-8_3.9x4.9mm_P1.27mm, symbol Interface_CAN_LIN:TJA1051T
- added U25: LM358, Package_SO:SO-8_3.9x4.9mm_P1.27mm, symbol Amplifier_Operational:LM358
- J1: value Conn_01x05_Pin -> Prog
- J3: value DE9_Receptacle -> 232
Connections:
- net +3.3V: now also D36.2 (A)
- net +5V: now also C34.2, U24.3 (VCC)
- net 24O: now also U25.8 (V+)
- net ADC0: now also C37.2, R89.1, R90.2
- net ADC1: now also C38.2, R94.1, R95.2
- net ADC2: now also C41.2, R96.1, R97.2
- net ADC3: now also R91.1, R92.2
- net ADC4: now also R100.2, R99.1
- net ADC5: now also R102.1, R103.2
- net COM0: now also J7.1 (Pin_1)
- net COM1: now also J7.6 (Pin_6)
- net COM2: now also J7.11 (Pin_11)
- net DAC0: now also R81.1
- net DAC1: now also R82.1
- net GND: now also U21.5 (GND), BT1.2 (-), C34.1, C35.2, C36.2, C37.1, C38.1, C39.1, C40.1, C41.1, D37.2 (A2), D38.2 (A2), J6.1 (Pin_1), J8.1 (Pin_1), J8.8 (Pin_8), R100.1, R101.2, R103.1, R85.1, R86.1, R90.1, R92.1, R93.2, R95.1, R97.1, R98.2, U24.2 (GND), U24.8 (S), U25.4 (V-)
- net Rx_CAN: now also U24.4 (RXD)
- net Tx_CAN: now also U24.1 (TXD)
- net YY0: now also J7.2 (Pin_2)
- net YY1: now also J7.3 (Pin_3)
- net YY10: now also J7.12 (Pin_12)
- net YY11: now also J7.13 (Pin_13)
- net YY2: now also J7.4 (Pin_4)
- net YY3: now also J7.5 (Pin_5)
- net YY4: now also J7.7 (Pin_7)
- net YY5: now also J7.8 (Pin_8)
- net YY6: now also J7.9 (Pin_9)
- net YY7: now also J7.10 (Pin_10)
- net BAT: now reaches U1.6 (VBAT)
- net BAT: now also D35.1 (K), D36.1 (K)
- new net: D38.1 (A1), J5.2 (Pin_2), R80.1, U24.6 (CANL)
- new net: D37.1 (A1), J5.1 (Pin_1), R80.2, U24.7 (CANH)
- new net: C36.1, R82.2, U25.5 (+)
- new net: R84.1, R86.2, U25.6 (-)
- new net: R84.2, R88.1, U25.7
- new net: R83.2, R87.1, U25.1
- new net: R83.1, R85.2, U25.2 (-)
- new net: C35.1, R81.2, U25.3 (+)
- new net: BT1.1 (+), D35.2 (A)
- new net ADi0: J8.2 (Pin_2), R89.2
- new net ADi1: J8.3 (Pin_3), R94.2
- new net ADi2: J8.4 (Pin_4), R96.2
- new net ADi3: J8.5 (Pin_5), R91.2, R93.1
- new net ADi4: J8.6 (Pin_6), R98.1, R99.2
- new net ADi5: J8.7 (Pin_7), R101.1, R102.2
- new net DAo0: C39.2, J8.9 (Pin_9), R87.2
- new net DAo1: C40.2, J8.10 (Pin_10), R88.2
- new net XX0: J6.2 (Pin_2)
- new net XX1: J6.3 (Pin_3)
- new net XX10: J6.10 (Pin_10)
- new net XX11: J6.11 (Pin_11)
- new net XX12: J6.12 (Pin_12)
- new net XX13: J6.13 (Pin_13)
- new net XX14: J6.14 (Pin_14)
- new net XX15: J6.15 (Pin_15)
- new net XX2: J6.4 (Pin_4)
- new net XX3: J6.5 (Pin_5)
- new net XX4: J6.6 (Pin_6)
- new net XX5: J6.7 (Pin_7)
- new net XX6: J6.8 (Pin_8)
- new net XX7: J6.9 (Pin_9)
- no-connect marks 18 -> 52
Other:
- note added: "3.3V power"
- note added: "5V power"
- note added: "ANALOG"
- note added: "Analog inputs"
- note added: "BAT"
- note added: "CAN bus"
- note added: "DAC output"
- note added: "Discrete inputs"
- note added: "Discrete outputs"
- note added: "EEPROM"
- note added: "INTERFACES"
- note added: "LEDs"
- note added: "MCU AND STUFF"
- note added: "Optional!"
- note added: "POWER"
- note added: "Power detect"
- note added: "Power input"
- note added: "Prog"
- note added: "RS-232"
- note added: "RS-485"
- moved on the sheet: C1, C10, C11, C12, C13, C14, C15, C16, C17, C18, C19, C2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
