File: F1:F103/FX3U/kicad/fx3u_24mr.kicad_sch (KiCad schematic)
At the start: 120 parts, among them J1 Prog, J2 DC, J3 232, J4 RS485, J5 CAN, J6 Xin, J7 Yout, J8 Analog, SW3 SW_DPDT_x2, U1 STM32F103VCTx, U19 AMS1117-3.3, U20 SP3232, U21 BL3085, U22 ATMLH202-64DM, U23 EL817, U24 TJA1050, U25 LM358, U3 ULN2003, U4 ULN2003, U5 XL1509-5.0, Y1 8MHz, Y2 32768

Commit message: fixed schematics
Parts:
- D18, D19, D2: value M7 -> 1N4007
- D23, D24, D37, D38: value SM6T6V8A -> P6SMB6.8; symbol Diode:SM6T6V8A -> Device:D_TVS
- D35, D36: value schottky -> 1N4148?
Other:
- note added: "(COM)"
- note added: "(Imax = 20mA)"
- note added: "Analog inputs (Umax = 10V)"
- note added: "DAC output (1mA max; 0..10V)"
- note added: "U_{Out} ≈ 3 U_{In}"
- note removed: "Analog inputs"
- note removed: "DAC output"
